Commit message: introduction of scaling factor

File: foot_control_xy/models/h_lower_limb/urdf/h_lower_limb.urdf (robot description, URDF)
Before this commit: robot h_lower_limb, 1 links, 0 joints
Links:
- removed link chaser_base_link
- added link chaser/base_link, mass 1; collision sphere radius=0.25; visual mesh filename=package://foot_control_xy/models/h_lower_limb/meshes/foot.d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 scale=0.05 0.05 0.05

File: foot_control_xy/models/h_lower_limb/urdf/h_lower_limb.urdf.xacro (robot description, xacro)
@@ -1,5 +1,7 @@
 <?xml version="1.0"?>
 <robot xmlns:xacro="http://ros.org/wiki/xacro" name="h_lower_limb">
-  <xacro:property name="scale" value="${0.05}"/>
+	  <xacro:arg name="_scale" default="0.5"/>
+	  <xacro:arg name="_enableWorldTf" default="false"/>
+	  <xacro:property name="_radius" value="${0.25* $(arg _scale)}"/>
   <link
     name="chaser/base_link">
@@ -20,24 +22,26 @@
     <collision>
       <origin
-        xyz="0 0 0"
+        xyz="0 0 0.25"
         rpy="0 0 0" />
       <geometry>
-        <sphere radius="0.25"/>
+        <sphere radius="${_radius}"/>
       </geometry>
     </collision>
     <visual>
       <origin
-        xyz="0 0 0"
-        rpy="0 0 3.1415" /> <!--${pi/2}  ${-pi} 0-->
+        xyz="0 0 ${2*_radius}"
+        rpy="0 0 3.1415"/>
       <geometry>
         <mesh
-          filename="package://foot_control_xy/models/h_lower_limb/meshes/foot.dae" scale="${scale} ${scale} ${scale}"/>
+          filename="package://foot_control_xy/models/h_lower_limb/meshes/foot.dae" scale="${0.05*$(arg _scale)} ${0.05*$(arg _scale)} ${0.05*$(arg _scale)}"/>
       </geometry>
     </visual>
   </link>
-  <gazebo>
-   <plugin name="gzTfUpdate" filename="libgzTfUpdate.so">
-		<actorName>chaser</actorName>
-   </plugin>
-  </gazebo>
+    <xacro:if value="$(arg _enableWorldTf)">
+	  <gazebo>
+	   <plugin name="gzTfUpdate" filename="libgzTfUpdate.so">
+			<actorName>chaser</actorName>
+	   </plugin>
+	  </gazebo>
+  </xacro:if>
 </robot>

File: foot_control_xy/models/number1/urdf/number1.urdf.xacro (robot description, xacro)
@@ -1,4 +1,7 @@
 <?xml version="1.0"?>
 <robot xmlns:xacro="http://ros.org/wiki/xacro" name="number1">
+	<xacro:arg name="_enableWorldTf" default="false"/>
+    <xacro:arg name="_scale" default="0.5"/>
+    <xacro:property name="_radius" value="${0.25* $(arg _scale)}"/>
   <link
     name="target/base_link">
@@ -19,24 +22,26 @@
     <collision>
       <origin
-        xyz="0 0 0"
+        xyz="0 0 ${2*_radius}"
         rpy="0 0 0" />
       <geometry>
-        <sphere radius="0.25"/>
+        <box size="${_radius}"/>
       </geometry>
     </collision>
       <visual name="visual">
 		<origin
-		xyz="0 0 0"
+		xyz="0 0 ${2*_radius}"
         rpy="0 0 -1.5707963267" />
         <geometry>
           <mesh
-            filename="package://foot_control_xy/models/number1/meshes/number.dae"/>
+            filename="package://foot_control_xy/models/number1/meshes/number.dae" scale="$(arg _scale) $(arg _scale) $(arg _scale)"/>
         </geometry>
       </visual>
   </link>
-   <gazebo>
-   <plugin name="gzTfUpdate" filename="libgzTfUpdate.so">
-		<actorName>target</actorName>
-   </plugin>
-  </gazebo>
+    <xacro:if value="$(arg _enableWorldTf)">
+	   <gazebo>
+	   <plugin name="gzTfUpdate" filename="libgzTfUpdate.so">
+			<actorName>target</actorName>
+	   </plugin>
+	  </gazebo>
+  </xacro:if>
 </robot>
