Commit message: last commit 20-feb

File: foot_control_xy/models/h_lower_limb/urdf/h_lower_limb.urdf.xacro (robot description, xacro)
@@ -1,12 +1,11 @@
 <?xml version="1.0"?>
 <robot xmlns:xacro="http://ros.org/wiki/xacro" name="h_lower_limb">
-  <xacro:property name="foot_lenght" value="0.266"/><!--size 43-->
-  <xacro:property name="foot_girth" value="0.110"/>
-  <xacro:property name="foot_l_mesh" value="0.267"/>
   <xacro:property name="scale" value="${0.05}"/>
-  <!--link
-	name="base_footprint"/-->
   <link
-    name="base_link">
+	name="world"/>
+  <link
+	name="chaser/base_footprint"/>
+  <link
+    name="chaser/base_link">
     <inertial>
       <origin
@@ -34,5 +33,5 @@
       <origin
         xyz="0 0 0"
-        rpy="${pi/2}  ${-pi} 0" /> <!--${pi/2}  ${-pi} 0-->
+        rpy="0 0 3.1415" /> <!--${pi/2}  ${-pi} 0-->
       <geometry>
         <mesh
@@ -41,16 +40,13 @@
     </visual>
   </link>
-<!-- POSE 3D GROUND TRUTH PLUGIN-->
-	<!--gazebo>
-	  <plugin name="ground_truth" filename="libgazebo_ros_p3d.so">
-		<frameName>map</frameName>
-		<bodyName>base_link</bodyName>
-		<topicName>/chaser/odom</topicName>
-		<updateRate>100</updateRate>
-	  </plugin>
-	</gazebo-->
-<!--joint name="base_joint" type="fixed">
-		<parent link="base_footprint"/>
-		<child link="base_link"/>
-</joint-->
+   <joint name="base_joint" type="fixed">
+		<origin xyz="0 0 0" rpy="0 0 0"/>
+		<parent link="chaser/base_footprint"/>
+		<child link="chaser/base_link"/>
+  </joint>
+  <joint name="base_footprint_joint" type="floating">
+		<origin xyz="0 0 0" rpy="0 0 0"/>
+		<parent link="world"/>
+		<child link="chaser/base_footprint"/>
+  </joint>
 </robot>

File: foot_control_xy/models/number1/urdf/number1.urdf.xacro (robot description, xacro)
@@ -1,6 +1,10 @@
 <?xml version="1.0"?>
 <robot xmlns:xacro="http://ros.org/wiki/xacro" name="number1">
+<link
+	name="world"/>
   <link
-    name="base_link">
+	name="target/base_footprint"/>
+  <link
+    name="target/base_link">
     <inertial>
       <origin
@@ -22,17 +26,26 @@
         rpy="0 0 0" />
       <geometry>
-        <box size="0.25"/>
+        <sphere radius="0.25"/>
       </geometry>
     </collision>
       <visual name="visual">
+		<origin
+		xyz="0 0 0"
+        rpy="0 0 -1.5707963267" />
         <geometry>
           <mesh
             filename="package://foot_control_xy/models/number1/meshes/number.dae"/>
         </geometry>
-        <!--material>
-          <script
-            filename="package://foot_control_xy/models/number1/materials/scripts"/>
-        </material-->
       </visual>
   </link>
+  <joint name="base_joint" type="fixed">
+		<origin xyz="0 0 0" rpy="0 0 0"/>
+		<parent link="target/base_footprint"/>
+		<child link="target/base_link"/>
+  </joint>
+  <joint name="base_footprint_joint" type="floating">
+		<origin xyz="0 0 0" rpy="0 0 0"/>
+		<parent link="world"/>
+		<child link="target/base_footprint"/>
+  </joint>
 </robot>

Commit message: replace world_chaser_tf to world_actor_tf for both chaser/target

File: foot_control_xy/models/h_lower_limb/urdf/h_lower_limb.urdf.xacro (robot description, xacro)
@@ -4,6 +4,4 @@
   <link
 	name="world"/>
-  <link
-	name="chaser/base_footprint"/>
   <link
     name="chaser/base_link">
@@ -40,13 +38,8 @@
     </visual>
   </link>
-   <joint name="base_joint" type="fixed">
+   <joint name="base_joint" type="floating">
 		<origin xyz="0 0 0" rpy="0 0 0"/>
-		<parent link="chaser/base_footprint"/>
+		<parent link="world"/>
 		<child link="chaser/base_link"/>
   </joint>
-  <joint name="base_footprint_joint" type="floating">
-		<origin xyz="0 0 0" rpy="0 0 0"/>
-		<parent link="world"/>
-		<child link="chaser/base_footprint"/>
-  </joint>
 </robot>

File: foot_control_xy/models/number1/urdf/number1.urdf.xacro (robot description, xacro)
@@ -3,6 +3,6 @@
 <link
 	name="world"/>
-  <link
-	name="target/base_footprint"/>
+  <!--link
+	name="target/base_footprint"/-->
   <link
     name="target/base_link">
@@ -39,13 +39,13 @@
       </visual>
   </link>
-  <joint name="base_joint" type="fixed">
+  <joint name="base_joint" type="floating">
 		<origin xyz="0 0 0" rpy="0 0 0"/>
-		<parent link="target/base_footprint"/>
+		<parent link="world"/>
 		<child link="target/base_link"/>
   </joint>
-  <joint name="base_footprint_joint" type="floating">
+  <!--joint name="base_footprint_joint" type="floating">
 		<origin xyz="0 0 0" rpy="0 0 0"/>
 		<parent link="world"/>
 		<child link="target/base_footprint"/>
-  </joint>
+  </joint-->
 </robot>

Commit message: change topic name to /chaser/pose or /target/pose - add gazebo plugin

File: foot_control_xy/models/h_lower_limb/urdf/h_lower_limb.urdf.xacro (robot description, xacro)
@@ -2,6 +2,4 @@
 <robot xmlns:xacro="http://ros.org/wiki/xacro" name="h_lower_limb">
   <xacro:property name="scale" value="${0.05}"/>
-  <link
-	name="world"/>
   <link
     name="chaser/base_link">
@@ -11,5 +9,5 @@
         rpy="0 0 0" />
       <mass
-        value="1" /> <!-- Look for real measurement -->
+        value="1" />
       <inertia
         ixx="1"
@@ -38,8 +36,8 @@
     </visual>
   </link>
-   <joint name="base_joint" type="floating">
-		<origin xyz="0 0 0" rpy="0 0 0"/>
-		<parent link="world"/>
-		<child link="chaser/base_link"/>
-  </joint>
+  <gazebo>
+   <plugin name="gzTfUpdate" filename="libgzTfUpdate.so">
+		<actorName>chaser</actorName>
+   </plugin>
+  </gazebo>
 </robot>

File: foot_control_xy/models/number1/urdf/number1.urdf.xacro (robot description, xacro)
@@ -1,8 +1,4 @@
 <?xml version="1.0"?>
 <robot xmlns:xacro="http://ros.org/wiki/xacro" name="number1">
-<link
-	name="world"/>
-  <!--link
-	name="target/base_footprint"/-->
   <link
     name="target/base_link">
@@ -12,5 +8,5 @@
         rpy="0 0 0" />
       <mass
-        value="1" /> <!-- Look for real measurement -->
+        value="1" />
       <inertia
         ixx="1"
@@ -39,13 +35,8 @@
       </visual>
   </link>
-  <joint name="base_joint" type="floating">
-		<origin xyz="0 0 0" rpy="0 0 0"/>
-		<parent link="world"/>
-		<child link="target/base_link"/>
-  </joint>
-  <!--joint name="base_footprint_joint" type="floating">
-		<origin xyz="0 0 0" rpy="0 0 0"/>
-		<parent link="world"/>
-		<child link="target/base_footprint"/>
-  </joint-->
+   <gazebo>
+   <plugin name="gzTfUpdate" filename="libgzTfUpdate.so">
+		<actorName>target</actorName>
+   </plugin>
+  </gazebo>
 </robot>

Commit message: change color plane

File: foot_control_xy/models/h_lower_limb/urdf/h_lower_limb.urdf.xacro (robot description, xacro)
@@ -2,6 +2,7 @@
 <robot xmlns:xacro="http://ros.org/wiki/xacro" name="h_lower_limb">
 	  <xacro:arg name="_scale" default="0.5"/>
-	  <xacro:arg name="_enableWorldTf" default="false"/>
+	  <xacro:arg name="_enableGzPlugin" default="false"/>
 	  <xacro:property name="_radius" value="${0.25* $(arg _scale)}"/>
+    <xacro:property name="_offset" value="${_radius*2.5}"/>
   <link
     name="chaser/base_link">
@@ -22,13 +23,17 @@
     <collision>
       <origin
-        xyz="0 0 0.25"
-        rpy="0 0 0" />
+        xyz="0 0 ${_offset}"
+        rpy="0 0 3.1415" />
+      <!-- <geometry>
+        <sphere radius="${_radius}"/>
+      </geometry> -->
       <geometry>
-        <sphere radius="${_radius}"/>
+        <mesh
+          filename="package://foot_control_xy/models/h_lower_limb/meshes/foot.dae" scale="${0.05*$(arg _scale)} ${0.05*$(arg _scale)} ${0.05*$(arg _scale)}"/>
       </geometry>
     </collision>
     <visual>
       <origin
-        xyz="0 0 ${2*_radius}"
+        xyz="0 0 ${_offset}"
         rpy="0 0 3.1415"/>
       <geometry>
@@ -38,5 +43,5 @@
     </visual>
   </link>
-    <xacro:if value="$(arg _enableWorldTf)">
+    <xacro:if value="$(arg _enableGzPlugin)">
 	  <gazebo>
 	   <plugin name="gzTfUpdate" filename="libgzTfUpdate.so">

File: foot_control_xy/models/number1/urdf/number1.urdf.xacro (robot description, xacro)
@@ -1,7 +1,7 @@
 <?xml version="1.0"?>
 <robot xmlns:xacro="http://ros.org/wiki/xacro" name="number1">
-	<xacro:arg name="_enableWorldTf" default="false"/>
-    <xacro:arg name="_scale" default="0.5"/>
-    <xacro:property name="_radius" value="${0.25* $(arg _scale)}"/>
+	<xacro:arg name="_enableGzPlugin" default="true"/>
+    <xacro:arg name="_scale" default="0.15"/>
+    <xacro:property name="_radius" value="${0.25*$(arg _scale)}"/>
   <link
     name="target/base_link">
@@ -25,5 +25,5 @@
         rpy="0 0 0" />
       <geometry>
-        <box size="${_radius}"/>
+        <box size="${_radius} ${_radius} ${_radius}"/>
       </geometry>
     </collision>
@@ -38,5 +38,5 @@
       </visual>
   </link>
-    <xacro:if value="$(arg _enableWorldTf)">
+    <xacro:if value="$(arg _enableGzPlugin)">
 	   <gazebo>
 	   <plugin name="gzTfUpdate" filename="libgzTfUpdate.so">

Commit message: add scaling factors to launch files scale.t and scale.c, modifications in xacro urdf

File: foot_control_xy/models/h_lower_limb/urdf/h_lower_limb.urdf.xacro (robot description, xacro)
@@ -1,8 +1,8 @@
 <?xml version="1.0"?>
 <robot xmlns:xacro="http://ros.org/wiki/xacro" name="h_lower_limb">
-	  <xacro:arg name="_scale" default="0.5"/>
-	  <xacro:arg name="_enableGzPlugin" default="false"/>
-	  <xacro:property name="_radius" value="${0.25* $(arg _scale)}"/>
-    <xacro:property name="_offset" value="${_radius*2.5}"/>
+	  <xacro:arg name="scale" default="0.5"/>
+	  <xacro:arg name="enableGzPlugin" default="false"/>
+	  <xacro:property name="radius" value="${0.25*$(arg scale)}"/>
+    <xacro:property name="offset" value="${radius*2.5}"/>
   <link
     name="chaser/base_link">
@@ -23,25 +23,22 @@
     <collision>
       <origin
-        xyz="0 0 ${_offset}"
-        rpy="0 0 3.1415" />
-      <!-- <geometry>
-        <sphere radius="${_radius}"/>
-      </geometry> -->
+        xyz="0 0 ${offset}"
+        rpy="0 0 3.1415"/>
       <geometry>
         <mesh
-          filename="package://foot_control_xy/models/h_lower_limb/meshes/foot.dae" scale="${0.05*$(arg _scale)} ${0.05*$(arg _scale)} ${0.05*$(arg _scale)}"/>
+          filename="package://foot_control_xy/models/h_lower_limb/meshes/foot.dae" scale="${0.05*$(arg scale)} ${0.05*$(arg scale)} ${0.05*$(arg scale)}"/>
       </geometry>
     </collision>
     <visual>
       <origin
-        xyz="0 0 ${_offset}"
+        xyz="0 0 ${offset}"
         rpy="0 0 3.1415"/>
       <geometry>
         <mesh
-          filename="package://foot_control_xy/models/h_lower_limb/meshes/foot.dae" scale="${0.05*$(arg _scale)} ${0.05*$(arg _scale)} ${0.05*$(arg _scale)}"/>
+          filename="package://foot_control_xy/models/h_lower_limb/meshes/foot.dae" scale="${0.05*$(arg scale)} ${0.05*$(arg scale)} ${0.05*$(arg scale)}"/>
       </geometry>
     </visual>
   </link>
-    <xacro:if value="$(arg _enableGzPlugin)">
+    <xacro:if value="$(arg enableGzPlugin)">
 	  <gazebo>
 	   <plugin name="gzTfUpdate" filename="libgzTfUpdate.so">

File: foot_control_xy/models/number1/urdf/number1.urdf.xacro (robot description, xacro)
@@ -1,7 +1,7 @@
 <?xml version="1.0"?>
 <robot xmlns:xacro="http://ros.org/wiki/xacro" name="number1">
-	<xacro:arg name="_enableGzPlugin" default="true"/>
-    <xacro:arg name="_scale" default="0.15"/>
-    <xacro:property name="_radius" value="${0.25*$(arg _scale)}"/>
+	<xacro:arg name="enableGzPlugin" default="true"/>
+  <xacro:arg name="scale" default="0.15"/>
+  <xacro:property name="radius" value="${0.25*$(arg scale)}"/>
   <link
     name="target/base_link">
@@ -20,5 +20,5 @@
         izz="1" />
     </inertial>
-    <collision>
+    <!--collision>
       <origin
         xyz="0 0 ${2*_radius}"
@@ -27,16 +27,16 @@
         <box size="${_radius} ${_radius} ${_radius}"/>
       </geometry>
-    </collision>
+    </collision-->
       <visual name="visual">
 		<origin
-		xyz="0 0 ${2*_radius}"
+		xyz="0 0 ${2*radius}"
         rpy="0 0 -1.5707963267" />
         <geometry>
           <mesh
-            filename="package://foot_control_xy/models/number1/meshes/number.dae" scale="$(arg _scale) $(arg _scale) $(arg _scale)"/>
+            filename="package://foot_control_xy/models/number1/meshes/number.dae" scale="$(arg scale) $(arg scale) $(arg scale)"/>
         </geometry>
       </visual>
   </link>
-    <xacro:if value="$(arg _enableGzPlugin)">
+    <xacro:if value="$(arg enableGzPlugin)">
 	   <gazebo>
 	   <plugin name="gzTfUpdate" filename="libgzTfUpdate.so">
