Commit message: [surgical_simulator][RobotsTaskGeneration]: Update trocar frame during the task + add transformation for left robot

File: surgical_simulator/models/kuka_lwr_on_table_with_tool.urdf.xacro (robot description, xacro)
@@ -4,4 +4,7 @@
   <xacro:arg name="origin.y" default="0"/>
   <xacro:arg name="origin.z" default="0"/>
+  <xacro:arg name="origin.ax" default="0"/>
+  <xacro:arg name="origin.ay" default="0"/>
+  <xacro:arg name="origin.az" default="0"/>
   <xacro:arg name="robotName" default="lwr"/>
   <xacro:arg name="addCamera" default="0"/>
@@ -31,5 +34,5 @@
   <xacro:kuka_lwr base_link="$(arg robotName)_table_plate_link" name="$(arg robotName)">
     <!-- <origin xyz="$(arg origin.x) $(arg origin.y) $(arg origin.z)" rpy="0 0 0"/> -->
-    <origin xyz="${tableLength/2} ${-tableWidth/2} 0" rpy="0 0 0"/>
+    <origin xyz="${tableLength/2} ${-tableWidth/2} 0" rpy="$(arg origin.ax) $(arg origin.ay) $(arg origin.az)"/>
   </xacro:kuka_lwr>
   <link name='$(arg robotName)_tool'>

File: surgical_simulator/models/surgical_environment.urdf.xacro (robot description, xacro)
@@ -28,5 +28,5 @@
                     height="${tableHeight}"
                     plate_thickness="0.1">
-    <origin xyz="${$(arg origin.x)-tableLength/2+xOffset} ${$(arg origin.y)+tableWidth/2} ${tableHeight}" rpy="0 0 0"/>
+    <origin xyz="${$(arg origin.x)-tableLength/2} ${$(arg origin.y)+tableWidth/2} ${tableHeight}" rpy="0 0 0"/>
   </xacro:model_table>
   <xacro:include filename="$(find surgical_simulator)/models/torso_upper.urdf.xacro"/>

Commit message: [surgical_simulator][robots_task_generation]: Fix camera orientation + move with respect to camera frame + add self rotation (thanks jacob)

File: surgical_simulator/models/kuka_lwr_on_table_with_tool.urdf.xacro (robot description, xacro)
@@ -71,5 +71,5 @@
         <parent link="$(arg robotName)_tool"/>
         <child link="$(arg robotName)_camera_link"/>
-        <origin xyz="0 0 ${toolLength}" rpy="0 ${-M_PI/2} 0"/>
+        <origin xyz="0 0 ${toolLength}" rpy="0 ${-M_PI/2} ${M_PI}"/>
   </joint>
   <gazebo reference='$(arg robotName)_camera_link'>

Commit message: [hasler_project][surgical_simulator]: push last changes

File: surgical_simulator/models/kuka_lwr_on_table_with_tool.urdf.xacro (robot description, xacro)
@@ -8,4 +8,5 @@
   <xacro:arg name="origin.az" default="0"/>
   <xacro:arg name="robotName" default="lwr"/>
+  <xacro:arg name="addFrame" default="0"/>
   <xacro:arg name="addCamera" default="0"/>
   <xacro:property name="toolMass" value="0.1"/>
@@ -60,4 +61,19 @@
     <child link="$(arg robotName)_tool"/>
   </joint>
+<xacro:if value="${$(arg addFrame)==1}">
+  <link name='$(arg robotName)_tipframe'>
+      <visual name='visual'>
+        <origin xyz="0 0 ${toolLength}" rpy="0 0 0" />
+          <geometry>
+           <mesh filename="package://surgical_simulator/models/frame.dae" scale="0.035 0.035 0.035"/>
+         </geometry>
+       </visual>
+  </link>
+  <joint name="$(arg robotName)_frame_joint" type="fixed">
+      <origin xyz="0 0 0" rpy="0 0 0"/>
+      <parent link="$(arg robotName)_tool"/>
+      <child link="$(arg robotName)_tipframe"/>
+  </joint>
+ </xacro:if>
 <xacro:if value="${$(arg addCamera)==1}">
   <link name="$(arg robotName)_camera_link">
@@ -77,5 +93,5 @@
       <alwaysOn>true</alwaysOn>
       <update_rate>30.0</update_rate>
-      <camera>
+    <camera>
         <pose>0 0 0 0 0 0</pose>
         <horizontal_fov>${85 * M_PI/180.0}</horizontal_fov>

File: surgical_simulator/models/surgical_environment.urdf.xacro (robot description, xacro)
@@ -37,5 +37,5 @@
                     zDim="${torsoZDim}"
                     scale="${torsoScale}">
-    <origin xyz="${tableLength/2} ${-0.6*tableWidth} ${torsoScale*0.4*torsoYDim}" rpy="0 0 0"/>
+    <origin xyz="${tableLength/2} ${-tableWidth/2} ${torsoScale*0.4*torsoYDim}" rpy="0 0 0"/>
   </xacro:torso_upper>
 </robot>
