Commit message: [demo_scientastic]: Update changes

File: demo_scientastic/models/h_lower_limb/urdf/foot_l.urdf.xacro (robot description, xacro)
@@ -17,4 +17,7 @@
         <box size="1 1 1"/>
       </geometry>
+<!--       <geometry>
+        <mesh filename="package://foot_control_xy/models/h_lower_limb/meshes/foot.dae" scale="${0.05*$(arg scale)} ${0.05*$(arg scale)} ${0.05*$(arg scale)}"/>
+      </geometry> -->
     </collision>
     <visual>
@@ -42,4 +45,7 @@
         <box size="0.1 1 1"/>
       </geometry>
+      <material name="white">
+        <color rgba="1.0 1.0 1.0 1.0"/>
+      </material>
     </visual>
   </link>
@@ -54,18 +60,20 @@
      <plugin name="footTfUpdate" filename="libfootTfUpdate.so">
         <actorName>$(arg link_name)</actorName>
-        <jointStiffness>1000</jointStiffness>
-        <jointDamping>10</jointDamping>
+        <jointStiffness>1500</jointStiffness>
+        <jointDamping>5</jointDamping>
      </plugin>
     </gazebo>
   </xacro:if>
 <!--   <gazebo reference="$(arg link_name)/sensor_joint">
-  <provideFeedback>true</provideFeedback>
-</gazebo>
+    <provideFeedback>true</provideFeedback>
+    <disableFixedJointLumping>true</disableFixedJointLumping>
+  </gazebo>
   <gazebo>
     <plugin name="ft_sensor" filename="libgazebo_ros_ft_sensor.so">
       <alwaysOn>true</alwaysOn>
-      <updateRate>30.0</updateRate>
-      <topicName>$(arg link_name)/ft_sensor</topicName>
+      <updateRate>200</updateRate>
+      <topicName>ft_sensor</topicName>
       <jointName>$(arg link_name)/sensor_joint</jointName>
+      <gaussianNoise>0.0001</gaussianNoise>
     </plugin>
   </gazebo> -->

File: demo_scientastic/models/h_lower_limb/urdf/h_lower_limb.urdf.xacro (robot description, xacro)
@@ -44,4 +44,7 @@
         <box size="0.1 1 1"/>
       </geometry>
+      <material name="white">
+        <color rgba="1.0 1.0 1.0 1.0"/>
+      </material>
     </visual>
   </link>
@@ -57,18 +60,20 @@
       <plugin name="footTfUpdate" filename="libfootTfUpdate.so">
 	      <actorName>$(arg link_name)</actorName>
-        <jointStiffness>1000</jointStiffness>
-        <jointDamping>10</jointDamping>
+        <jointStiffness>1500</jointStiffness>
+        <jointDamping>5</jointDamping>
       </plugin>
     </gazebo>
   </xacro:if>
 <!--   <gazebo reference="$(arg link_name)/sensor_joint">
-  <provideFeedback>true</provideFeedback>
-</gazebo>
+    <provideFeedback>true</provideFeedback>
+    <disableFixedJointLumping>true</disableFixedJointLumping>
+  </gazebo>
   <gazebo>
     <plugin name="ft_sensor" filename="libgazebo_ros_ft_sensor.so">
       <alwaysOn>true</alwaysOn>
-      <updateRate>30.0</updateRate>
-      <topicName>$(arg link_name)/ft_sensor</topicName>
+      <updateRate>200</updateRate>
+      <topicName>ft_sensor</topicName>
       <jointName>$(arg link_name)/sensor_joint</jointName>
+      <gaussianNoise>0.0001</gaussianNoise>
     </plugin>
   </gazebo> -->

File: foot_control_xy/models/h_lower_limb/urdf/h_lower_limb.urdf.xacro (robot description, xacro)
@@ -21,5 +21,4 @@
         izz="1" />
     </inertial>
-<!--
     <collision>
       <origin
@@ -31,5 +30,4 @@
       </geometry>
     </collision>
--->
     <visual>
       <origin

File: surgical_simulator/models/table.urdf.xacro (robot description, xacro)
@@ -15,5 +15,17 @@
     <inertia ixx="${table_mass * 10 * mm2_to_m2}" ixy="0.0" ixz="0.0" iyy="${table_mass * 10 * mm2_to_m2}" iyz="0.0" izz="${table_mass * 10 * mm2_to_m2}"/>
 </xacro:property>
-<xacro:macro name="table_leg" params="parent name *origin">
+<material name="green">
+    <color rgba="0.0 1.0 0.0 1.0"/>
+</material>
+<material name="red">
+    <color rgba="1.0 0.0 0.0 1.0"/>
+</material>
+<material name="blue">
+    <color rgba="0.0 0.0 1.0 1.0"/>
+</material>
+<material name="grey">
+    <color rgba="0.5 0.5 0.5 1.0"/>
+</material>
+<xacro:macro name="table_leg" params="parent name *origin color">
     <joint name="${name}_joint" type="fixed">
         <xacro:insert_block name="origin"/>
@@ -29,5 +41,5 @@
 				<box size="${leg_width/2} -${leg_width} ${height - plate_thickness}"/>
 			</geometry>
-			<material name="Vito/Black"/>
+			<material name="${color}"/>
 		</visual>
 		<collision>
@@ -41,5 +53,5 @@
     </gazebo>
 </xacro:macro>
-<xacro:macro name="model_table" params="parent name *origin length width height plate_thickness">
+<xacro:macro name="model_table" params="parent name *origin length width height plate_thickness color">
     <joint name="${parent}_${name}_base_joint" type="fixed">
         <xacro:insert_block name="origin"/>
@@ -56,5 +68,8 @@
                 <box size="${length} ${width} ${plate_thickness}"/>
 			</geometry>
-			<material name="Vito/LightGrey"/>
+			<!-- <material name="Vito/LightGrey"/> -->
+            <material name="${color}">
+                <!-- <color rgba="0.0 1.0 0.0 1.0"/> -->
+            </material>
 		</visual>
         <collision>
@@ -65,14 +80,14 @@
         </collision>
     </link>
-    <xacro:table_leg parent="${name}_plate_link" name="${name}_leg_0">
+    <xacro:table_leg parent="${name}_plate_link" name="${name}_leg_0" color="${color}">
         <origin xyz="${border_offset} -${border_offset} -${1/2 * (plate_thickness + height)}"/>
     </xacro:table_leg>
-    <xacro:table_leg parent="${name}_plate_link" name="${name}_leg_1">
+    <xacro:table_leg parent="${name}_plate_link" name="${name}_leg_1" color="${color}">
         <origin xyz="${length - border_offset} -${border_offset} -${1/2 * (plate_thickness + height)}"/>
     </xacro:table_leg>
-    <xacro:table_leg parent="${name}_plate_link" name="${name}_leg_2">
+    <xacro:table_leg parent="${name}_plate_link" name="${name}_leg_2" color="${color}">
         <origin xyz="${border_offset} -${width - border_offset} -${1/2 * (plate_thickness + height)}"/>
     </xacro:table_leg>
-    <xacro:table_leg parent="${name}_plate_link" name="${name}_leg_3">
+    <xacro:table_leg parent="${name}_plate_link" name="${name}_leg_3" color="${color}">
         <origin xyz="${length - border_offset} -${width - border_offset} -${1/2 * (plate_thickness + height)}"/>
     </xacro:table_leg>
