Commit message: Update trocar feet telemanipulation with spherical trocars

File: robotic_experiments/models/lwr_with_tool.urdf.xacro (robot description, xacro)
@@ -11,5 +11,5 @@
   <xacro:arg name="addCamera" default="0"/>
   <xacro:property name="toolMass" value="0.1"/>
-  <xacro:property name="toolLength" value="0.40"/>
+  <xacro:property name="toolLength" value="0.533"/>
   <xacro:property name="toolRadius" value="0.005"/>
   <link name="world"/>

Commit message: [robotic_experiments][TrocarFeetTelemanipulation]: Add second robot

File: robotic_experiments/models/lwr_with_tool.urdf.xacro (robot description, xacro)
@@ -11,5 +11,5 @@
   <xacro:arg name="addCamera" default="0"/>
   <xacro:property name="toolMass" value="0.1"/>
-  <xacro:property name="toolLength" value="0.533"/>
+  <xacro:property name="toolLength" value="0.433"/>
   <xacro:property name="toolRadius" value="0.005"/>
   <link name="world"/>
@@ -22,6 +22,5 @@
   <!-- <xacro:include filename="$(find kuka_lwr_bringup)/models/table/table.urdf.xacro"/> -->
   <xacro:kuka_lwr base_link="world" name="$(arg robotName)">
-    <!-- <origin xyz="$(arg origin.x) $(arg origin.y) $(arg origin.z)" rpy="0 0 0"/> -->
-    <origin xyz="0 0 0" rpy="0 0 0"/>
+    <origin xyz="$(arg origin.x) $(arg origin.y) $(arg origin.z)" rpy="0 0 0"/>
   </xacro:kuka_lwr>
   <link name='$(arg robotName)_tool'>
@@ -64,5 +63,5 @@
   </joint>
  </xacro:if>
-<!-- <xacro:if value="${$(arg addCamera)==1}">
+<xacro:if value="${$(arg addCamera)==1}">
   <link name="$(arg robotName)_camera_link">
     <inertial>
@@ -72,11 +71,9 @@
     </inertial>
   </link>
- -->
-<!--   <joint name="$(arg robotName)_camera_joint" type="fixed">
+  <joint name="$(arg robotName)_camera_joint" type="fixed">
         <parent link="$(arg robotName)_tool"/>
         <child link="$(arg robotName)_camera_link"/>
         <origin xyz="0 0 ${toolLength}" rpy="0 ${-M_PI/2} ${M_PI}"/>
-  </joint> -->
-<!--
+  </joint>
   <gazebo reference='$(arg robotName)_camera_link'>
     <sensor type="camera" name="camera_camera_sensor">
@@ -111,6 +108,6 @@
       </plugin>
     </sensor>
-  </gazebo> -->
-<!-- </xacro:if> -->
+  </gazebo>
+</xacro:if>
 <!-- <xacro:if value="${$(arg addCamera)==0}"> -->
 <!--   <link name="ft_sensor_link">

Commit message: Push changes from last year (new shared four arm manipulation + surgical experiment)

File: robotic_experiments/models/lwr_with_tool.urdf.xacro (robot description, xacro)
@@ -11,5 +11,5 @@
   <xacro:arg name="addCamera" default="0"/>
   <xacro:property name="toolMass" value="0.1"/>
-  <xacro:property name="toolLength" value="0.433"/>
+  <xacro:property name="toolLength" value="0.13"/>
   <xacro:property name="toolRadius" value="0.005"/>
   <link name="world"/>
