Commit message: backup 13.7.2020

File: leg_as_robot/urdf/leg.joints.xacro (robot description, xacro)
@@ -35,5 +35,5 @@
       <parent link="hip_adduction_link"/>
       <child link="hip_extension_link"/>
-      <limit effort="30" velocity="10.0" lower="${radians(-5)}" upper="${radians(32)}"/>
+      <limit effort="30" velocity="10.0" lower="${radians(-30)}" upper="${radians(32)}"/>
       <axis xyz="0 0 1"/>
     </joint>

File: leg_as_robot/urdf/leg.links.xacro (robot description, xacro)
@@ -1,5 +1,5 @@
 <?xml version="1.0"?>
 <robot xmlns:xacro="http://www.ros.org/wiki/xacro">
-  <xacro:property name="body_weight" value="83"/>  <!-- [kg] -->
+  <xacro:property name="body_weight" value="${83}"/>  <!-- [kg] -->
   <xacro:property name="thigh_mass" value="${14.47 * body_weight / 100}"/> <!-- [kg] -->
   <xacro:property name="shin_mass" value="${4.57 * body_weight / 100}"/> <!-- [kg] -->

Commit message: much better with the newton raphson method with joint limits

File: leg_as_robot/urdf/leg.joints.xacro (robot description, xacro)
@@ -1,20 +1,11 @@
 <?xml version="1.0"?>
 <robot xmlns:xacro="http://www.ros.org/wiki/xacro">
-  <xacro:property name="leg_geom_data_yaml" value="$(find leg_as_robot)/config/leg_geom_data.yaml"/>
-  <xacro:property name="platform_geom_data_yaml" value="$(find foot_platform_ros)/config/right_platform_geom_data.yaml"/>
-  <xacro:property name="leg_geom_data" value="${load_yaml(leg_geom_data_yaml)}"/>
-  <xacro:property name="platform_geom_data" value="${load_yaml(platform_geom_data_yaml)}"/>
-  <xacro:property name="d3_leg" value="${leg_geom_data['thigh_length']}"/> <!-- d3_leg [m]-->
-  <xacro:property name="r4_leg" value="${leg_geom_data['shin_length']}"/> <!-- r4_leg [m]-->
-  <xacro:property name="d7_leg" value="${leg_geom_data['ankle_to_foot_base_z']}"/> <!-- d7_leg [m]-->
-  <xacro:property name="r7_leg" value="${leg_geom_data['ankle_to_foot_base_x']}"/> <!-- r7_leg [m]-->
-  <xacro:property name="r8_leg" value="${leg_geom_data['foot_base_to_foot_tip']}"/> <!-- r8_leg_foot_tip [m]-->
-  <xacro:property name="r3_platform" value="${platform_geom_data['r3']}"/> <!-- [m]-->
-  <xacro:property name="d6_platform" value="${platform_geom_data['d6']}"/> <!-- [m]-->
-  <xacro:property name="d7_platform" value="${platform_geom_data['d7']}"/> <!-- [m]-->
-  <xacro:property name="r8_platform" value="${platform_geom_data['r8']}"/> <!-- [m]-->
-  <xacro:property name="r8_leg_extra" value="${r8_platform-r8_leg}"/> <!-- [m]-->
-  <xacro:property name="base_to_hip_offset">
-    <origin xyz="0 ${- r7_leg - d3_leg} ${r3_platform + d6_platform + d7_platform +  d7_leg + r4_leg}" rpy="0 0 0"/> <!-- <origin xyz="0 -0.5100 0.9246" rpy="0 0 0"/> -->
+  <xacro:property name="base_to_hip_offset_x" value="0"/>
+  <xacro:property name="base_to_hip_offset_y" value="${- r7_leg - d3_leg}"/>
+  <xacro:property name="base_to_hip_offset_z" value="${r3_platform + d6_platform + d7_platform +  d7_leg + r4_leg}"/>
+  <xacro:property name="base_to_hip_offset_baseline_y" value="${- r7Baseline_leg - d3Baseline_leg}"/>
+  <xacro:property name="base_to_hip_offset_baseline_z" value="${r3_platform + d6_platform + d7_platform +  d7Baseline_leg + r4Baseline_leg}"/>
+   <xacro:property name="base_to_hip_offset">
+      <origin xyz="${base_to_hip_offset_x} ${base_to_hip_offset_y} ${base_to_hip_offset_z}" rpy="0 0 0"/> <!-- <origin xyz="0 -0.5100 0.9246" rpy="0 0 0"/> -->
   </xacro:property>
   <xacro:macro name="define_leg_joints">

File: leg_as_robot/urdf/leg.links.xacro (robot description, xacro)
@@ -1,8 +1,20 @@
 <?xml version="1.0"?>
 <robot xmlns:xacro="http://www.ros.org/wiki/xacro">
-  <xacro:property name="body_weight" value="${83}"/>  <!-- [kg] -->
   <xacro:property name="thigh_mass" value="${14.47 * body_weight / 100}"/> <!-- [kg] -->
   <xacro:property name="shin_mass" value="${4.57 * body_weight / 100}"/> <!-- [kg] -->
   <xacro:property name="foot_mass" value="${1.33 * body_weight / 100}"/> <!--[kg] -->
+  <xacro:property name="scale_mass" value="${body_weight / body_weight_baseline}"/>
+  <xacro:property name="base_scale_x" value="${1.0}"/>
+  <xacro:property name="base_scale_y" value="${base_to_hip_offset_y/base_to_hip_offset_baseline_y}"/>
+  <xacro:property name="base_scale_z" value="${base_to_hip_offset_z/base_to_hip_offset_baseline_z}"/>
+  <xacro:property name="thigh_scale_x" value="${1.0}"/>
+  <xacro:property name="thigh_scale_y" value="${1.0}"/>
+  <xacro:property name="thigh_scale_z" value="${d3_leg / d3Baseline_leg}"/>
+  <xacro:property name="shin_scale_x" value="${r4_leg / r4Baseline_leg}"/>
+  <xacro:property name="shin_scale_y" value="${1.0}"/>
+  <xacro:property name="shin_scale_z" value="${1.0}"/>
+  <xacro:property name="foot_scale_x" value="${1.0}"/>
+  <xacro:property name="foot_scale_y" value="${r7_leg / r7Baseline_leg}"/>
+  <xacro:property name="foot_scale_z" value="${d7_leg / d7Baseline_leg}"/>
   <xacro:macro name="define_leg_links">
     <link name="virtual_platform_base_link"/>
@@ -11,5 +23,5 @@
           <origin rpy="0 0 0" xyz="0 0 0"/>
           <geometry>
-            <mesh filename="package://leg_as_robot/model/meshes/dae/leg_base_visual.dae"/>
+            <mesh filename="package://leg_as_robot/model/meshes/dae/leg_base_visual.dae" scale ="${base_scale_x} ${base_scale_y} ${base_scale_z}"/>
           </geometry>
         </visual>
@@ -17,5 +29,5 @@
           <origin rpy="0 0 0" xyz="0 0 0"/>
           <geometry>
-            <mesh filename="package://leg_as_robot/model/meshes/stl/leg_base_collision.stl"/>
+            <mesh filename="package://leg_as_robot/model/meshes/stl/leg_base_collision.stl" scale ="${base_scale_x} ${base_scale_y} ${base_scale_z}"/>
           </geometry>
         </collision>
@@ -25,12 +37,12 @@
     <link name="hip_roll_link" >
       <inertial>
-      <origin xyz="0.00265863 -0.00827375 0.17215567" rpy="0 0 0"/>
+      <origin xyz="${0.00265863 * thigh_scale_x} ${-0.00827375 * thigh_scale_y } ${0.17215567 * thigh_scale_z}" rpy="0 0 0"/>
       <mass value="${thigh_mass}"/><!-- kg -->
-      <inertia ixx="0.25495934"  ixy="0.00092859"  ixz="-0.00803351" iyy="0.25972836" iyz="0.00151866" izz="0.05431793" />
+      <inertia ixx="${0.25495934 * scale_mass * thigh_scale_x * thigh_scale_x}"  ixy="${0.00092859 * scale_mass * thigh_scale_x * thigh_scale_y}"  ixz="${-0.00803351 * scale_mass * thigh_scale_x * thigh_scale_z}" iyy="${0.25972836 * scale_mass * thigh_scale_y * thigh_scale_y}" iyz="${0.00151866 * scale_mass * thigh_scale_y * thigh_scale_z}" izz="${0.05431793 * scale_mass * thigh_scale_z * thigh_scale_z}" />
     </inertial>
       <visual>
         <origin rpy="0 0 0" xyz="0 0 0"/>
         <geometry>
-          <mesh filename="package://leg_as_robot/model/meshes/dae/thigh_visual.dae"/>
+          <mesh filename="package://leg_as_robot/model/meshes/dae/thigh_visual.dae" scale ="${thigh_scale_x} ${thigh_scale_y } ${thigh_scale_z}"/>
         </geometry>
       </visual>
@@ -38,5 +50,5 @@
         <origin rpy="0 0 0" xyz="0 0 0"/>
         <geometry>
-          <mesh filename="package://leg_as_robot/model/meshes/stl/thigh_collision.stl"/>
+          <mesh filename="package://leg_as_robot/model/meshes/stl/thigh_collision.stl" scale ="${thigh_scale_x} ${thigh_scale_y} ${thigh_scale_z}"/>
         </geometry>
       </collision>
@@ -44,12 +56,12 @@
     <link name="knee_extension_link" >
       <inertial>
-          <origin xyz="0.14893265 0.01010783 -0.00938572" rpy="0 0 0"/>
+          <origin xyz="${0.14893265 * shin_scale_x} ${0.01010783 * shin_scale_y } ${-0.00938572 * shin_scale_z}" rpy="0 0 0"/>
           <mass value="${shin_mass}"/><!-- kg -->
-          <inertia ixx="0.00474593"  ixy="0.00116322"  ixz="0.00035670" iyy="0.04707968" iyz="0.00006150" izz="0.04724374" />
+          <inertia ixx="${0.00474593 * scale_mass * shin_scale_x * shin_scale_x}"  ixy="${0.00116322 * scale_mass * shin_scale_x * shin_scale_y}"  ixz="${0.00035670 * scale_mass * shin_scale_x * shin_scale_z}" iyy="${0.04707968 * scale_mass * shin_scale_y * shin_scale_y }" iyz="${0.00006150 * scale_mass * shin_scale_y * shin_scale_z }" izz="${0.04724374 * scale_mass * shin_scale_z * shin_scale_z }" />
       </inertial>
           <visual>
         <origin rpy="0 0 0" xyz="0 0 0"/>
         <geometry>
-          <mesh filename="package://leg_as_robot/model/meshes/dae/shin_visual.dae"/>
+          <mesh filename="package://leg_as_robot/model/meshes/dae/shin_visual.dae" scale ="${shin_scale_x } ${shin_scale_y} ${shin_scale_z}"/>
         </geometry>
       </visual>
@@ -57,5 +69,5 @@
         <origin rpy="0 0 0" xyz="0 0 0"/>
         <geometry>
-          <mesh filename="package://leg_as_robot/model/meshes/stl/shin_collision.stl"/>
+          <mesh filename="package://leg_as_robot/model/meshes/stl/shin_collision.stl" scale ="${shin_scale_x } ${shin_scale_y} ${shin_scale_z}"/>
         </geometry>
       </collision>
@@ -65,19 +77,19 @@
     <link name="ankle_yaw_link">
         <inertial>
-          <origin xyz="-0.00089807 -0.04499748 -0.04201224" rpy="0 0 0"/>
+          <origin xyz="${-0.00089807 * foot_scale_x} ${-0.04499748 * foot_scale_y} ${-0.04201224 * foot_scale_z}" rpy="0 0 0"/>
           <mass value="${foot_mass}"/><!-- kg -->
-          <inertia ixx="0.00322038"  ixy="-0.00005516"  ixz="0.00007652" iyy="0.00084882" iyz="0.00056936" izz="0.00297569" />
+          <inertia ixx="${0.00322038 * scale_mass * foot_scale_x * foot_scale_x}"  ixy="${-0.00005516 * scale_mass * foot_scale_x * foot_scale_y}"  ixz="${0.00007652 * scale_mass * foot_scale_x * foot_scale_z}" iyy="${0.00084882 * scale_mass * foot_scale_y * foot_scale_y }" iyz="${0.00056936 * scale_mass * foot_scale_y * foot_scale_z }" izz="${0.00297569 * scale_mass * foot_scale_z * foot_scale_z }" />
       </inertial>
           <visual>
         <origin rpy="0 0 0" xyz="0 0 0"/>
         <geometry>
-          <mesh filename="package://leg_as_robot/model/meshes/dae/foot_visual.dae"/>
-        </geometry>
+          <mesh filename="package://leg_as_robot/model/meshes/dae/foot_visual.dae" scale ="${foot_scale_x} ${foot_scale_y} ${foot_scale_z}"/>}
+${        </geometry>
       </visual>
       <collision>
         <origin rpy="0 0 0" xyz="0 0 0"/>
         <geometry>
-          <mesh filename="package://leg_as_robot/model/meshes/stl/foot_collision.stl"/>
-        </geometry>
+          <mesh filename="package://leg_as_robot/model/meshes/stl/foot_collision.stl" scale ="${foot_scale_x} ${foot_scale_y} ${foot_scale_z}"/>}
+${        </geometry>
       </collision>
     </link>

File: leg_as_robot/urdf/leg.urdf.xacro (robot description, xacro)
@@ -2,4 +2,5 @@
 <robot xmlns:xacro="http://www.ros.org/wiki/xacro" name="leg_as_robot">
  <xacro:macro name="create_leg">
+  <xacro:include filename="$(find leg_as_robot)/urdf/leg.yaml.xacro"/>
   <xacro:include filename="$(find leg_as_robot)/urdf/leg.links.xacro"/>
   <xacro:include filename="$(find leg_as_robot)/urdf/leg.joints.xacro"/>

Commit message: add scales foot

File: leg_as_robot/urdf/leg.joints.xacro (robot description, xacro)
@@ -3,5 +3,5 @@
   <xacro:property name="base_to_hip_offset_x" value="0"/>
   <xacro:property name="base_to_hip_offset_y" value="${- r7_leg - d3_leg}"/>
-  <xacro:property name="base_to_hip_offset_z" value="${r3_platform + d6_platform + d7_platform +  d7_leg + r4_leg}"/>
+  <xacro:property name="base_to_hip_offset_z" value="${r3_platform + d6_platform + d7_platform + d7_leg + r4_leg}"/>
   <xacro:property name="base_to_hip_offset_baseline_y" value="${- r7Baseline_leg - d3Baseline_leg}"/>
   <xacro:property name="base_to_hip_offset_baseline_z" value="${r3_platform + d6_platform + d7_platform +  d7Baseline_leg + r4Baseline_leg}"/>
@@ -37,5 +37,5 @@
     </joint>
     <joint name="knee_extension" type="revolute">
-      <origin xyz="0 0 ${d3_leg}" rpy="-${pi/2} 0 ${pi}"/>
+      <origin xyz="0 0 ${d3_leg}" rpy="${-pi/2} 0 ${pi}"/>
       <parent link="hip_roll_link"/>
       <child link="knee_extension_link"/>
@@ -58,5 +58,5 @@
     </joint>
     <joint name="ankle_yaw" type="revolute">
-      <origin xyz="0 0 0" rpy="-${pi/2} 0 -${pi/2}"/>
+      <origin xyz="0 0 0" rpy="${-pi/2} 0 ${-pi/2}"/>
       <parent link="ankle_roll_link"/>
       <child link="ankle_yaw_link"/>
@@ -65,5 +65,5 @@
     </joint>
       <joint name="fixed_foot_base" type="fixed">
-          <origin xyz="0 -${r7_leg} -${d7_leg}" rpy="0 0 -${pi/2}"/>
+          <origin xyz="0 ${-r7_leg} ${-d7_leg}" rpy="0 0 ${-pi/2}"/>
           <parent link="ankle_yaw_link"/>
           <child link="foot_base"/>

File: leg_as_robot/urdf/leg.links.xacro (robot description, xacro)
@@ -8,13 +8,13 @@
   <xacro:property name="base_scale_y" value="${base_to_hip_offset_y/base_to_hip_offset_baseline_y}"/>
   <xacro:property name="base_scale_z" value="${base_to_hip_offset_z/base_to_hip_offset_baseline_z}"/>
-  <xacro:property name="thigh_scale_x" value="${1.0}"/>
-  <xacro:property name="thigh_scale_y" value="${1.0}"/>
-  <xacro:property name="thigh_scale_z" value="${d3_leg / d3Baseline_leg}"/>
-  <xacro:property name="shin_scale_x" value="${r4_leg / r4Baseline_leg}"/>
-  <xacro:property name="shin_scale_y" value="${1.0}"/>
-  <xacro:property name="shin_scale_z" value="${1.0}"/>
-  <xacro:property name="foot_scale_x" value="${1.0}"/>
-  <xacro:property name="foot_scale_y" value="${r7_leg / r7Baseline_leg}"/>
-  <xacro:property name="foot_scale_z" value="${d7_leg / d7Baseline_leg}"/>
+  <xacro:property name="thigh_scale_x" value="${thigh_d/thighBaseline_d}"/>
+  <xacro:property name="thigh_scale_y" value="${thigh_w/thighBaseline_w}"/>
+  <xacro:property name="thigh_scale_z" value="${d3_leg/d3Baseline_leg}"/>
+  <xacro:property name="shin_scale_x" value="${r4_leg/r4Baseline_leg}"/>
+  <xacro:property name="shin_scale_y" value="${shin_d/shinBaseline_d}"/>
+  <xacro:property name="shin_scale_z" value="${shin_w/shinBaseline_w}"/>
+  <xacro:property name="foot_scale_x" value="${foot_l/footBaseline_l}"/>
+  <xacro:property name="foot_scale_y" value="${r7_leg/r7Baseline_leg}"/>
+  <xacro:property name="foot_scale_z" value="${d7_leg/d7Baseline_leg}"/>
   <xacro:macro name="define_leg_links">
     <link name="virtual_platform_base_link"/>
@@ -85,5 +85,5 @@
         <geometry>
           <mesh filename="package://leg_as_robot/model/meshes/dae/foot_visual.dae" scale ="${foot_scale_x} ${foot_scale_y} ${foot_scale_z}"/>}
-${        </geometry>
+        </geometry>
       </visual>
       <collision>
@@ -91,5 +91,5 @@
         <geometry>
           <mesh filename="package://leg_as_robot/model/meshes/stl/foot_collision.stl" scale ="${foot_scale_x} ${foot_scale_y} ${foot_scale_z}"/>}
-${        </geometry>
+        </geometry>
       </collision>
     </link>

File: leg_as_robot/urdf/leg.yaml.xacro (robot description, xacro)
@@ -12,11 +12,21 @@
     <xacro:property name="r7_leg" value="${leg_geom_data['ankle_to_foot_base_x']}"/> <!-- r7_leg [m]-->
     <xacro:property name="r8_leg" value="${leg_geom_data['foot_base_to_foot_tip']}"/> <!-- r8_leg_foot_tip [m]-->
+    <xacro:property name="thigh_w" value="${leg_geom_data['thigh_width']}"/>
+    <xacro:property name="thigh_d" value="${leg_geom_data['thigh_depth']}"/>
+    <xacro:property name="shin_w" value="${leg_geom_data['shin_width']}"/>
+    <xacro:property name="shin_d" value="${leg_geom_data['shin_depth']}"/>
+    <xacro:property name="foot_l" value="${leg_geom_data['foot_length']}"/>
     <xacro:property name="body_weight" value="${leg_geom_data['body_weight']}"/>
     <xacro:property name="body_weight_baseline" value="${leg_geom_data['body_weight']}"/>
-    <xacro:property name="d3Baseline_leg" value="${leg_geom_data_baseline['thigh_length']}"/> <!-- d3_leg [m]-->
-    <xacro:property name="r4Baseline_leg" value="${leg_geom_data_baseline['shin_length']}"/> <!-- r4_leg [m]-->
-    <xacro:property name="d7Baseline_leg" value="${leg_geom_data_baseline['ankle_to_foot_base_z']}"/> <!-- d7_leg [m]-->
-    <xacro:property name="r7Baseline_leg" value="${leg_geom_data_baseline['ankle_to_foot_base_x']}"/> <!-- r7_leg [m]-->
-    <xacro:property name="r8Baseline_leg" value="${leg_geom_data_baseline['foot_base_to_foot_tip']}"/> <!-- r8_leg_foot_tip [m]-->
+    <xacro:property name="d3Baseline_leg" value="${leg_geom_data_baseline['thigh_length']}"/>
+    <xacro:property name="r4Baseline_leg" value="${leg_geom_data_baseline['shin_length']}"/>
+    <xacro:property name="d7Baseline_leg" value="${leg_geom_data_baseline['ankle_to_foot_base_z']}"/>
+    <xacro:property name="r7Baseline_leg" value="${leg_geom_data_baseline['ankle_to_foot_base_x']}"/>
+    <xacro:property name="r8Baseline_leg" value="${leg_geom_data_baseline['foot_base_to_foot_tip']}"/>
+    <xacro:property name="thighBaseline_w" value="${leg_geom_data_baseline['thigh_width']}"/>
+    <xacro:property name="thighBaseline_d" value="${leg_geom_data_baseline['thigh_depth']}"/>
+    <xacro:property name="shinBaseline_w" value="${leg_geom_data_baseline['shin_width']}"/>
+    <xacro:property name="shinBaseline_d" value="${leg_geom_data_baseline['shin_depth']}"/>
+    <xacro:property name="footBaseline_l" value="${leg_geom_data_baseline['foot_length']}"/>
     <xacro:property name="r3_platform" value="${platform_geom_data['r3']}"/> <!-- [m]-->
     <xacro:property name="d6_platform" value="${platform_geom_data['d6']}"/> <!-- [m]-->

Commit message: add new nodes for force sensor biasing and gravity compensation

File: leg_as_robot/urdf/leg.joints.xacro (robot description, xacro)
@@ -1,5 +1,5 @@
 <?xml version="1.0"?>
 <robot xmlns:xacro="http://www.ros.org/wiki/xacro">
-  <xacro:property name="base_to_hip_offset_x" value="0"/>
+  <xacro:property name="base_to_hip_offset_x" value="${chair_x_offset}"/>
   <xacro:property name="base_to_hip_offset_y" value="${- r7_leg - d3_leg}"/>
   <xacro:property name="base_to_hip_offset_z" value="${r3_platform + d6_platform + d7_platform + d7_leg + r4_leg}"/>
@@ -19,5 +19,5 @@
       <parent link="hip_base_link"/>
       <child link="hip_adduction_link"/>
-      <limit effort="30" velocity="10.0" lower="${radians(-44)}" upper="${radians(0)}"/>
+      <limit effort="30" velocity="10.0" lower="${radians(-44)}" upper="${radians(10)}"/>
       <axis xyz="0 0 1"/>
     </joint>

File: leg_as_robot/urdf/leg.links.xacro (robot description, xacro)
@@ -1,7 +1,7 @@
 <?xml version="1.0"?>
 <robot xmlns:xacro="http://www.ros.org/wiki/xacro">
-  <xacro:property name="thigh_mass" value="${14.47 * body_weight / 100}"/> <!-- [kg] -->
-  <xacro:property name="shin_mass" value="${4.57 * body_weight / 100}"/> <!-- [kg] -->
-  <xacro:property name="foot_mass" value="${1.33 * body_weight / 100}"/> <!--[kg] -->
+  <xacro:property name="thigh_mass" value="${14.47 * 100.0/165.0 * body_weight / 100}"/> <!-- [kg] -->
+  <xacro:property name="shin_mass" value="${4.57 * 100.0/165.0 * body_weight / 100}"/> <!-- [kg] -->
+  <xacro:property name="foot_mass" value="${1.33 * 100.0/165.0 *body_weight / 100}"/> <!--[kg] -->
   <xacro:property name="scale_mass" value="${body_weight / body_weight_baseline}"/>
   <xacro:property name="base_scale_x" value="${1.0}"/>

File: leg_as_robot/urdf/leg.yaml.xacro (robot description, xacro)
@@ -17,4 +17,5 @@
     <xacro:property name="shin_d" value="${leg_geom_data['shin_depth']}"/>
     <xacro:property name="foot_l" value="${leg_geom_data['foot_length']}"/>
+    <xacro:property name="chair_x_offset" value="${leg_geom_data['offset_chair_x']}"/>
     <xacro:property name="body_weight" value="${leg_geom_data['body_weight']}"/>
     <xacro:property name="body_weight_baseline" value="${leg_geom_data['body_weight']}"/>
