Commit message: added manipulability ellipsoid

File: leg_as_robot/urdf/left/leg.create.xacro (robot description, xacro)
@@ -1,5 +1,5 @@
 <?xml version="1.0"?>
 <robot xmlns:xacro="http://www.ros.org/wiki/xacro" name="leg_as_robot">
-  <xacro:include filename="$(find leg_as_robot)/urdf/leg.urdf.xacro"/>
+  <xacro:include filename="$(find leg_as_robot)/urdf/left/leg.urdf.xacro"/>
   <xacro:create_leg/>
 </robot>

File: leg_as_robot/urdf/left/leg.yaml.xacro (robot description, xacro)
@@ -3,5 +3,5 @@
     <xacro:property name="leg_geom_data_yaml" value="$(find leg_as_robot)/config/leg_geom_data.yaml"/>
     <xacro:property name="leg_geom_data_baseline_yaml" value="$(find leg_as_robot)/config/leg_geom_data.baseline.yaml"/>
-    <xacro:property name="platform_geom_data_yaml" value="$(find foot_platform_ros)/config/right_platform_geom_data.yaml"/>
+    <xacro:property name="platform_geom_data_yaml" value="$(find foot_platform_ros)/config/platform_geom_data.yaml"/>
     <xacro:property name="leg_geom_data" value="${load_yaml(leg_geom_data_yaml)}"/>
     <xacro:property name="leg_geom_data_baseline" value="${load_yaml(leg_geom_data_baseline_yaml)}"/>
@@ -17,5 +17,4 @@
     <xacro:property name="shin_d" value="${leg_geom_data['shin_depth']}"/>
     <xacro:property name="foot_l" value="${leg_geom_data['foot_length']}"/>
-    <xacro:property name="chair_x_offset" value="${leg_geom_data['offset_chair_x']}"/>
     <xacro:property name="body_weight" value="${leg_geom_data['body_weight']}"/>
     <xacro:property name="body_weight_baseline" value="${leg_geom_data['body_weight']}"/>

File: leg_as_robot/urdf/right/leg.joints.xacro (robot description, xacro)
@@ -1,23 +1,10 @@
 <?xml version="1.0"?>
 <robot xmlns:xacro="http://www.ros.org/wiki/xacro">
-  <xacro:property name="base_to_hip_offset_x" value="${chair_x_offset}"/>
-  <xacro:property name="base_to_hip_offset_y" value="${- r7_leg - d3_leg}"/>
-  <xacro:property name="base_to_hip_offset_z" value="${r3_platform + d6_platform + d7_platform + d7_leg + r4_leg}"/>
-  <xacro:property name="base_to_hip_offset_baseline_y" value="${- r7Baseline_leg - d3Baseline_leg}"/>
-  <xacro:property name="base_to_hip_offset_baseline_z" value="${r3_platform + d6_platform + d7_platform +  d7Baseline_leg + r4Baseline_leg}"/>
-   <xacro:property name="base_to_hip_offset">
-      <origin xyz="${base_to_hip_offset_x} ${base_to_hip_offset_y} ${base_to_hip_offset_z}" rpy="0 0 0"/> <!-- <origin xyz="0 -0.5100 0.9246" rpy="0 0 0"/> -->
-  </xacro:property>
   <xacro:macro name="define_leg_joints">
-    <joint name="hip_fixed" type="fixed">
-      <xacro:insert_block name="base_to_hip_offset"/>
-      <parent link="virtual_platform_base_link"/>
-      <child link="hip_base_link"/>
-    </joint>
     <joint name="hip_adduction" type="revolute">
       <origin xyz="0 0 0" rpy="0 0 0"/>
       <parent link="hip_base_link"/>
       <child link="hip_adduction_link"/>
-      <limit effort="30" velocity="10.0" lower="${radians(-44)}" upper="${radians(10)}"/>
+      <limit effort="30" velocity="10.0" lower="${radians(-44)}" upper="${radians(0)}"/>
       <axis xyz="0 0 1"/>
     </joint>

File: leg_as_robot/urdf/right/leg.links.xacro (robot description, xacro)
@@ -1,11 +1,9 @@
 <?xml version="1.0"?>
 <robot xmlns:xacro="http://www.ros.org/wiki/xacro">
+  <xacro:arg name="with_chair" default="true"/>
   <xacro:property name="thigh_mass" value="${14.47 * 100.0/165.0 * body_weight / 100}"/> <!-- [kg] -->
-  <xacro:property name="shin_mass" value="${4.57 * 100.0/165.0 * body_weight / 100}"/> <!-- [kg] -->
-  <xacro:property name="foot_mass" value="${1.33 * 100.0/165.0 *body_weight / 100}"/> <!--[kg] -->
+  <xacro:property name="shin_mass" value="${4.57 * 100.0/165.0  * body_weight / 100}"/> <!-- [kg] -->
+  <xacro:property name="foot_mass" value="${1.33 * 100.0/165.0  *body_weight / 100}"/> <!--[kg] -->
   <xacro:property name="scale_mass" value="${body_weight / body_weight_baseline}"/>
-  <xacro:property name="base_scale_x" value="${1.0}"/>
-  <xacro:property name="base_scale_y" value="${base_to_hip_offset_y/base_to_hip_offset_baseline_y}"/>
-  <xacro:property name="base_scale_z" value="${base_to_hip_offset_z/base_to_hip_offset_baseline_z}"/>
   <xacro:property name="thigh_scale_x" value="${thigh_d/thighBaseline_d}"/>
   <xacro:property name="thigh_scale_y" value="${thigh_w/thighBaseline_w}"/>
@@ -18,19 +16,5 @@
   <xacro:property name="foot_scale_z" value="${d7_leg/d7Baseline_leg}"/>
   <xacro:macro name="define_leg_links">
-    <link name="virtual_platform_base_link"/>
-    <link name="hip_base_link">
-        <visual>
-          <origin rpy="0 0 0" xyz="0 0 0"/>
-          <geometry>
-            <mesh filename="package://leg_as_robot/model/meshes/dae/leg_base_visual.dae" scale ="${base_scale_x} ${base_scale_y} ${base_scale_z}"/>
-          </geometry>
-        </visual>
-        <collision>
-          <origin rpy="0 0 0" xyz="0 0 0"/>
-          <geometry>
-            <mesh filename="package://leg_as_robot/model/meshes/stl/leg_base_collision.stl" scale ="${base_scale_x} ${base_scale_y} ${base_scale_z}"/>
-          </geometry>
-        </collision>
-    </link>
+    <link name="hip_base_link"/>
     <link name="hip_adduction_link"/> <!-- virtual link-->
     <link name="hip_extension_link"/> <!-- virtual link-->
