Commit message: partial upgrade of robot definitions ( leg, platform, tool ) to be able to transition to Gazebo

File: leg_as_robot/urdf/left/leg.joints.xacro (robot description, xacro)
@@ -1,75 +1,75 @@
 <?xml version="1.0"?>
 <robot xmlns:xacro="http://www.ros.org/wiki/xacro">
-  <xacro:macro name="define_leg_joints">
-    <joint name="hip_adduction" type="revolute">
+  <xacro:macro name="define_leg_joints" params="leg_id:=left">
+    <joint name="${leg_id}_hip_adduction" type="revolute">
       <origin xyz="0 0 0" rpy="0 0 0"/>
-      <parent link="hip_base_link"/>
-      <child link="hip_adduction_link"/>
+      <parent link="${leg_id}_hip_base_link"/>
+      <child link="${leg_id}_hip_adduction_link"/>
       <limit effort="30" velocity="10.0" lower="${radians(0)}" upper="${radians(44)}"/>
       <axis xyz="0 0 1"/>
     </joint>
-    <joint name="hip_extension" type="revolute">
+    <joint name="${leg_id}_hip_extension" type="revolute">
       <origin xyz="0 0 0" rpy="${pi/2} 0 ${pi/2}"/>
-      <parent link="hip_adduction_link"/>
-      <child link="hip_extension_link"/>
+      <parent link="${leg_id}_hip_adduction_link"/>
+      <child link="${leg_id}_hip_extension_link"/>
       <limit effort="30" velocity="10.0" lower="${radians(-30)}" upper="${radians(32)}"/>
       <axis xyz="0 0 1"/>
     </joint>
-    <joint name="hip_roll" type="revolute">
+    <joint name="${leg_id}_hip_roll" type="revolute">
       <origin xyz="0 0 0" rpy="${pi/2} 0 ${pi/2}"/>
-      <parent link="hip_extension_link"/>
-      <child link="hip_roll_link"/>
+      <parent link="${leg_id}_hip_extension_link"/>
+      <child link="${leg_id}_hip_roll_link"/>
       <limit effort="30" velocity="10.0" lower="${radians(-33)}" upper="${radians(33)}"/>
       <axis xyz="0 0 1"/>
     </joint>
-    <joint name="knee_extension" type="revolute">
+    <joint name="${leg_id}_knee_extension" type="revolute">
       <origin xyz="0 0 ${d3_leg}" rpy="${-pi/2} 0 ${pi}"/>
-      <parent link="hip_roll_link"/>
-      <child link="knee_extension_link"/>
+      <parent link="${leg_id}_hip_roll_link"/>
+      <child link="${leg_id}_knee_extension_link"/>
       <limit effort="30" velocity="10.0" lower="${radians(-90)}" upper="${radians(30)}"/>
       <axis xyz="0 0 1"/>
     </joint>
-    <joint name="ankle_pitch" type="revolute">
+    <joint name="${leg_id}_ankle_pitch" type="revolute">
       <origin xyz="${r4_leg} 0 0" rpy="${pi} 0 ${pi}"/>
-      <parent link="knee_extension_link"/>
-      <child link="ankle_pitch_link"/>
+      <parent link="${leg_id}_knee_extension_link"/>
+      <child link="${leg_id}_ankle_pitch_link"/>
       <limit effort="30" velocity="10.0" lower="${radians(-45.8)}" upper="${radians(29.8)}"/>
       <axis xyz="0 0 1"/>
     </joint>
-    <joint name="ankle_roll" type="revolute">
+    <joint name="${leg_id}_ankle_roll" type="revolute">
       <origin xyz="0 0 0" rpy="${pi/2} 0 0"/>
-      <parent link="ankle_pitch_link"/>
-      <child link="ankle_roll_link"/>
+      <parent link="${leg_id}_ankle_pitch_link"/>
+      <child link="${leg_id}_ankle_roll_link"/>
       <limit effort="30" velocity="10.0" lower="${radians(-22)}" upper="${radians(17)}"/>
       <axis xyz="0 0 1"/>
     </joint>
-    <!-- <joint name="ankle_yaw" type="revolute">
+    <!-- <joint name="${leg_id}_ankle_yaw" type="revolute">
       <origin xyz="0 0 0" rpy="${-pi/2} 0 ${-pi/2}"/>
-      <parent link="ankle_roll_link"/>
-      <child link="ankle_yaw_link"/>
+      <parent link="${leg_id}_ankle_roll_link"/>
+      <child link="${leg_id}_ankle_yaw_link"/>
       <limit effort="30" velocity="10.0" lower="${radians(-36)}" upper="${radians(25.9)}"/>
       <axis xyz="0 0 1"/>
     </joint> -->
-    <joint name="ankle_yaw" type="revolute">
+    <joint name="${leg_id}_ankle_yaw" type="revolute">
       <origin xyz="0 0 0" rpy="${-pi/2} 0 ${-pi/2}"/>
-      <parent link="ankle_roll_link"/>
-      <child link="ankle_yaw_link"/>
+      <parent link="${leg_id}_ankle_roll_link"/>
+      <child link="${leg_id}_ankle_yaw_link"/>
       <limit effort="30" velocity="10.0" lower="${radians(-10)}" upper="${radians(5)}"/>
       <axis xyz="0 0 1"/>
     </joint>
-      <joint name="fixed_foot_base" type="fixed">
+      <joint name="${leg_id}_fixed_foot_base" type="fixed">
           <origin xyz="0 ${-r7_leg} ${-d7_leg}" rpy="0 0 ${-pi/2}"/>
-          <parent link="ankle_yaw_link"/>
-          <child link="foot_base"/>
+          <parent link="${leg_id}_ankle_yaw_link"/>
+          <child link="${leg_id}_foot_base"/>
       </joint>
-      <joint name="fixed_foot_tip" type="fixed">
+      <joint name="${leg_id}_fixed_foot_tip" type="fixed">
           <origin xyz="${r8_leg} 0 0" rpy="0 0 0"/>
-          <parent link="foot_base"/>
-          <child link="foot_tip"/>
+          <parent link="${leg_id}_foot_base"/>
+          <child link="${leg_id}_foot_tip"/>
       </joint>
-      <joint name="fixed_pedal_tip" type="fixed">
+      <joint name="${leg_id}_fixed_pedal_tip" type="fixed">
           <origin xyz="${r8_leg_extra} 0 0" rpy="0 0 0"/>
-          <parent link="foot_tip"/>
-          <child link="virtual_pedal_tip"/>
+          <parent link="${leg_id}_foot_tip"/>
+          <child link="${leg_id}_virtual_pedal_tip"/>
       </joint>
   </xacro:macro>

File: leg_as_robot/urdf/left/leg.links.xacro (robot description, xacro)
@@ -14,9 +14,9 @@
   <xacro:property name="foot_scale_y" value="${r8_leg/r8Baseline_leg}"/>
   <xacro:property name="foot_scale_z" value="${d7_leg/d7Baseline_leg}"/>
-  <xacro:macro name="define_leg_links">
-    <link name="hip_base_link"/>
-    <link name="hip_adduction_link"/> <!-- virtual link-->
-    <link name="hip_extension_link"/> <!-- virtual link-->
-    <link name="hip_roll_link" >
+  <xacro:macro name="define_leg_links" params="leg_id:=left">
+    <link name="${leg_id}_hip_base_link"/>
+    <link name="${leg_id}_hip_adduction_link"/> <!-- virtual link-->
+    <link name="${leg_id}_hip_extension_link"/> <!-- virtual link-->
+    <link name="${leg_id}_hip_roll_link" >
       <inertial>
       <origin xyz="${0.00265863 * thigh_scale_x} ${--0.00827375 * thigh_scale_y } ${0.17215567 * thigh_scale_z}" rpy="0 0 0"/>
@@ -37,5 +37,5 @@
       </collision>
     </link>
-    <link name="knee_extension_link" >
+    <link name="${leg_id}_knee_extension_link" >
       <inertial>
           <origin xyz="${0.14893265 * shin_scale_x} ${0.01010783 * shin_scale_y } ${--0.00938572 * shin_scale_z}" rpy="0 0 0"/>
@@ -56,7 +56,7 @@
       </collision>
     </link>
-    <link name="ankle_pitch_link" /> <!-- virtual link-->
-    <link name="ankle_roll_link" /> <!-- virtual link-->
-    <link name="ankle_yaw_link">
+    <link name="${leg_id}_ankle_pitch_link" /> <!-- virtual link-->
+    <link name="${leg_id}_ankle_roll_link" /> <!-- virtual link-->
+    <link name="${leg_id}_ankle_yaw_link">
         <inertial>
           <origin xyz="${--0.00089807 * foot_scale_x} ${-0.04499748 * foot_scale_y} ${-0.04201224 * foot_scale_z}" rpy="0 0 0"/>
@@ -77,7 +77,7 @@
       </collision>
     </link>
-    <link name="foot_base"/>
-    <link name="foot_tip"/>
-    <link name="virtual_pedal_tip"/>
+    <link name="${leg_id}_foot_base"/>
+    <link name="${leg_id}_foot_tip"/>
+    <link name="${leg_id}_virtual_pedal_tip"/>
   </xacro:macro>
 </robot>

File: leg_as_robot/urdf/right/leg.joints.xacro (robot description, xacro)
@@ -1,75 +1,75 @@
 <?xml version="1.0"?>
 <robot xmlns:xacro="http://www.ros.org/wiki/xacro">
-  <xacro:macro name="define_leg_joints">
-    <joint name="hip_adduction" type="revolute">
+  <xacro:macro name="define_leg_joints" params="leg_id:=right">
+    <joint name="${leg_id}_hip_adduction" type="revolute">
       <origin xyz="0 0 0" rpy="0 0 0"/>
-      <parent link="hip_base_link"/>
-      <child link="hip_adduction_link"/>
+      <parent link="${leg_id}_hip_base_link"/>
+      <child link="${leg_id}_hip_adduction_link"/>
       <limit effort="30" velocity="10.0" lower="${radians(-44)}" upper="${radians(30)}"/>
       <axis xyz="0 0 1"/>
     </joint>
-    <joint name="hip_extension" type="revolute">
+    <joint name="${leg_id}_hip_extension" type="revolute">
       <origin xyz="0 0 0" rpy="${pi/2} 0 ${pi/2}"/>
-      <parent link="hip_adduction_link"/>
-      <child link="hip_extension_link"/>
+      <parent link="${leg_id}_hip_adduction_link"/>
+      <child link="${leg_id}_hip_extension_link"/>
       <limit effort="30" velocity="10.0" lower="${radians(-30)}" upper="${radians(32)}"/>
       <axis xyz="0 0 1"/>
     </joint>
-    <joint name="hip_roll" type="revolute">
+    <joint name="${leg_id}_hip_roll" type="revolute">
       <origin xyz="0 0 0" rpy="${pi/2} 0 ${pi/2}"/>
-      <parent link="hip_extension_link"/>
-      <child link="hip_roll_link"/>
+      <parent link="${leg_id}_hip_extension_link"/>
+      <child link="${leg_id}_hip_roll_link"/>
       <limit effort="30" velocity="10.0" lower="${radians(-45)}" upper="${radians(45)}"/>
       <axis xyz="0 0 1"/>
     </joint>
-    <joint name="knee_extension" type="revolute">
+    <joint name="${leg_id}_knee_extension" type="revolute">
       <origin xyz="0 0 ${d3_leg}" rpy="${-pi/2} 0 ${pi}"/>
-      <parent link="hip_roll_link"/>
-      <child link="knee_extension_link"/>
+      <parent link="${leg_id}_hip_roll_link"/>
+      <child link="${leg_id}_knee_extension_link"/>
       <limit effort="30" velocity="10.0" lower="${radians(-90)}" upper="${radians(30)}"/>
       <axis xyz="0 0 1"/>
     </joint>
-    <joint name="ankle_pitch" type="revolute">
+    <joint name="${leg_id}_ankle_pitch" type="revolute">
       <origin xyz="${r4_leg} 0 0" rpy="${pi} 0 ${pi}"/>
-      <parent link="knee_extension_link"/>
-      <child link="ankle_pitch_link"/>
+      <parent link="${leg_id}_knee_extension_link"/>
+      <child link="${leg_id}_ankle_pitch_link"/>
       <limit effort="30" velocity="10.0" lower="${radians(-45.8)}" upper="${radians(29.8)}"/>
       <axis xyz="0 0 1"/>
     </joint>
-    <joint name="ankle_roll" type="revolute">
+    <joint name="${leg_id}_ankle_roll" type="revolute">
       <origin xyz="0 0 0" rpy="${pi/2} 0 0"/>
-      <parent link="ankle_pitch_link"/>
-      <child link="ankle_roll_link"/>
+      <parent link="${leg_id}_ankle_pitch_link"/>
+      <child link="${leg_id}_ankle_roll_link"/>
       <limit effort="30" velocity="10.0" lower="${radians(-17)}" upper="${radians(22)}"/>
       <axis xyz="0 0 1"/>
     </joint>
-    <joint name="ankle_yaw" type="revolute">
+    <joint name="${leg_id}_ankle_yaw" type="revolute">
       <origin xyz="0 0 0" rpy="${-pi/2} 0 ${-pi/2}"/>
-      <parent link="ankle_roll_link"/>
-      <child link="ankle_yaw_link"/>
+      <parent link="${leg_id}_ankle_roll_link"/>
+      <child link="${leg_id}_ankle_yaw_link"/>
       <limit effort="30" velocity="10.0" lower="${radians(-25.9)}" upper="${radians(36)}"/>
       <axis xyz="0 0 1"/>
     </joint>
-     <!-- <joint name="ankle_yaw" type="revolute">
+     <!-- <joint name="${leg_id}_ankle_yaw" type="revolute">
       <origin xyz="0 0 0" rpy="${-pi/2} 0 ${-pi/2}"/>
-      <parent link="ankle_roll_link"/>
-      <child link="ankle_yaw_link"/>
+      <parent link="${leg_id}_ankle_roll_link"/>
+      <child link="${leg_id}_ankle_yaw_link"/>
       <limit effort="30" velocity="10.0" lower="${radians(-5)}" upper="${radians(10)}"/>
       <axis xyz="0 0 1"/>
     </joint> -->
-      <joint name="fixed_foot_base" type="fixed">
+      <joint name="${leg_id}_fixed_foot_base" type="fixed">
           <origin xyz="0 ${-r7_leg} ${-d7_leg}" rpy="0 0 ${-pi/2}"/>
-          <parent link="ankle_yaw_link"/>
-          <child link="foot_base"/>
+          <parent link="${leg_id}_ankle_yaw_link"/>
+          <child link="${leg_id}_foot_base"/>
       </joint>
-      <joint name="fixed_foot_tip" type="fixed">
+      <joint name="${leg_id}_fixed_foot_tip" type="fixed">
           <origin xyz="${r8_leg} 0 0" rpy="0 0 0"/>
-          <parent link="foot_base"/>
-          <child link="foot_tip"/>
+          <parent link="${leg_id}_foot_base"/>
+          <child link="${leg_id}_foot_tip"/>
       </joint>
-      <joint name="fixed_pedal_tip" type="fixed">
+      <joint name="${leg_id}_fixed_pedal_tip" type="fixed">
           <origin xyz="${r8_leg_extra} 0 0" rpy="0 0 0"/>
-          <parent link="foot_tip"/>
-          <child link="virtual_pedal_tip"/>
+          <parent link="${leg_id}_foot_tip"/>
+          <child link="${leg_id}_virtual_pedal_tip"/>
       </joint>
   </xacro:macro>

File: leg_as_robot/urdf/right/leg.links.xacro (robot description, xacro)
@@ -20,9 +20,9 @@
   <xacro:property name="foot_scale_y" value="${r8_leg/r8Baseline_leg}"/>
   <xacro:property name="foot_scale_z" value="${d7_leg/d7Baseline_leg}"/>
-  <xacro:macro name="define_leg_links">
-    <link name="hip_base_link"/>
-    <link name="hip_adduction_link"/> <!-- virtual link-->
-    <link name="hip_extension_link"/> <!-- virtual link-->
-    <link name="hip_roll_link" >
+  <xacro:macro name="define_leg_links" params="leg_id:=right">
+    <link name="${leg_id}_hip_base_link"/>
+    <link name="${leg_id}_hip_adduction_link"/> <!-- virtual link-->
+    <link name="${leg_id}_hip_extension_link"/> <!-- virtual link-->
+    <link name="${leg_id}_hip_roll_link" >
       <inertial>
       <origin xyz="${0.00265863 * thigh_scale_x} ${-0.00827375 * thigh_scale_y } ${0.17215567 * thigh_scale_z}" rpy="0 0 0"/>
@@ -43,5 +43,5 @@
       </collision>
     </link>
-    <link name="knee_extension_link" >
+    <link name="${leg_id}_knee_extension_link" >
       <inertial>
           <origin xyz="${0.14893265 * shin_scale_x} ${0.01010783 * shin_scale_y } ${-0.00938572 * shin_scale_z}" rpy="0 0 0"/>
@@ -62,7 +62,7 @@
       </collision>
     </link>
-    <link name="ankle_pitch_link" /> <!-- virtual link-->
-    <link name="ankle_roll_link" /> <!-- virtual link-->
-    <link name="ankle_yaw_link">
+    <link name="${leg_id}_ankle_pitch_link" /> <!-- virtual link-->
+    <link name="${leg_id}_ankle_roll_link" /> <!-- virtual link-->
+    <link name="${leg_id}_ankle_yaw_link">
         <inertial>
           <origin xyz="${-0.00089807 * foot_scale_x} ${-0.04499748 * foot_scale_y} ${-0.04201224 * foot_scale_z}" rpy="0 0 0"/>
@@ -83,7 +83,7 @@
       </collision>
     </link>
-    <link name="foot_base"/>
-    <link name="foot_tip"/>
-    <link name="virtual_pedal_tip"/>
+    <link name="${leg_id}_foot_base"/>
+    <link name="${leg_id}_foot_tip"/>
+    <link name="${leg_id}_virtual_pedal_tip"/>
   </xacro:macro>
 </robot>

File: surgical_sim/urdf/body/body_create.urdf.xacro (robot description, xacro)
@@ -20,5 +20,5 @@
   <xacro:unless value="$(arg with_liver)">
   </xacro:unless>
-    <!-- <gazebo>
+    <gazebo>
         <plugin name="gazebo_ros_control" filename="libgazebo_ros_control.so">
         <robotNamespace>/body</robotNamespace>
@@ -26,4 +26,4 @@
         <legacyModeNS>true</legacyModeNS>
         </plugin>
-    </gazebo> -->
+    </gazebo>
 </robot>

File: surgical_sim/urdf/surgical_tool/templates/joint.transmissions.xacro (robot description, xacro)
@@ -5,8 +5,8 @@
 			<type>transmission_interface/SimpleTransmission</type>
 			<joint name="${name}">
-				<hardwareInterface>hardware_interface/EffortJointInterface</hardwareInterface>
+				<hardwareInterface>hardware_interface/PositionJointInterface</hardwareInterface>
 			</joint>
 			<actuator name="${name}_motor">
-				<hardwareInterface>hardware_interface/EffortJointInterface</hardwareInterface>
+				<hardwareInterface>hardware_interface/PositionJointInterface</hardwareInterface>
 				<mechanicalReduction>${reduction}</mechanicalReduction>
 			</actuator>

File: surgical_sim/urdf/surgical_tool/tool_create.urdf.xacro (robot description, xacro)
@@ -22,5 +22,5 @@
   </xacro:macro>
  <!--  -->
-  <link name="/world"/>
+  <link name="world"/>
   <link name="tool_base_link">
     <inertial>
@@ -43,5 +43,5 @@
   </xacro:unless>
   <joint name="world_fixed" type="fixed">
-      <parent link="/world"/>
+      <parent link="world"/>
       <child link="tool_base_link"/>
       <origin rpy="0 0 0" xyz="${0+0.015} ${0.5 + 0.015} ${1.1 + 0.2} "/>
@@ -49,8 +49,8 @@
     <gazebo>
         <plugin name="gazebo_ros_control" filename="libgazebo_ros_control.so">
-        <robotNamespace>surgical_tool</robotNamespace>
-        <robotParam>/$(arg toolID)/tool_description</robotParam>
+        <robotNamespace>$(arg toolID)_tool</robotNamespace>
+        <robotParam>/$(arg toolID)_tool/robot_description</robotParam>
         <robotSimType>gazebo_ros_control/DefaultRobotHWSim</robotSimType>
-        <legacyModeNS>true</legacyModeNS>
+        <legacyModeNS>false</legacyModeNS>
         </plugin>
     </gazebo>

File: surgical_sim/urdf/surgical_tool/tool_forceps/tool_t_forceps.joints.xacro (robot description, xacro)
@@ -27,5 +27,5 @@
       <axis xyz="0 0 1"/>
       <origin rpy="0 0 0" xyz="0 0 0"/>
-      <limit lower="0" upper="${radians(30)}" velocity="3.0" effort="1000"/>
+      <limit lower="0" upper="${radians(20.5)}" velocity="3.0" effort="1000"/>
     </joint>
   <!-- joint 6-2: tool open angle 2  -->
@@ -35,5 +35,5 @@
       <axis xyz="0 0 1"/>
       <origin rpy="3.1415926 0 0" xyz="0 0 0"/>
-      <limit lower="0" upper="${radians(30)}" velocity="3.0" effort="1000"/>
+      <limit lower="0" upper="${radians(20.5)}" velocity="3.0" effort="1000"/>
       <mimic joint="tool_wrist_open_angle" multiplier="1"/>
     </joint>
