Commit message: changed the namespace of the topics in footVarSync and ForceMeas. Now the leg compensation works and the force sensor compensation

File: leg_as_robot/urdf/left/leg.joints.xacro (robot description, xacro)
@@ -2,74 +2,74 @@
 <robot xmlns:xacro="http://www.ros.org/wiki/xacro">
   <xacro:macro name="define_leg_joints" params="leg_id:=left">
-    <joint name="${leg_id}_hip_adduction" type="revolute">
+    <joint name="${leg_id}_leg_hip_adduction" type="revolute">
       <origin xyz="0 0 0" rpy="0 0 0"/>
-      <parent link="${leg_id}_hip_base_link"/>
-      <child link="${leg_id}_hip_adduction_link"/>
+      <parent link="${leg_id}_leg_hip_base_link"/>
+      <child link="${leg_id}_leg_hip_adduction_link"/>
       <limit effort="30" velocity="10.0" lower="${radians(0)}" upper="${radians(44)}"/>
       <axis xyz="0 0 1"/>
     </joint>
-    <joint name="${leg_id}_hip_extension" type="revolute">
+    <joint name="${leg_id}_leg_hip_extension" type="revolute">
       <origin xyz="0 0 0" rpy="${pi/2} 0 ${pi/2}"/>
-      <parent link="${leg_id}_hip_adduction_link"/>
-      <child link="${leg_id}_hip_extension_link"/>
+      <parent link="${leg_id}_leg_hip_adduction_link"/>
+      <child link="${leg_id}_leg_hip_extension_link"/>
       <limit effort="30" velocity="10.0" lower="${radians(-30)}" upper="${radians(32)}"/>
       <axis xyz="0 0 1"/>
     </joint>
-    <joint name="${leg_id}_hip_roll" type="revolute">
+    <joint name="${leg_id}_leg_hip_roll" type="revolute">
       <origin xyz="0 0 0" rpy="${pi/2} 0 ${pi/2}"/>
-      <parent link="${leg_id}_hip_extension_link"/>
-      <child link="${leg_id}_hip_roll_link"/>
+      <parent link="${leg_id}_leg_hip_extension_link"/>
+      <child link="${leg_id}_leg_hip_roll_link"/>
       <limit effort="30" velocity="10.0" lower="${radians(-33)}" upper="${radians(33)}"/>
       <axis xyz="0 0 1"/>
     </joint>
-    <joint name="${leg_id}_knee_extension" type="revolute">
+    <joint name="${leg_id}_leg_knee_extension" type="revolute">
       <origin xyz="0 0 ${d3_leg}" rpy="${-pi/2} 0 ${pi}"/>
-      <parent link="${leg_id}_hip_roll_link"/>
-      <child link="${leg_id}_knee_extension_link"/>
+      <parent link="${leg_id}_leg_hip_roll_link"/>
+      <child link="${leg_id}_leg_knee_extension_link"/>
       <limit effort="30" velocity="10.0" lower="${radians(-90)}" upper="${radians(30)}"/>
       <axis xyz="0 0 1"/>
     </joint>
-    <joint name="${leg_id}_ankle_pitch" type="revolute">
+    <joint name="${leg_id}_leg_ankle_pitch" type="revolute">
       <origin xyz="${r4_leg} 0 0" rpy="${pi} 0 ${pi}"/>
-      <parent link="${leg_id}_knee_extension_link"/>
-      <child link="${leg_id}_ankle_pitch_link"/>
+      <parent link="${leg_id}_leg_knee_extension_link"/>
+      <child link="${leg_id}_leg_ankle_pitch_link"/>
       <limit effort="30" velocity="10.0" lower="${radians(-45.8)}" upper="${radians(29.8)}"/>
       <axis xyz="0 0 1"/>
     </joint>
-    <joint name="${leg_id}_ankle_roll" type="revolute">
+    <joint name="${leg_id}_leg_ankle_roll" type="revolute">
       <origin xyz="0 0 0" rpy="${pi/2} 0 0"/>
-      <parent link="${leg_id}_ankle_pitch_link"/>
-      <child link="${leg_id}_ankle_roll_link"/>
+      <parent link="${leg_id}_leg_ankle_pitch_link"/>
+      <child link="${leg_id}_leg_ankle_roll_link"/>
       <limit effort="30" velocity="10.0" lower="${radians(-22)}" upper="${radians(17)}"/>
       <axis xyz="0 0 1"/>
     </joint>
-    <!-- <joint name="${leg_id}_ankle_yaw" type="revolute">
+    <!-- <joint name="${leg_id}_leg_ankle_yaw" type="revolute">
       <origin xyz="0 0 0" rpy="${-pi/2} 0 ${-pi/2}"/>
-      <parent link="${leg_id}_ankle_roll_link"/>
-      <child link="${leg_id}_ankle_yaw_link"/>
+      <parent link="${leg_id}_leg_ankle_roll_link"/>
+      <child link="${leg_id}_leg_ankle_yaw_link"/>
       <limit effort="30" velocity="10.0" lower="${radians(-36)}" upper="${radians(25.9)}"/>
       <axis xyz="0 0 1"/>
     </joint> -->
-    <joint name="${leg_id}_ankle_yaw" type="revolute">
+    <joint name="${leg_id}_leg_ankle_yaw" type="revolute">
       <origin xyz="0 0 0" rpy="${-pi/2} 0 ${-pi/2}"/>
-      <parent link="${leg_id}_ankle_roll_link"/>
-      <child link="${leg_id}_ankle_yaw_link"/>
+      <parent link="${leg_id}_leg_ankle_roll_link"/>
+      <child link="${leg_id}_leg_ankle_yaw_link"/>
       <limit effort="30" velocity="10.0" lower="${radians(-10)}" upper="${radians(5)}"/>
       <axis xyz="0 0 1"/>
     </joint>
-      <joint name="${leg_id}_fixed_foot_base" type="fixed">
+      <joint name="${leg_id}_leg_fixed_foot_base" type="fixed">
           <origin xyz="0 ${-r7_leg} ${-d7_leg}" rpy="0 0 ${-pi/2}"/>
-          <parent link="${leg_id}_ankle_yaw_link"/>
-          <child link="${leg_id}_foot_base"/>
+          <parent link="${leg_id}_leg_ankle_yaw_link"/>
+          <child link="${leg_id}_leg_foot_base"/>
       </joint>
-      <joint name="${leg_id}_fixed_foot_tip" type="fixed">
+      <joint name="${leg_id}_leg_fixed_foot_tip" type="fixed">
           <origin xyz="${r8_leg} 0 0" rpy="0 0 0"/>
-          <parent link="${leg_id}_foot_base"/>
-          <child link="${leg_id}_foot_tip"/>
+          <parent link="${leg_id}_leg_foot_base"/>
+          <child link="${leg_id}_leg_foot_tip"/>
       </joint>
-      <joint name="${leg_id}_fixed_pedal_tip" type="fixed">
+      <joint name="${leg_id}_leg_fixed_pedal_tip" type="fixed">
           <origin xyz="${r8_leg_extra} 0 0" rpy="0 0 0"/>
-          <parent link="${leg_id}_foot_tip"/>
-          <child link="${leg_id}_virtual_pedal_tip"/>
+          <parent link="${leg_id}_leg_foot_tip"/>
+          <child link="${leg_id}_leg_virtual_pedal_tip"/>
       </joint>
   </xacro:macro>

File: leg_as_robot/urdf/left/leg.links.xacro (robot description, xacro)
@@ -15,8 +15,8 @@
   <xacro:property name="foot_scale_z" value="${d7_leg/d7Baseline_leg}"/>
   <xacro:macro name="define_leg_links" params="leg_id:=left">
-    <link name="${leg_id}_hip_base_link"/>
-    <link name="${leg_id}_hip_adduction_link"/> <!-- virtual link-->
-    <link name="${leg_id}_hip_extension_link"/> <!-- virtual link-->
-    <link name="${leg_id}_hip_roll_link" >
+    <link name="${leg_id}_leg_hip_base_link"/>
+    <link name="${leg_id}_leg_hip_adduction_link"/> <!-- virtual link-->
+    <link name="${leg_id}_leg_hip_extension_link"/> <!-- virtual link-->
+    <link name="${leg_id}_leg_hip_roll_link" >
       <inertial>
       <origin xyz="${0.00265863 * thigh_scale_x} ${--0.00827375 * thigh_scale_y } ${0.17215567 * thigh_scale_z}" rpy="0 0 0"/>
@@ -37,5 +37,5 @@
       </collision>
     </link>
-    <link name="${leg_id}_knee_extension_link" >
+    <link name="${leg_id}_leg_knee_extension_link" >
       <inertial>
           <origin xyz="${0.14893265 * shin_scale_x} ${0.01010783 * shin_scale_y } ${--0.00938572 * shin_scale_z}" rpy="0 0 0"/>
@@ -56,7 +56,7 @@
       </collision>
     </link>
-    <link name="${leg_id}_ankle_pitch_link" /> <!-- virtual link-->
-    <link name="${leg_id}_ankle_roll_link" /> <!-- virtual link-->
-    <link name="${leg_id}_ankle_yaw_link">
+    <link name="${leg_id}_leg_ankle_pitch_link" /> <!-- virtual link-->
+    <link name="${leg_id}_leg_ankle_roll_link" /> <!-- virtual link-->
+    <link name="${leg_id}_leg_ankle_yaw_link">
         <inertial>
           <origin xyz="${--0.00089807 * foot_scale_x} ${-0.04499748 * foot_scale_y} ${-0.04201224 * foot_scale_z}" rpy="0 0 0"/>
@@ -77,7 +77,7 @@
       </collision>
     </link>
-    <link name="${leg_id}_foot_base"/>
-    <link name="${leg_id}_foot_tip"/>
-    <link name="${leg_id}_virtual_pedal_tip"/>
+    <link name="${leg_id}_leg_foot_base"/>
+    <link name="${leg_id}_leg_foot_tip"/>
+    <link name="${leg_id}_leg_virtual_pedal_tip"/>
   </xacro:macro>
 </robot>

File: leg_as_robot/urdf/right/leg.joints.xacro (robot description, xacro)
@@ -2,74 +2,74 @@
 <robot xmlns:xacro="http://www.ros.org/wiki/xacro">
   <xacro:macro name="define_leg_joints" params="leg_id:=right">
-    <joint name="${leg_id}_hip_adduction" type="revolute">
+    <joint name="${leg_id}_leg_hip_adduction" type="revolute">
       <origin xyz="0 0 0" rpy="0 0 0"/>
-      <parent link="${leg_id}_hip_base_link"/>
-      <child link="${leg_id}_hip_adduction_link"/>
+      <parent link="${leg_id}_leg_hip_base_link"/>
+      <child link="${leg_id}_leg_hip_adduction_link"/>
       <limit effort="30" velocity="10.0" lower="${radians(-44)}" upper="${radians(30)}"/>
       <axis xyz="0 0 1"/>
     </joint>
-    <joint name="${leg_id}_hip_extension" type="revolute">
+    <joint name="${leg_id}_leg_hip_extension" type="revolute">
       <origin xyz="0 0 0" rpy="${pi/2} 0 ${pi/2}"/>
-      <parent link="${leg_id}_hip_adduction_link"/>
-      <child link="${leg_id}_hip_extension_link"/>
+      <parent link="${leg_id}_leg_hip_adduction_link"/>
+      <child link="${leg_id}_leg_hip_extension_link"/>
       <limit effort="30" velocity="10.0" lower="${radians(-30)}" upper="${radians(32)}"/>
       <axis xyz="0 0 1"/>
     </joint>
-    <joint name="${leg_id}_hip_roll" type="revolute">
+    <joint name="${leg_id}_leg_hip_roll" type="revolute">
       <origin xyz="0 0 0" rpy="${pi/2} 0 ${pi/2}"/>
-      <parent link="${leg_id}_hip_extension_link"/>
-      <child link="${leg_id}_hip_roll_link"/>
+      <parent link="${leg_id}_leg_hip_extension_link"/>
+      <child link="${leg_id}_leg_hip_roll_link"/>
       <limit effort="30" velocity="10.0" lower="${radians(-45)}" upper="${radians(45)}"/>
       <axis xyz="0 0 1"/>
     </joint>
-    <joint name="${leg_id}_knee_extension" type="revolute">
+    <joint name="${leg_id}_leg_knee_extension" type="revolute">
       <origin xyz="0 0 ${d3_leg}" rpy="${-pi/2} 0 ${pi}"/>
-      <parent link="${leg_id}_hip_roll_link"/>
-      <child link="${leg_id}_knee_extension_link"/>
+      <parent link="${leg_id}_leg_hip_roll_link"/>
+      <child link="${leg_id}_leg_knee_extension_link"/>
       <limit effort="30" velocity="10.0" lower="${radians(-90)}" upper="${radians(30)}"/>
       <axis xyz="0 0 1"/>
     </joint>
-    <joint name="${leg_id}_ankle_pitch" type="revolute">
+    <joint name="${leg_id}_leg_ankle_pitch" type="revolute">
       <origin xyz="${r4_leg} 0 0" rpy="${pi} 0 ${pi}"/>
-      <parent link="${leg_id}_knee_extension_link"/>
-      <child link="${leg_id}_ankle_pitch_link"/>
+      <parent link="${leg_id}_leg_knee_extension_link"/>
+      <child link="${leg_id}_leg_ankle_pitch_link"/>
       <limit effort="30" velocity="10.0" lower="${radians(-45.8)}" upper="${radians(29.8)}"/>
       <axis xyz="0 0 1"/>
     </joint>
-    <joint name="${leg_id}_ankle_roll" type="revolute">
+    <joint name="${leg_id}_leg_ankle_roll" type="revolute">
       <origin xyz="0 0 0" rpy="${pi/2} 0 0"/>
-      <parent link="${leg_id}_ankle_pitch_link"/>
-      <child link="${leg_id}_ankle_roll_link"/>
+      <parent link="${leg_id}_leg_ankle_pitch_link"/>
+      <child link="${leg_id}_leg_ankle_roll_link"/>
       <limit effort="30" velocity="10.0" lower="${radians(-17)}" upper="${radians(22)}"/>
       <axis xyz="0 0 1"/>
     </joint>
-    <joint name="${leg_id}_ankle_yaw" type="revolute">
+    <joint name="${leg_id}_leg_ankle_yaw" type="revolute">
       <origin xyz="0 0 0" rpy="${-pi/2} 0 ${-pi/2}"/>
-      <parent link="${leg_id}_ankle_roll_link"/>
-      <child link="${leg_id}_ankle_yaw_link"/>
+      <parent link="${leg_id}_leg_ankle_roll_link"/>
+      <child link="${leg_id}_leg_ankle_yaw_link"/>
       <limit effort="30" velocity="10.0" lower="${radians(-25.9)}" upper="${radians(36)}"/>
       <axis xyz="0 0 1"/>
     </joint>
-     <!-- <joint name="${leg_id}_ankle_yaw" type="revolute">
+     <!-- <joint name="${leg_id}_leg_ankle_yaw" type="revolute">
       <origin xyz="0 0 0" rpy="${-pi/2} 0 ${-pi/2}"/>
-      <parent link="${leg_id}_ankle_roll_link"/>
-      <child link="${leg_id}_ankle_yaw_link"/>
+      <parent link="${leg_id}_leg_ankle_roll_link"/>
+      <child link="${leg_id}_leg_ankle_yaw_link"/>
       <limit effort="30" velocity="10.0" lower="${radians(-5)}" upper="${radians(10)}"/>
       <axis xyz="0 0 1"/>
     </joint> -->
-      <joint name="${leg_id}_fixed_foot_base" type="fixed">
+      <joint name="${leg_id}_leg_fixed_foot_base" type="fixed">
           <origin xyz="0 ${-r7_leg} ${-d7_leg}" rpy="0 0 ${-pi/2}"/>
-          <parent link="${leg_id}_ankle_yaw_link"/>
-          <child link="${leg_id}_foot_base"/>
+          <parent link="${leg_id}_leg_ankle_yaw_link"/>
+          <child link="${leg_id}_leg_foot_base"/>
       </joint>
-      <joint name="${leg_id}_fixed_foot_tip" type="fixed">
+      <joint name="${leg_id}_leg_fixed_foot_tip" type="fixed">
           <origin xyz="${r8_leg} 0 0" rpy="0 0 0"/>
-          <parent link="${leg_id}_foot_base"/>
-          <child link="${leg_id}_foot_tip"/>
+          <parent link="${leg_id}_leg_foot_base"/>
+          <child link="${leg_id}_leg_foot_tip"/>
       </joint>
-      <joint name="${leg_id}_fixed_pedal_tip" type="fixed">
+      <joint name="${leg_id}_leg_fixed_pedal_tip" type="fixed">
           <origin xyz="${r8_leg_extra} 0 0" rpy="0 0 0"/>
-          <parent link="${leg_id}_foot_tip"/>
-          <child link="${leg_id}_virtual_pedal_tip"/>
+          <parent link="${leg_id}_leg_foot_tip"/>
+          <child link="${leg_id}_leg_virtual_pedal_tip"/>
       </joint>
   </xacro:macro>

File: leg_as_robot/urdf/right/leg.links.xacro (robot description, xacro)
@@ -21,8 +21,8 @@
   <xacro:property name="foot_scale_z" value="${d7_leg/d7Baseline_leg}"/>
   <xacro:macro name="define_leg_links" params="leg_id:=right">
-    <link name="${leg_id}_hip_base_link"/>
-    <link name="${leg_id}_hip_adduction_link"/> <!-- virtual link-->
-    <link name="${leg_id}_hip_extension_link"/> <!-- virtual link-->
-    <link name="${leg_id}_hip_roll_link" >
+    <link name="${leg_id}_leg_hip_base_link"/>
+    <link name="${leg_id}_leg_hip_adduction_link"/> <!-- virtual link-->
+    <link name="${leg_id}_leg_hip_extension_link"/> <!-- virtual link-->
+    <link name="${leg_id}_leg_hip_roll_link" >
       <inertial>
       <origin xyz="${0.00265863 * thigh_scale_x} ${-0.00827375 * thigh_scale_y } ${0.17215567 * thigh_scale_z}" rpy="0 0 0"/>
@@ -43,5 +43,5 @@
       </collision>
     </link>
-    <link name="${leg_id}_knee_extension_link" >
+    <link name="${leg_id}_leg_knee_extension_link" >
       <inertial>
           <origin xyz="${0.14893265 * shin_scale_x} ${0.01010783 * shin_scale_y } ${-0.00938572 * shin_scale_z}" rpy="0 0 0"/>
@@ -62,7 +62,7 @@
       </collision>
     </link>
-    <link name="${leg_id}_ankle_pitch_link" /> <!-- virtual link-->
-    <link name="${leg_id}_ankle_roll_link" /> <!-- virtual link-->
-    <link name="${leg_id}_ankle_yaw_link">
+    <link name="${leg_id}_leg_ankle_pitch_link" /> <!-- virtual link-->
+    <link name="${leg_id}_leg_ankle_roll_link" /> <!-- virtual link-->
+    <link name="${leg_id}_leg_ankle_yaw_link">
         <inertial>
           <origin xyz="${-0.00089807 * foot_scale_x} ${-0.04499748 * foot_scale_y} ${-0.04201224 * foot_scale_z}" rpy="0 0 0"/>
@@ -83,7 +83,7 @@
       </collision>
     </link>
-    <link name="${leg_id}_foot_base"/>
-    <link name="${leg_id}_foot_tip"/>
-    <link name="${leg_id}_virtual_pedal_tip"/>
+    <link name="${leg_id}_leg_foot_base"/>
+    <link name="${leg_id}_leg_foot_tip"/>
+    <link name="${leg_id}_leg_virtual_pedal_tip"/>
   </xacro:macro>
 </robot>

File: surgical_sim/models/urdf/target_object/templates/gazebo.links.xacro (robot description, xacro)
@@ -1,6 +1,6 @@
 <?xml version="1.0"?>
 <robot xmlns:xacro="http://www.ros.org/wiki/xacro">
-	<xacro:property name="fricCoeff1" value="2.0"/>
-	<xacro:property name="fricCoeff2" value="2.0"/>
+	<xacro:property name="fricCoeff1" value="100.0"/>
+	<xacro:property name="fricCoeff2" value="100.0"/>
 	<xacro:property name="kpCollision" value="100000000.0"/>
 	<xacro:property name="kdCollision" value="100000000.0"/>
@@ -10,6 +10,6 @@
 			<mu1>${fricCoeff1}</mu1>
 			<mu2>${fricCoeff2}</mu2>
-			<kp>${kpCollision}</kp>
-			<kd>${kdCollision}</kd>
+			<!-- <kp>${kpCollision}</kp> -->
+			<!-- <kd>${kdCollision}</kd> -->
 			<selfCollide>true</selfCollide>
 			<!-- <maxVel>0.01</maxVel> -->
