Commit message: latest stable version

File: leg_as_robot/urdf/left/leg.links.xacro (robot description, xacro)
@@ -1,5 +1,5 @@
 <?xml version="1.0"?>
 <robot xmlns:xacro="http://www.ros.org/wiki/xacro">
-  <xacro:property name="thigh_mass" value="${14.47 * 100.0/165.0 * body_weight / 100}"/> <!-- [kg] -->
+  <xacro:property name="thigh_mass" value="${14.47 * 90.0/165.0 * body_weight / 100}"/> <!-- [kg] -->
   <xacro:property name="shin_mass" value="${4.57 * body_weight / 100}"/> <!-- [kg] -->
   <xacro:property name="foot_mass" value="${1.33 * body_weight / 100}"/> <!--[kg] -->

File: leg_as_robot/urdf/right/leg.links.xacro (robot description, xacro)
@@ -4,5 +4,5 @@
   <xacro:property name="thigh_mass" value="${14.47 * 100.0/165.0 * body_weight / 100}"/> <!-- [kg] -->
   <xacro:property name="shin_mass" value="${4.57 * body_weight / 100}"/> <!-- [kg] -->
-  <xacro:property name="foot_mass" value="${1.33 * 100.0/165.0  *body_weight / 100}"/> <!--[kg] -->
+  <xacro:property name="foot_mass" value="${1.33 * body_weight / 100}"/> <!--[kg] -->
   <xacro:property name="scale_mass" value="${body_weight / body_weight_baseline}"/>
   <xacro:property name="thigh_scale_x" value="${thigh_d/thighBaseline_d}"/>

File: surgical_sim/urdf/body/templates/gazebo.joints.xacro (robot description, xacro)
@@ -5,7 +5,7 @@
 			<implicitSpringDamper>0</implicitSpringDamper>
 			<provideFeedback>1</provideFeedback>
-			<!--stopCfm></stopCfm--> <!-- Force Mixing Error -->
-			<!--stopErp></stopErp--> <!-- Error Reduction Parameter -->
-			<!-- <fudgeFactor>0.5</fudgeFactor> -->
+			<stopCfm></stopCfm> <!-- Force Mixing Error -->
+			<stopErp></stopErp> <!-- Error Reduction Parameter -->
+			<fudgeFactor>0.5</fudgeFactor>
 		</gazebo>
 	</xacro:macro>

File: surgical_sim/urdf/body/torso/torso.joints.xacro (robot description, xacro)
@@ -27,5 +27,5 @@
     </joint>
     <!-- <xacro:joint_trans name="torso_joint" reduction="1"/> -->
-    <!-- <xacro:gazebo_joints name="torso_joint"/> -->
+    <xacro:gazebo_joints name="torso_joint"/>
   </xacro:macro>
 </robot>

File: surgical_sim/urdf/body/torso/torso.links.xacro (robot description, xacro)
@@ -11,13 +11,15 @@
         </geometry>
       </visual>
-      <!-- <inertial>
+      <inertial>
 				<origin xyz="0 0 0" rpy="0 0 0"/>
-				<mass value="1"/>
-				<inertia ixx="1" ixy="0.0" ixz="0.0" iyy="1" iyz="0.0" izz="1"/>
-			</inertial>  -->
+				<mass value="30"/>
+				<inertia ixx="0.5" ixy="0.0" ixz="0.0" iyy="0.5" iyz="0.0" izz="0.5"/>
+			</inertial>
     </link>
    <link name="/left/trocar_link"/>
    <link name="/right/trocar_link"/>
    <xacro:gazebo_links name="torso_link"/>
+   <!-- <xacro:gazebo_links name="/left/trocar_link"/>
+   <xacro:gazebo_links name="/right/trocar_link"/> -->
   </xacro:macro>
 </robot>

File: surgical_sim/urdf/surgical_tool/templates/gazebo.joints.xacro (robot description, xacro)
@@ -5,7 +5,7 @@
 			<implicitSpringDamper>0</implicitSpringDamper>
 			<provideFeedback>1</provideFeedback>
-			<!--stopCfm></stopCfm--> <!-- Force Mixing Error -->
-			<!--stopErp></stopErp--> <!-- Error Reduction Parameter -->
-			<!-- <fudgeFactor>0.5</fudgeFactor> -->
+			<stopCfm></stopCfm>
+			<stopErp></stopErp>
+			<fudgeFactor>0.5</fudgeFactor>
 		</gazebo>
 	</xacro:macro>

File: surgical_sim/urdf/surgical_tool/tool_base/tool_base.joints.xacro (robot description, xacro)
@@ -4,36 +4,42 @@
   <xacro:include filename="$(find surgical_sim)/urdf/surgical_tool/templates/gazebo.joints.xacro"/>
   <xacro:macro name="create_tool_base_joints" params="parent_link xyz rpy">
-    <!-- joint 1 -->
+    <!-- joint 1: tool_yaw -->
+    <joint name="tool_pitch" type="revolute">
+      <parent link="${parent_link}"/>
+      <child link="tool_pitch_link"/>
+      <axis xyz="0 0 1"/>
+      <origin rpy="0 -${pi/2} ${pi}" xyz="0.0 0.0 0.0"/>
+      <limit lower="-1.5707" upper="1.5707" velocity="3" effort="1000"/>
+    </joint>
+    <!-- joint 2: tool_pitch -->
+    <joint name="tool_roll" type="revolute">
+      <parent link="tool_pitch_link"/>
+      <child link="tool_roll_link"/>
+      <axis xyz="0 0 1"/>
+      <origin rpy="-${pi/2} -${pi/2} 0" xyz="0 0 0"/>
+      <limit lower="-1.5707" upper="1.5707" velocity="3" effort="1000"/>
+    </joint>
+    <!-- joint : tool Roll -->
     <joint name="tool_yaw" type="revolute">
-      <parent link="${parent_link}"/>
+      <parent link="tool_roll_link"/>
       <child link="tool_yaw_link"/>
       <axis xyz="0 0 1"/>
-      <origin rpy="0 -1.5708 1.5708" xyz="0.0 0.0 0.0"/>
-      <limit lower="-1.5707" upper="1.5707" velocity=".4" effort="1000"/>
-    </joint>
-    <!-- joint 2: tool_pitch -->
-    <joint name="tool_pitch" type="revolute">
-      <parent link="tool_yaw_link"/>
-      <child link="tool_pitch_link"/>
-      <axis xyz="0 0 1"/>
-      <origin rpy="-1.5708 -1.5708 0" xyz="0 0 0"/>
-      <limit lower="-0.7854" upper="0.7854" velocity=".4" effort="1000"/>
+      <origin rpy="${pi/2} 0 0" xyz="0 0 0"/>
+      <limit lower="-${1.5*pi}" upper="${1.5*pi}" velocity="3" effort="1000"/>
     </joint>
     <!-- joint 3: insertion -->
     <joint name="tool_insertion" type="prismatic">
-      <parent link="tool_pitch_link"/>
+      <parent link="tool_yaw_link"/>
       <child link="tool_main_link"/>
       <axis xyz="0 0 1"/>
-      <origin rpy="1.5708 0 0" xyz="0 ${0.4318-0.041} 0"/>
-      <limit lower="0" upper="0.240" velocity=".4" effort="1000"/>
+      <origin rpy="0 0 0" xyz="0 0 -${0.4318-0.041}"/>
+      <limit lower="0" upper="0.240" velocity="3" effort="1000"/>
     </joint>
-    <!-- joint 4: tool Roll -->
-    <joint name="tool_roll" type="revolute">
+    <joint name="tool_wrist_fixed" type="fixed">
       <parent link="tool_main_link"/>
       <child link="tool_wrist_link"/>
       <axis xyz="0 0 1"/>
       <origin rpy="0 0 0" xyz="0 0 ${0.4162-0.041}"/>
-      <limit lower="-2.2689" upper="2.2689" velocity=".4" effort="1000"/>
-    </joint>
+    </joint> -->
     <!-- joint 4-1: tool roll shaft joint FIXED-->
     <joint name="wrist_fixed" type="fixed">
@@ -43,11 +49,11 @@
       <origin rpy="0 0 0" xyz="0 0 0.0"/>
     </joint>
-    <xacro:joint_trans name="tool_yaw" reduction="1"/>
     <xacro:joint_trans name="tool_pitch" reduction="1"/>
     <xacro:joint_trans name="tool_roll" reduction="1"/>
+    <xacro:joint_trans name="tool_yaw" reduction="1"/>
     <xacro:joint_trans name="tool_insertion" reduction="1"/>
-    <xacro:gazebo_joints name="tool_yaw"/>
     <xacro:gazebo_joints name="tool_pitch"/>
     <xacro:gazebo_joints name="tool_roll"/>
+    <xacro:gazebo_joints name="tool_yaw"/>
     <xacro:gazebo_joints name="tool_insertion"/>
   </xacro:macro>

File: surgical_sim/urdf/surgical_tool/tool_base/tool_base.links.xacro (robot description, xacro)
@@ -13,4 +13,11 @@
     <!-- link 2: tool_pitch_link -->
     <link name="tool_pitch_link">
+      <inertial>
+				<origin xyz="0 0 0" rpy="0 0 0"/>
+				<mass value="0.05"/>
+				<inertia ixx="0.01" ixy="0.0" ixz="0.0" iyy="0.01" iyz="0.0" izz="0.005"/>
+			</inertial>
+    </link>
+    <link name="tool_roll_link">
       <inertial>
 				<origin xyz="0 0 0" rpy="0 0 0"/>

File: surgical_sim/urdf/surgical_tool/tool_create.urdf.xacro (robot description, xacro)
@@ -36,5 +36,5 @@
     <gazebo>
         <plugin name="gazebo_ros_control" filename="libgazebo_ros_control.so">
-        <robotNamespace>/surgical_tool</robotNamespace>
+        <robotNamespace></robotNamespace>
         <robotSimType>gazebo_ros_control/DefaultRobotHWSim</robotSimType>
         <legacyModeNS>true</legacyModeNS>

File: surgical_sim/urdf/surgical_tool/tool_forceps/tool_t_forceps.joints.xacro (robot description, xacro)
@@ -11,5 +11,5 @@
       <axis xyz="0 0 1"/>
       <origin rpy="-1.5708 -1.5708 ${pi}" xyz="0 0 0"/>
-      <limit lower="-1.5707" upper="1.5707" velocity=".4" effort="1000"/>
+      <limit lower="-${pi/2}" upper="${pi/2}" velocity=".4" effort="1000"/>
     </joint>
     <!-- joint 6: Tool wrist yaw joint -->
@@ -19,5 +19,5 @@
       <axis xyz="0 0 1"/>
       <origin rpy="0.00 -1.5708 -1.5708" xyz="0.0091 0 0"/>
-      <limit lower="-1.5707" upper="1.5707" velocity=".4" effort="1000"/>
+      <limit lower="-${pi/2}" upper="${pi/2}" velocity=".4" effort="1000"/>
     </joint>
     <!-- joint 6-1: tool open angle 1 -->
@@ -27,5 +27,5 @@
       <axis xyz="0 0 1"/>
       <origin rpy="0 0 0" xyz="0 0 0"/>
-      <limit lower="0" upper="1.5707" velocity=".4" effort="1000"/>
+      <limit lower="0" upper="${pi/2}" velocity=".4" effort="1000"/>
     </joint>
   <!-- joint 6-2: tool open angle 2  -->
@@ -35,5 +35,5 @@
       <axis xyz="0 0 1"/>
       <origin rpy="3.1415926 0 0" xyz="0 0 0"/>
-      <limit lower="0" upper="1.5707" velocity=".4" effort="1000"/>
+      <limit lower="0" upper="${pi/4}" velocity=".4" effort="1000"/>
       <mimic joint="tool_wrist_open_angle" multiplier="1"/>
     </joint>

File: surgical_sim/urdf/target_object/base_object/base_object.joints.xacro (robot description, xacro)
@@ -15,5 +15,4 @@
       <child link="target_object_link"/>
       <axis xyz="0.0 0.0 1.0"/>
-      <!-- <limit effort="0" velocity="0.0" lower="${-0.4}" upper="${0.4}"/> -->
     </joint>
     <xacro:joint_trans name="base_object_joint" reduction="1"/>

File: surgical_sim/urdf/target_object/base_object/base_object.links.xacro (robot description, xacro)
@@ -9,13 +9,12 @@
         <origin rpy="${-pi/2} 0 0" xyz="0 0 0"/>
         <geometry>
-          <!-- <mesh filename="package://surgical_sim/model/meshes/dae/target_object/torso.dae"/>       -->
-          <box size="0.050 0.050 0.050"/>
+          <sphere radius="0.007"/>
         </geometry>
       </visual>
-      <!-- <inertial>
+      <inertial>
 				<origin xyz="0 0 0" rpy="0 0 0"/>
 				<mass value="1"/>
-				<inertia ixx="1" ixy="0.0" ixz="0.0" iyy="1" iyz="0.0" izz="1"/>
-			</inertial>  -->
+				<inertia ixx="${2/5 * 1 * 0.019 * 0.019 }" ixy="0.0" ixz="0.0" iyy="${2/5 * 1 * 0.019 * 0.019 }" iyz="0.0" izz="${2/5 * 1 * 0.019 * 0.019 }"/>
+			</inertial>
     </link>
    <xacro:gazebo_links name="base_object_link"/>

Commit message: add package for camera feedback

File: leg_as_robot/urdf/left/leg.links.xacro (robot description, xacro)
@@ -1,7 +1,7 @@
 <?xml version="1.0"?>
 <robot xmlns:xacro="http://www.ros.org/wiki/xacro">
-  <xacro:property name="thigh_mass" value="${14.47 * 90.0/165.0 * body_weight / 100}"/> <!-- [kg] -->
-  <xacro:property name="shin_mass" value="${4.57 * body_weight / 100}"/> <!-- [kg] -->
-  <xacro:property name="foot_mass" value="${1.33 * body_weight / 100}"/> <!--[kg] -->
+  <xacro:property name="thigh_mass" value="${10.5 * (1.0-32/56) * (1.0-32/56) * body_weight / 100}"/>
+  <xacro:property name="shin_mass" value="${4.75 * body_weight / 100}"/> <!-- [kg] -->
+  <xacro:property name="foot_mass" value="${1.43  * body_weight / 100}"/> <!--[kg] -->
   <xacro:property name="scale_mass" value="${body_weight / body_weight_baseline}"/>
   <xacro:property name="thigh_scale_x" value="${thigh_d/thighBaseline_d}"/>

Commit message: latest updates

File: leg_as_robot/urdf/left/leg.links.xacro (robot description, xacro)
@@ -1,4 +1,5 @@
 <?xml version="1.0"?>
 <robot xmlns:xacro="http://www.ros.org/wiki/xacro">
+  <!-- <xacro:property name="thigh_mass" value="${10.5 * (1.0-32/56) * (1.0-32/56) * body_weight / 100}"/> -->
   <xacro:property name="thigh_mass" value="${10.5 * (1.0-32/56) * (1.0-32/56) * body_weight / 100}"/>
   <xacro:property name="shin_mass" value="${4.75 * body_weight / 100}"/> <!-- [kg] -->

File: leg_as_robot/urdf/right/leg.links.xacro (robot description, xacro)
@@ -2,12 +2,7 @@
 <robot xmlns:xacro="http://www.ros.org/wiki/xacro">
   <xacro:arg name="with_chair" default="true"/>
-  <!-- <xacro:property name="thigh_mass" value="${10.5 * 0.125 * body_weight / 100}"/>  -->
-  <!-- <xacro:property name="thigh_mass" value="${14.47 * 28/60 * body_weight / 100}"/> P01 -->
-  <!--xacro:property name="thigh_mass" value="${10.5 * (1.0-13/43) * (1.0-13/43) * body_weight / 100}"/--> <!--P02 -->
-  <!-- <xacro:property name="thigh_mass" value="${10.5 * (1.0-20/54) * (1.0-20/54) * body_weight / 100}"/> -->
-  <!-- <xacro:property name="thigh_mass" value="${10.5 * (1.0-26/59) * (1.0-26/59) * body_weight / 100}"/> -->
   <xacro:property name="thigh_mass" value="${10.5 * (1.0-32/56) * (1.0-32/56) * body_weight / 100}"/>
-  <xacro:property name="shin_mass" value="${4.75 * body_weight / 100}"/> <!-- [kg] -->
-  <xacro:property name="foot_mass" value="${1.43  * body_weight / 100}"/> <!--[kg] -->
+  <xacro:property name="shin_mass" value="${4.75 * body_weight / 100}"/>
+  <xacro:property name="foot_mass" value="${1.43  * body_weight / 100}"/>
   <xacro:property name="scale_mass" value="${body_weight / body_weight_baseline}"/>
   <xacro:property name="thigh_scale_x" value="${thigh_d/thighBaseline_d}"/>
