Commit message: latest stable version

File: leg_as_robot/urdf/chair/chair.joints.xacro (robot description, xacro)
@@ -4,12 +4,12 @@
     <joint name="chair_x_joint" type="prismatic">
       <origin xyz="0 0 0.0" rpy="0 0 0"/>
-      <parent link="/world"/>
-      <child link="chair_intermediate_link"/>
+      <parent link="chair_intermediate_link1"/>
+      <child link="chair_intermediate_link2"/>
       <axis xyz="1.0 0.0 0.0"/>
       <limit effort="0" velocity="0.0" lower="${-0.4}" upper="${0.4}"/>
     </joint>
     <joint name="chair_y_joint" type="prismatic">
-      <origin xyz="0 0 0.9246" rpy="0 0 0"/>
-      <parent link="chair_intermediate_link"/>
+      <origin xyz="0 0 ${hip_height}" rpy="0 0 0"/>
+      <parent link="chair_intermediate_link2"/>
       <child link="chair_base_link"/>
       <axis xyz="0.0 1.0 0.0"/>

File: leg_as_robot/urdf/chair/chair.links.xacro (robot description, xacro)
@@ -5,6 +5,6 @@
   <xacro:property name="base_scale_z" value="${hip_height/hip_heightBaseline}"/>
   <xacro:macro name="define_chair_link">
-    <link name="/world"/>
-    <link name="chair_intermediate_link"/>
+    <link name="chair_intermediate_link1"/>
+    <link name="chair_intermediate_link2"/>
     <link name="chair_base_link">
         <visual>

File: leg_as_robot/urdf/left/leg.joints.xacro (robot description, xacro)
@@ -44,9 +44,16 @@
       <axis xyz="0 0 1"/>
     </joint>
+    <!-- <joint name="ankle_yaw" type="revolute">
+      <origin xyz="0 0 0" rpy="${-pi/2} 0 ${-pi/2}"/>
+      <parent link="ankle_roll_link"/>
+      <child link="ankle_yaw_link"/>
+      <limit effort="30" velocity="10.0" lower="${radians(-36)}" upper="${radians(25.9)}"/>
+      <axis xyz="0 0 1"/>
+    </joint> -->
     <joint name="ankle_yaw" type="revolute">
       <origin xyz="0 0 0" rpy="${-pi/2} 0 ${-pi/2}"/>
       <parent link="ankle_roll_link"/>
       <child link="ankle_yaw_link"/>
-      <limit effort="30" velocity="10.0" lower="${radians(-36)}" upper="${radians(25.9)}"/>
+      <limit effort="30" velocity="10.0" lower="${radians(-10)}" upper="${radians(5)}"/>
       <axis xyz="0 0 1"/>
     </joint>

File: leg_as_robot/urdf/left/leg.links.xacro (robot description, xacro)
@@ -2,6 +2,6 @@
 <robot xmlns:xacro="http://www.ros.org/wiki/xacro">
   <xacro:property name="thigh_mass" value="${14.47 * 100.0/165.0 * body_weight / 100}"/> <!-- [kg] -->
-  <xacro:property name="shin_mass" value="${4.57 * 100.0/165.0 * body_weight / 100}"/> <!-- [kg] -->
-  <xacro:property name="foot_mass" value="${1.33 * 100.0/165.0 *body_weight / 100}"/> <!--[kg] -->
+  <xacro:property name="shin_mass" value="${4.57 * body_weight / 100}"/> <!-- [kg] -->
+  <xacro:property name="foot_mass" value="${1.33 * body_weight / 100}"/> <!--[kg] -->
   <xacro:property name="scale_mass" value="${body_weight / body_weight_baseline}"/>
   <xacro:property name="thigh_scale_x" value="${thigh_d/thighBaseline_d}"/>
@@ -12,5 +12,5 @@
   <xacro:property name="shin_scale_z" value="${shin_w/shinBaseline_w}"/>
   <xacro:property name="foot_scale_x" value="${foot_l/footBaseline_l}"/>
-  <xacro:property name="foot_scale_y" value="${r7_leg/r7Baseline_leg}"/>
+  <xacro:property name="foot_scale_y" value="${r8_leg/r8Baseline_leg}"/>
   <xacro:property name="foot_scale_z" value="${d7_leg/d7Baseline_leg}"/>
   <xacro:macro name="define_leg_links">

File: leg_as_robot/urdf/right/leg.joints.xacro (robot description, xacro)
@@ -6,5 +6,5 @@
       <parent link="hip_base_link"/>
       <child link="hip_adduction_link"/>
-      <limit effort="30" velocity="10.0" lower="${radians(-44)}" upper="${radians(0)}"/>
+      <limit effort="30" velocity="10.0" lower="${radians(-44)}" upper="${radians(30)}"/>
       <axis xyz="0 0 1"/>
     </joint>
@@ -20,5 +20,5 @@
       <parent link="hip_extension_link"/>
       <child link="hip_roll_link"/>
-      <limit effort="30" velocity="10.0" lower="${radians(-33)}" upper="${radians(33)}"/>
+      <limit effort="30" velocity="10.0" lower="${radians(-45)}" upper="${radians(45)}"/>
       <axis xyz="0 0 1"/>
     </joint>
@@ -51,4 +51,11 @@
       <axis xyz="0 0 1"/>
     </joint>
+     <!-- <joint name="ankle_yaw" type="revolute">
+      <origin xyz="0 0 0" rpy="${-pi/2} 0 ${-pi/2}"/>
+      <parent link="ankle_roll_link"/>
+      <child link="ankle_yaw_link"/>
+      <limit effort="30" velocity="10.0" lower="${radians(-5)}" upper="${radians(10)}"/>
+      <axis xyz="0 0 1"/>
+    </joint> -->
       <joint name="fixed_foot_base" type="fixed">
           <origin xyz="0 ${-r7_leg} ${-d7_leg}" rpy="0 0 ${-pi/2}"/>

File: leg_as_robot/urdf/right/leg.links.xacro (robot description, xacro)
@@ -3,5 +3,5 @@
   <xacro:arg name="with_chair" default="true"/>
   <xacro:property name="thigh_mass" value="${14.47 * 100.0/165.0 * body_weight / 100}"/> <!-- [kg] -->
-  <xacro:property name="shin_mass" value="${4.57 * 100.0/165.0  * body_weight / 100}"/> <!-- [kg] -->
+  <xacro:property name="shin_mass" value="${4.57 * body_weight / 100}"/> <!-- [kg] -->
   <xacro:property name="foot_mass" value="${1.33 * 100.0/165.0  *body_weight / 100}"/> <!--[kg] -->
   <xacro:property name="scale_mass" value="${body_weight / body_weight_baseline}"/>
@@ -13,5 +13,5 @@
   <xacro:property name="shin_scale_z" value="${shin_w/shinBaseline_w}"/>
   <xacro:property name="foot_scale_x" value="${foot_l/footBaseline_l}"/>
-  <xacro:property name="foot_scale_y" value="${r7_leg/r7Baseline_leg}"/>
+  <xacro:property name="foot_scale_y" value="${r8_leg/r8Baseline_leg}"/>
   <xacro:property name="foot_scale_z" value="${d7_leg/d7Baseline_leg}"/>
   <xacro:macro name="define_leg_links">
