Commit message: latest changes to the protocol, add visual feedback to positioning and then grasping

File: surgical_sim/urdf/surgical_tool/tool_base/tool_base.joints.xacro (robot description, xacro)
@@ -34,5 +34,5 @@
       <axis xyz="0 0 1"/>
       <origin rpy="0 0 0" xyz="0 0 -${0.4318-0.041}"/>
-      <limit lower="0" upper="0.240" velocity="3" effort="1000"/>
+      <limit lower="0.0" upper="0.240" velocity="3" effort="1000"/>
     </joint>
     <joint name="tool_wrist_fixed" type="fixed">
