Commit message: backup 16-09

File: leg_as_robot/urdf/right/leg.links.xacro (robot description, xacro)
@@ -2,7 +2,9 @@
 <robot xmlns:xacro="http://www.ros.org/wiki/xacro">
   <xacro:arg name="with_chair" default="true"/>
-  <xacro:property name="thigh_mass" value="${14.47 * 100.0/165.0 * body_weight / 100}"/> <!-- [kg] -->
-  <xacro:property name="shin_mass" value="${4.57 * body_weight / 100}"/> <!-- [kg] -->
-  <xacro:property name="foot_mass" value="${1.33 * body_weight / 100}"/> <!--[kg] -->
+  <!-- <xacro:property name="thigh_mass" value="${10.5 * 0.125 * body_weight / 100}"/>  -->
+  <!-- <xacro:property name="thigh_mass" value="${14.47 * 28/60 * body_weight / 100}"/> P01 -->
+  <xacro:property name="thigh_mass" value="${10.5 * 0.25 * body_weight / 100}"/> <!--P02 -->
+  <xacro:property name="shin_mass" value="${4.75 * body_weight / 100}"/> <!-- [kg] -->
+  <xacro:property name="foot_mass" value="${1.43  * body_weight / 100}"/> <!--[kg] -->
   <xacro:property name="scale_mass" value="${body_weight / body_weight_baseline}"/>
   <xacro:property name="thigh_scale_x" value="${thigh_d/thighBaseline_d}"/>

File: surgical_sim/urdf/body/body_create.urdf.xacro (robot description, xacro)
@@ -16,9 +16,9 @@
     <xacro:attach_liver
         parent_link="world"
-        xyz="0.0 0.5 1.1" rpy="0.0 0.0 ${-pi/2}" />
+        xyz="0.0 0.5 1.1" rpy="0.0 0.0 0" />
   </xacro:if>
   <xacro:unless value="$(arg with_liver)">
   </xacro:unless>
-    <gazebo>
+    <!-- <gazebo>
         <plugin name="gazebo_ros_control" filename="libgazebo_ros_control.so">
         <robotNamespace>/body</robotNamespace>
@@ -26,4 +26,4 @@
         <legacyModeNS>true</legacyModeNS>
         </plugin>
-    </gazebo>
+    </gazebo> -->
 </robot>

File: surgical_sim/urdf/body/templates/gazebo.joints.xacro (robot description, xacro)
@@ -3,9 +3,6 @@
 	<xacro:macro name="gazebo_joints" params="name">
 		<gazebo reference="${name}">
-			<implicitSpringDamper>0</implicitSpringDamper>
-			<provideFeedback>1</provideFeedback>
-			<stopCfm></stopCfm> <!-- Force Mixing Error -->
-			<stopErp></stopErp> <!-- Error Reduction Parameter -->
-			<fudgeFactor>0.5</fudgeFactor>
+			<!-- <implicitSpringDamper>0</implicitSpringDamper>
+			<provideFeedback>1</provideFeedback> -->
 		</gazebo>
 	</xacro:macro>

File: surgical_sim/urdf/body/torso/torso.joints.xacro (robot description, xacro)
@@ -10,5 +10,4 @@
       <axis xyz="0 0 1"/>
       <origin rpy="${rpy}" xyz="${xyz}"/>
-      <!-- <limit lower="-1.5707" upper="1.5707" velocity=".4" effort="1000"/> -->
     </joint>
     <joint name="right_trocar_joint" type="fixed">
@@ -17,5 +16,4 @@
       <axis xyz="0 0 1"/>
       <origin rpy="0 0 ${pi/2}" xyz="0.015 0.015 0.2"/>
-      <!-- <limit lower="-1.5707" upper="1.5707" velocity=".4" effort="1000"/> -->
     </joint>
     <joint name="left_trocar_joint" type="fixed">
@@ -24,7 +22,5 @@
       <axis xyz="0 0 1"/>
       <origin rpy="0 0 ${pi/2}" xyz="0.0 0.0 0.2"/>
-      <!-- <limit lower="-1.5707" upper="1.5707" velocity=".4" effort="1000"/> -->
     </joint>
-    <!-- <xacro:joint_trans name="torso_joint" reduction="1"/> -->
     <xacro:gazebo_joints name="torso_joint"/>
   </xacro:macro>

File: surgical_sim/urdf/body/torso/torso.links.xacro (robot description, xacro)
@@ -11,4 +11,10 @@
         </geometry>
       </visual>
+      <collision>
+        <origin rpy="${-pi/2} 0 0" xyz="0 0 0"/>
+        <geometry>
+          <mesh filename="package://surgical_sim/model/meshes/stl/body/torso_simp.stl"/>
+        </geometry>
+      </collision>
       <inertial>
 				<origin xyz="0 0 0" rpy="0 0 0"/>

File: surgical_sim/urdf/surgical_tool/templates/gazebo.joints.xacro (robot description, xacro)
@@ -3,9 +3,6 @@
 	<xacro:macro name="gazebo_joints" params="name">
 		<gazebo reference="${name}">
-			<implicitSpringDamper>0</implicitSpringDamper>
-			<provideFeedback>1</provideFeedback>
-			<stopCfm></stopCfm>
-			<stopErp></stopErp>
-			<fudgeFactor>0.5</fudgeFactor>
+			<!-- <implicitSpringDamper>0</implicitSpringDamper>
+			<provideFeedback>1</provideFeedback> -->
 		</gazebo>
 	</xacro:macro>

File: surgical_sim/urdf/surgical_tool/tool_base/tool_base.joints.xacro (robot description, xacro)
@@ -41,7 +41,7 @@
       <axis xyz="0 0 1"/>
       <origin rpy="0 0 0" xyz="0 0 ${0.4162-0.041}"/>
-    </joint> -->
+    </joint>
     <!-- joint 4-1: tool roll shaft joint FIXED-->
-    <joint name="wrist_fixed" type="fixed">
+    <joint name="tool_wrist_shaft_fixed" type="fixed">
       <parent link="tool_wrist_link"/>
       <child link="tool_wrist_shaft_link"/>
@@ -57,4 +57,6 @@
     <xacro:gazebo_joints name="tool_yaw"/>
     <xacro:gazebo_joints name="tool_insertion"/>
+    <!-- <xacro:gazebo_joints name="tool_wrist_fixed"/>
+    <xacro:gazebo_joints name="tool_wrist_shaft_fixed"/>  -->
   </xacro:macro>
 </robot>

File: surgical_sim/urdf/surgical_tool/tool_base/tool_base.links.xacro (robot description, xacro)
@@ -34,4 +34,10 @@
         </geometry>
       </visual>
+       <collision>
+        <origin rpy="0 0 1.5708" xyz="0 0 0"/>
+        <geometry>
+          <mesh filename="package://surgical_sim/model/meshes/dae/tool/tool_main_.dae"/>
+        </geometry>
+      </collision>
       <inertial>
 				<origin xyz="0 0 0" rpy="0 0 0"/>
@@ -48,4 +54,10 @@
         </geometry>
       </visual>
+      <collision>
+        <origin rpy="0 0 1.5708" xyz="0 0 -0.0091"/>
+        <geometry>
+          <mesh filename="package://surgical_sim/model/meshes/dae/tool/tool_wrist_link.dae"/>
+        </geometry>
+      </collision>
       <inertial>
 				<origin xyz="0 0 0" rpy="0 0 0"/>
@@ -62,4 +74,10 @@
         </geometry>
       </visual>
+      <collision>
+        <origin rpy="1.5708 0 0" xyz="0 0.00401 0"/>
+        <geometry>
+          <mesh filename="package://surgical_sim/model/meshes/dae/tool/tool_wrist_shaft_link.dae"/>
+        </geometry>
+      </collision>
       <inertial>
 				<origin xyz="0 0 0" rpy="0 0 0"/>
@@ -70,7 +88,8 @@
     <xacro:gazebo_links name="tool_yaw_link"/>
     <xacro:gazebo_links name="tool_pitch_link"/>
+    <xacro:gazebo_links name="tool_roll_link"/>
     <xacro:gazebo_links name="tool_main_link"/>
     <xacro:gazebo_links name="tool_wrist_link"/>
-    <xacro:gazebo_links name="tool_shaft_link"/>
+    <xacro:gazebo_links name="tool_wrist_shaft_link"/>
   </xacro:macro>
 </robot>

File: surgical_sim/urdf/surgical_tool/tool_create.urdf.xacro (robot description, xacro)
@@ -8,4 +8,5 @@
   <xacro:arg name="with_forceps" default="true"/>
   <xacro:arg name="with_gripper" default="false"/>
+  <xacro:arg name="toolID" default="right"/>
   <xacro:macro name="attach_gripper" params="parent_link xyz rpy">
     <xacro:create_tool_base
@@ -21,5 +22,12 @@
   </xacro:macro>
  <!--  -->
-  <link name="tool_base_link"/>
+  <link name="/world"/>
+  <link name="tool_base_link">
+    <inertial>
+      <origin xyz="0.0 0.0 0.0" rpy="0.0 0.0 0.0"/>
+      <mass value="0.001"/>
+      <inertia ixx="0.001" ixy="0.0" ixz="0.0" iyy="0.0001" iyz="0.0" izz="0.0001"/>
+    </inertial>
+  </link>
   <xacro:if value="$(arg with_forceps)">
     <xacro:attach_forceps
@@ -34,7 +42,13 @@
     </xacro:if>
   </xacro:unless>
+  <joint name="world_fixed" type="fixed">
+      <parent link="/world"/>
+      <child link="tool_base_link"/>
+      <origin rpy="0 0 0" xyz="${0+0.015} ${0.5 + 0.015} ${1.1 + 0.2} "/>
+  </joint>
     <gazebo>
         <plugin name="gazebo_ros_control" filename="libgazebo_ros_control.so">
-        <robotNamespace></robotNamespace>
+        <robotNamespace>surgical_tool</robotNamespace>
+        <robotParam>/$(arg toolID)/tool_description</robotParam>
         <robotSimType>gazebo_ros_control/DefaultRobotHWSim</robotSimType>
         <legacyModeNS>true</legacyModeNS>

File: surgical_sim/urdf/surgical_tool/tool_forceps/tool_t_forceps.joints.xacro (robot description, xacro)
@@ -27,5 +27,5 @@
       <axis xyz="0 0 1"/>
       <origin rpy="0 0 0" xyz="0 0 0"/>
-      <limit lower="0" upper="${pi/2}" velocity=".4" effort="1000"/>
+      <limit lower="0" upper="${30*pi/180}" velocity=".4" effort="1000"/>
     </joint>
   <!-- joint 6-2: tool open angle 2  -->
@@ -35,5 +35,5 @@
       <axis xyz="0 0 1"/>
       <origin rpy="3.1415926 0 0" xyz="0 0 0"/>
-      <limit lower="0" upper="${pi/4}" velocity=".4" effort="1000"/>
+      <limit lower="0" upper="${30*pi/180}" velocity=".4" effort="1000"/>
       <mimic joint="tool_wrist_open_angle" multiplier="1"/>
     </joint>
@@ -57,4 +57,6 @@
     <xacro:gazebo_joints name="tool_wrist_open_angle"/>
     <xacro:gazebo_joints name="tool_wrist_open_angle_mimic"/>
+    <!-- <xacro:gazebo_joints name="tool_tip_"/>
+    <xacro:gazebo_joints name="tool_tip_ee"/> -->
   </xacro:macro>
 </robot>

File: surgical_sim/urdf/surgical_tool/tool_forceps/tool_t_forceps.links.xacro (robot description, xacro)
@@ -91,6 +91,4 @@
     <xacro:gazebo_links name="tool_wrist_forceps_link_2_left"/>
     <xacro:gazebo_links name="tool_wrist_forceps_link_2_right"/>
-    <xacro:gazebo_links name="tool_wrist_link"/>
-    <xacro:gazebo_links name="tool_shaft_link"/>
   </xacro:macro>
 </robot>

File: surgical_sim/urdf/target_object/base_object/base_object.links.xacro (robot description, xacro)
@@ -11,4 +11,7 @@
           <sphere radius="0.007"/>
         </geometry>
+      <material name="Cyan">
+       <color rgba="0 1.0 1.0 0.5"/>
+     </material>
       </visual>
       <inertial>

Commit message: separate targets and shared control

File: leg_as_robot/urdf/right/leg.links.xacro (robot description, xacro)
@@ -4,5 +4,8 @@
   <!-- <xacro:property name="thigh_mass" value="${10.5 * 0.125 * body_weight / 100}"/>  -->
   <!-- <xacro:property name="thigh_mass" value="${14.47 * 28/60 * body_weight / 100}"/> P01 -->
-  <xacro:property name="thigh_mass" value="${10.5 * 0.25 * body_weight / 100}"/> <!--P02 -->
+  <!--xacro:property name="thigh_mass" value="${10.5 * (1.0-13/43) * (1.0-13/43) * body_weight / 100}"/--> <!--P02 -->
+  <!-- <xacro:property name="thigh_mass" value="${10.5 * (1.0-20/54) * (1.0-20/54) * body_weight / 100}"/> -->
+  <!-- <xacro:property name="thigh_mass" value="${10.5 * (1.0-26/59) * (1.0-26/59) * body_weight / 100}"/> -->
+  <xacro:property name="thigh_mass" value="${10.5 * (1.0-32/56) * (1.0-32/56) * body_weight / 100}"/>
   <xacro:property name="shin_mass" value="${4.75 * body_weight / 100}"/> <!-- [kg] -->
   <xacro:property name="foot_mass" value="${1.43  * body_weight / 100}"/> <!--[kg] -->

File: surgical_sim/urdf/surgical_tool/tool_forceps/tool_t_forceps.joints.xacro (robot description, xacro)
@@ -11,5 +11,5 @@
       <axis xyz="0 0 1"/>
       <origin rpy="-1.5708 -1.5708 ${pi}" xyz="0 0 0"/>
-      <limit lower="-${pi/2}" upper="${pi/2}" velocity=".4" effort="1000"/>
+      <limit lower="-${pi/2}" upper="${pi/2}" velocity="3.0" effort="1000"/>
     </joint>
     <!-- joint 6: Tool wrist yaw joint -->
@@ -19,5 +19,5 @@
       <axis xyz="0 0 1"/>
       <origin rpy="0.00 -1.5708 -1.5708" xyz="0.0091 0 0"/>
-      <limit lower="-${pi/2}" upper="${pi/2}" velocity=".4" effort="1000"/>
+      <limit lower="-${pi/2}" upper="${pi/2}" velocity="3.0" effort="1000"/>
     </joint>
     <!-- joint 6-1: tool open angle 1 -->
@@ -27,5 +27,5 @@
       <axis xyz="0 0 1"/>
       <origin rpy="0 0 0" xyz="0 0 0"/>
-      <limit lower="0" upper="${30*pi/180}" velocity=".4" effort="1000"/>
+      <limit lower="0" upper="${radians(30)}" velocity="3.0" effort="1000"/>
     </joint>
   <!-- joint 6-2: tool open angle 2  -->
@@ -35,5 +35,5 @@
       <axis xyz="0 0 1"/>
       <origin rpy="3.1415926 0 0" xyz="0 0 0"/>
-      <limit lower="0" upper="${30*pi/180}" velocity=".4" effort="1000"/>
+      <limit lower="0" upper="${radians(30)}" velocity="3.0" effort="1000"/>
       <mimic joint="tool_wrist_open_angle" multiplier="1"/>
     </joint>
