Commit message: [surgical_task]: Add last changes

File: surgical_task/models/environment.urdf.xacro (robot description, xacro)
@@ -18,5 +18,11 @@
   <xacro:property name="pillarsYdim" value="0.12"/>
   <xacro:property name="pillarsZdim" value="0.032"/>
-  <link name="world"/>
+  <link name="world">
+      <inertial>
+        <origin xyz="0 0 0" rpy="0 0 0"/>
+        <mass value="1e-6"/>
+        <inertia ixx="1e-6" ixy="0" ixz="0" iyy="1e-6" iyz="0" izz="1e-6"/>
+      </inertial>
+  </link>
   <gazebo reference="world">
 <!--     <static>true</static>

File: surgical_task/models/panda_arm.urdf.xacro (robot description, xacro)
@@ -1,4 +1,6 @@
-<?xml version="1.0"?>
-<robot xmlns:xacro="http://www.ros.org/wiki/xacro" name="lwr_with_tool">
+<?xml version='1.0' encoding='utf-8'?>
+<robot xmlns:xacro="http://www.ros.org/wiki/xacro" name="panda">
+	<xacro:arg name="gazebo" default="true"/>
+	<xacro:arg name="robotName" default="panda"/>
   <xacro:arg name="origin.x" default="0"/>
   <xacro:arg name="origin.y" default="0"/>
@@ -7,32 +9,20 @@
   <xacro:arg name="origin.ay" default="0"/>
   <xacro:arg name="origin.az" default="0"/>
-  <xacro:arg name="robotName" default="lwr"/>
   <xacro:arg name="addFrame" default="0"/>
-  <xacro:arg name="addCamera" default="0"/>
+  <xacro:arg name="addCamera" default="1"/>
   <xacro:arg name="useInstrument" default="0"/>
   <xacro:property name="toolMass" value="0.1"/>
-  <xacro:property name="toolLength" value="0.40"/>
+  <xacro:property name="toolLength" value="0.4"/>
   <xacro:property name="toolRadius" value="0.005"/>
-  <xacro:property name="tableLength" value="0.3"/>
-  <xacro:property name="tableWidth" value="0.3"/>
-  <xacro:property name="tableHeight" value="0.8"/>
-  <link name="world">
-      <inertial>
-        <origin xyz="0 0 0" rpy="0 0 0"/>
-        <mass value="1e-6"/>
-        <inertia ixx="1e-6" ixy="0" ixz="0" iyy="1e-6" iyz="0" izz="1e-6"/>
-      </inertial>
-  </link>
+  <xacro:property name="M_PI" value="3.14159265359" />
   <gazebo reference="world">
 <!--     <static>true</static>
     <turnGravityOff>true</turnGravityOff> -->
   </gazebo>
-  <!-- Include all models -->
-  <xacro:include filename="$(find surgical_simulator)/models/kuka_lwr.urdf.xacro"/>
-  <xacro:kuka_lwr base_link="world" name="$(arg robotName)">
-    <!-- <origin xyz="$(arg origin.x) $(arg origin.y) $(arg origin.z)" rpy="0 0 0"/> -->
-    <origin xyz="$(arg origin.x) $(arg origin.y) $(arg origin.z)" rpy="$(arg origin.ax) $(arg origin.ay) $(arg origin.az)"/>
-  </xacro:kuka_lwr>
-  <xacro:if value="${$(arg useInstrument)==0}">
+  <xacro:include filename="$(find surgical_task)/models/panda_arm.xacro" >
+  	<xacro:arg name="gazebo" value="${gazebo}"/>
+  </xacro:include>
+  <xacro:panda_arm connected_to='world' arm_id="$(arg robotName)" xyz='$(arg origin.x) $(arg origin.y) $(arg origin.z)' rpy='$(arg origin.ax) $(arg origin.ay) $(arg origin.az)'/>
+ <xacro:if value="${$(arg useInstrument)==0}">
     <link name='$(arg robotName)_tool'>
       <inertial>
@@ -56,5 +46,5 @@
     <joint name="$(arg robotName)_tool_joint" type="fixed">
       <origin xyz="0 0 0" rpy="0 0 0"/>
-      <parent link="$(arg robotName)_7_link"/>
+      <parent link="$(arg robotName)_link8"/>
       <child link="$(arg robotName)_tool"/>
     </joint>
@@ -64,5 +54,5 @@
     <joint name="instrument_base_joint" type="fixed">
       <origin xyz="0 0 0" rpy="0 0 0"/>
-      <parent link="$(arg robotName)_7_link"/>
+      <parent link="$(arg robotName)_link8"/>
       <child link="$(arg robotName)_instrument"/>
     </joint>
@@ -149,46 +139,3 @@
   </gazebo>
 </xacro:if>
-<!-- <xacro:if value="${$(arg addCamera)==0}"> -->
-<!--   <link name="ft_sensor_link">
-    <inertial>
-      <mass value="0.001" />
-      <origin xyz="0 0 0" />
-      <inertia ixx="0.0001" ixy="0.0" ixz="0.0" iyy="0.0001" iyz="0.0" izz="0.0001" />
-    </inertial>
-  </link>
-  <joint name="ft_sensor_joint" type="fixed">
-        <parent link="$(arg robotName)_tool"/>
-        <child link="ft_sensor_link"/>
-        <origin xyz="0 0 ${toolLength}" rpy="0 0 0"/>
-        <limit effort="400" velocity="0" lower="0" upper="0" />
-  </joint> -->
-<!--   <joint name="ft_sensor_joint" type="prismatic">
-      <origin xyz="0 0 ${toolLength}" rpy="0 0 0"/>
-      <parent link="$(arg robotName)_tool"/>
-      <child link="ft_sensor_link"/>
-      <limit effort="200" velocity="0" lower="0" upper="0"/>
-      <axis xyz="0 0 1"/>
-  </joint> -->
-<!--
-  <joint name="ft_sensor_joint" type="revolute">
-      <origin xyz="0 0 ${toolLength}" rpy="0 0 0"/>
-      <parent link="$(arg robotName)_tool"/>
-      <child link="ft_sensor_link"/>
-    <axis xyz="0 0 1"/>
-    <limit lower="0" upper="0" effort="0.0" velocity="0.0"/>
-</joint> -->
-<!--   <gazebo reference="$(arg robotName)_tool_joint">
-    <provideFeedback>true</provideFeedback>
-    <disableFixedJointLumping>true</disableFixedJointLumping>
-  </gazebo> -->
-<!--   <gazebo>
-    <plugin name="ft_sensor" filename="libgazebo_ros_ft_sensor.so">
-      <alwaysOn>true</alwaysOn>
-      <updateRate>200</updateRate>
-      <topicName>ft_sensor</topicName>
-      <jointName>$(arg robotName)_tool_joint</jointName>
-      <gaussianNoise>0.0001</gaussianNoise>
-    </plugin>
-  </gazebo> -->
-<!-- </xacro:if> -->
 </robot>
