Commit message: [surgical_task]: fix urdf file and launch files for compatibility issue to ros noetic

File: surgical_task/models/axis.urdf.xacro (robot description, xacro)
@@ -1,7 +1,7 @@
 <?xml version="1.0"?>
 <robot xmlns:xacro="http://www.ros.org/wiki/xacro" name="axis.urdf.xacro">
-  <xacro:arg name="origin.x" default="0"/>
-  <xacro:arg name="origin.y" default="0"/>
-  <xacro:arg name="origin.z" default="0"/>
+  <xacro:arg name="origin_x" default="0"/>
+  <xacro:arg name="origin_y" default="0"/>
+  <xacro:arg name="origin_z" default="0"/>
   <xacro:arg name="name" default="target"/>
   <!-- <link name="world"/> -->
@@ -42,8 +42,8 @@
     </visual>
   </link>
-    <gazebo>
+<!--     <gazebo>
     <plugin name="objectPosePublishing" filename="libobjectPosePublishing.so">
       <actorName>$(arg name)</actorName>
     </plugin>
-  </gazebo>
+  </gazebo> -->
 </robot>

File: surgical_task/models/environment.urdf.xacro (robot description, xacro)
@@ -1,7 +1,7 @@
 <?xml version="1.0"?>
 <robot xmlns:xacro="http://www.ros.org/wiki/xacro" name="surgical_environment.urdf.xacro">
-  <xacro:arg name="orgin.x" default="0"/>
-  <xacro:arg name="orgin.y" default="0"/>
-  <xacro:arg name="orgin.z" default="0"/>
+  <xacro:arg name="origin_x" default="0"/>
+  <xacro:arg name="origin_y" default="0"/>
+  <xacro:arg name="origin_z" default="0"/>
   <!-- Surgical frame dimensions after proper rotation -->
   <xacro:property name="surgicalFrameXdim" value="0.169996"/>
@@ -36,9 +36,9 @@
                     width="${tableYdim}" height="${tableZdim}" plate_thickness="0.05"
                     color="grey">
-    <origin xyz="${$(arg origin.x)-tableXdim/2} ${$(arg origin.y)+tableYdim/2} ${tableZdim}" rpy="0 0 0"/>
+    <origin xyz="${$(arg origin_x)-tableXdim/2} ${$(arg origin_y)+tableYdim/2} ${tableZdim}" rpy="0 0 0"/>
   </xacro:model_table>
  -->
   <xacro:surgical_frame name="surgical_frame" base_link="world">
-    <origin xyz="$(arg origin.x) $(arg origin.y) $(arg origin.z)" rpy="0 0 0"/>
+    <origin xyz="$(arg origin_x) $(arg origin_y) $(arg origin_z)" rpy="0 0 0"/>
   </xacro:surgical_frame>
   <xacro:pillars name="pillars" base_link="surgical_frame_base_link">

File: surgical_task/models/panda_arm.gazebo.xacro (robot description, xacro)
@@ -18,7 +18,7 @@
     <type>transmission_interface/SimpleTransmission</type>
     <joint name="${arm_id}_joint1">
-      <!-- <hardwareInterface>hardware_interface/PositionJointInterface</hardwareInterface> -->
-      <hardwareInterface>PositionJointInterface</hardwareInterface>
-    </joint>
+      <hardwareInterface>hardware_interface/PositionJointInterface</hardwareInterface>
+<!--       <hardwareInterface>PositionJointInterface</hardwareInterface>
+ -->    </joint>
     <actuator name="${arm_id}_joint1_motor">
       <mechanicalReduction>1</mechanicalReduction>
@@ -28,7 +28,7 @@
     <type>transmission_interface/SimpleTransmission</type>
     <joint name="${arm_id}_joint2">
-      <!-- <hardwareInterface>hardware_interface/PositionJointInterface</hardwareInterface> -->
-      <hardwareInterface>PositionJointInterface</hardwareInterface>
-    </joint>
+      <hardwareInterface>hardware_interface/PositionJointInterface</hardwareInterface>
+<!--       <hardwareInterface>PositionJointInterface</hardwareInterface>
+ -->    </joint>
     <actuator name="${arm_id}_joint2_motor">
       <mechanicalReduction>1</mechanicalReduction>
@@ -38,6 +38,7 @@
     <type>transmission_interface/SimpleTransmission</type>
     <joint name="${arm_id}_joint3">
-      <!-- <hardwareInterface>hardware_interface/PositionJointInterface</hardwareInterface> -->
-      <hardwareInterface>PositionJointInterface</hardwareInterface>
+      <hardwareInterface>hardware_interface/PositionJointInterface</hardwareInterface>
+<!--       <hardwareInterface>PositionJointInterface</hardwareInterface>
+ -->
     </joint>
     <actuator name="${arm_id}_joint3_motor">
@@ -48,7 +49,7 @@
     <type>transmission_interface/SimpleTransmission</type>
     <joint name="${arm_id}_joint4">
-      <!-- <hardwareInterface>hardware_interface/PositionJointInterface</hardwareInterface> -->
-      <hardwareInterface>PositionJointInterface</hardwareInterface>
-    </joint>
+      <hardwareInterface>hardware_interface/PositionJointInterface</hardwareInterface>
+<!--       <hardwareInterface>PositionJointInterface</hardwareInterface>
+ -->    </joint>
     <actuator name="${arm_id}_joint4_motor">
       <mechanicalReduction>1</mechanicalReduction>
@@ -58,7 +59,7 @@
     <type>transmission_interface/SimpleTransmission</type>
     <joint name="${arm_id}_joint5">
-      <!-- <hardwareInterface>hardware_interface/PositionJointInterface</hardwareInterface> -->
-      <hardwareInterface>PositionJointInterface</hardwareInterface>
-    </joint>
+      <hardwareInterface>hardware_interface/PositionJointInterface</hardwareInterface>
+<!--       <hardwareInterface>PositionJointInterface</hardwareInterface>
+ -->    </joint>
     <actuator name="${arm_id}_joint5_motor">
       <mechanicalReduction>1</mechanicalReduction>
@@ -68,7 +69,7 @@
     <type>transmission_interface/SimpleTransmission</type>
     <joint name="${arm_id}_joint6">
-      <!-- <hardwareInterface>hardware_interface/PositionJointInterface</hardwareInterface> -->
-      <hardwareInterface>PositionJointInterface</hardwareInterface>
-    </joint>
+      <hardwareInterface>hardware_interface/PositionJointInterface</hardwareInterface>
+<!--       <hardwareInterface>PositionJointInterface</hardwareInterface>
+ -->    </joint>
     <actuator name="${arm_id}_joint6_motor">
       <mechanicalReduction>1</mechanicalReduction>
@@ -78,7 +79,7 @@
     <type>transmission_interface/SimpleTransmission</type>
     <joint name="${arm_id}_joint7">
-      <!-- <hardwareInterface>hardware_interface/PositionJointInterface</hardwareInterface> -->
-      <hardwareInterface>PositionJointInterface</hardwareInterface>
-    </joint>
+      <hardwareInterface>hardware_interface/PositionJointInterface</hardwareInterface>
+<!--       <hardwareInterface>PositionJointInterface</hardwareInterface>
+ -->    </joint>
     <actuator name="${arm_id}_joint7_motor">
       <mechanicalReduction>1</mechanicalReduction>

File: surgical_task/models/panda_arm.urdf.xacro (robot description, xacro)
@@ -3,10 +3,10 @@
 	<xacro:arg name="gazebo" default="true"/>
 	<xacro:arg name="robotName" default="panda"/>
-  <xacro:arg name="origin.x" default="0"/>
-  <xacro:arg name="origin.y" default="0"/>
-  <xacro:arg name="origin.z" default="0"/>
-  <xacro:arg name="origin.ax" default="0"/>
-  <xacro:arg name="origin.ay" default="0"/>
-  <xacro:arg name="origin.az" default="0"/>
+  <xacro:arg name="origin_x" default="0"/>
+  <xacro:arg name="origin_y" default="0"/>
+  <xacro:arg name="origin_z" default="0"/>
+  <xacro:arg name="origin_ax" default="0"/>
+  <xacro:arg name="origin_ay" default="0"/>
+  <xacro:arg name="origin_az" default="0"/>
   <xacro:arg name="addFrame" default="0"/>
   <xacro:arg name="addCamera" default="1"/>
@@ -23,5 +23,5 @@
   	<xacro:arg name="gazebo" value="${gazebo}"/>
   </xacro:include>
-  <xacro:panda_arm connected_to='world' arm_id="$(arg robotName)" xyz='$(arg origin.x) $(arg origin.y) $(arg origin.z)' rpy='$(arg origin.ax) $(arg origin.ay) $(arg origin.az)'/>
+  <xacro:panda_arm connected_to='world' arm_id="$(arg robotName)" xyz='$(arg origin_x) $(arg origin_y) $(arg origin_z)' rpy='$(arg origin_ax) $(arg origin_ay) $(arg origin_az)'/>
  <xacro:if value="${$(arg useInstrument)==0}">
     <link name='$(arg robotName)_tool'>

File: surgical_task/models/surgical_frame.urdf.xacro (robot description, xacro)
@@ -10,6 +10,5 @@
     <!-- First (shoulder) element of the arm. Fixed to its parent. -->
     <joint name="${name}_base_joint" type="fixed">
-      <insert_block name="origin"/>
-      <origin xyz="0 0 0" rpy="0 0 0"/>
+      <xacro:insert_block name="origin"/>
       <parent link="${base_link}"/>
       <child link="${name}_base_link"/>
