Commit message: [surgical_task]: surgical task refactorization + tool tracking with camera

File: surgical_task/models/panda_arm.urdf.xacro (robot description, xacro)
@@ -114,6 +114,8 @@
         <image>
           <format>R8G8B8</format>
-          <width>1020</width>
+<!--           <width>1020</width>
           <height>1020</height>
+ -->          <width>640</width>
+          <height>480</height>
         </image>
         <clip>

File: surgical_task/models/surgical_frame.urdf.xacro (robot description, xacro)
@@ -20,10 +20,10 @@
       <inertia ixx="1" ixy="0" ixz="0" iyy="1" iyz="0" izz="1"/>
     </inertial>
-    <collision>
+<!--     <collision>
       <origin xyz="0 0 0" rpy="0 0 ${3.1415/2}"/>
       <geometry>
         <mesh filename="package://surgical_task/models/surgical_frame.stl" scale="0.001 0.001 0.001"/>
       </geometry>
-    </collision>
+    </collision> -->
     <visual>
       <origin xyz="0 0 0" rpy="0 0 ${3.1415/2}"/>

Commit message: [surgical_task]: surgical task refactorization + tool tracking with camera

File: surgical_task/models/panda_arm.urdf.xacro (robot description, xacro)
@@ -114,6 +114,8 @@
         <image>
           <format>R8G8B8</format>
-          <width>1020</width>
+<!--           <width>1020</width>
           <height>1020</height>
+ -->          <width>640</width>
+          <height>480</height>
         </image>
         <clip>

File: surgical_task/models/surgical_frame.urdf.xacro (robot description, xacro)
@@ -21,10 +21,10 @@
       <inertia ixx="1" ixy="0" ixz="0" iyy="1" iyz="0" izz="1"/>
     </inertial>
-    <collision>
+<!--     <collision>
       <origin xyz="0 0 0" rpy="0 0 ${3.1415/2}"/>
       <geometry>
         <mesh filename="package://surgical_task/models/surgical_frame.stl" scale="0.001 0.001 0.001"/>
       </geometry>
-    </collision>
+    </collision> -->
     <visual>
       <origin xyz="0 0 0" rpy="0 0 ${3.1415/2}"/>
