Commit message: fix bug in the tool.urdf.xacro, missing tool_id in macro create forceps

File: surgical_sim/models/urdf/surgical_tool/tool_base/tool_base.joints.xacro (robot description, xacro)
@@ -3,5 +3,5 @@
   <xacro:include filename="$(find surgical_sim)/models/urdf/surgical_tool/templates/joint.transmissions.xacro"/>
   <xacro:include filename="$(find surgical_sim)/models/urdf/surgical_tool/templates/gazebo.joints.xacro"/>
-  <xacro:macro name="create_tool_base_joints" params="parent_link xyz rpy tool_id:=right">
+  <xacro:macro name="create_tool_base_joints" params="parent_link xyz rpy tool_id">
     <!-- joint 1: tool_yaw -->
     <joint name="${tool_id}_tool_pitch" type="revolute">

File: surgical_sim/models/urdf/surgical_tool/tool_base/tool_base.links.xacro (robot description, xacro)
@@ -2,5 +2,5 @@
 <robot name="surgical_tool" xmlns:xacro="http://www.ros.org/wiki/xacro">
 <xacro:include filename="$(find surgical_sim)/models/urdf/surgical_tool/templates/gazebo.links.xacro"/>
-  <xacro:macro name="create_tool_base_links" params="parent_link xyz rpy tool_id:=right">
+  <xacro:macro name="create_tool_base_links" params="parent_link xyz rpy tool_id">
     <!-- link 1: tool_yaw -->
     <link name="${tool_id}_tool_yaw_link">

File: surgical_sim/models/urdf/surgical_tool/tool_base/tool_base.urdf.xacro (robot description, xacro)
@@ -3,5 +3,5 @@
   <xacro:include filename="$(find surgical_sim)/models/urdf/surgical_tool/tool_base/tool_base.links.xacro"/>
   <xacro:include filename="$(find surgical_sim)/models/urdf/surgical_tool/tool_base/tool_base.joints.xacro"/>
-  <xacro:macro name="create_tool_base" params="parent_link xyz rpy tool_id:=right">
+  <xacro:macro name="create_tool_base" params="parent_link xyz rpy tool_id">
     <xacro:create_tool_base_links
           parent_link="${parent_link}"

File: surgical_sim/models/urdf/surgical_tool/tool_create.urdf.xacro (robot description, xacro)
@@ -22,5 +22,5 @@
         parent_link="${parent_link}"
         xyz="${xyz}" rpy="${rpy}" tool_id="${tool_id}"/>
-     <xacro:create_forceps connected_to="${tool_id}_tool_wrist_shaft_link"/>
+     <xacro:create_forceps tool_id="${tool_id}" connected_to="$(arg toolID)_tool_wrist_shaft_link"/>
   </xacro:macro>
  <!--  -->

File: surgical_sim/models/urdf/surgical_tool/tool_forceps/tool_t_forceps.joints.xacro (robot description, xacro)
@@ -3,5 +3,5 @@
   <xacro:include filename="$(find surgical_sim)/models/urdf/surgical_tool/templates/joint.transmissions.xacro"/>
   <xacro:include filename="$(find surgical_sim)/models/urdf/surgical_tool/templates/gazebo.joints.xacro"/>
-  <xacro:macro name="create_forceps_joints" params="tool_id:=right connected_to">
+  <xacro:macro name="create_forceps_joints" params="tool_id connected_to">
     <!-- joint 5: tool wrist pitch joint -->
     <joint name="${tool_id}_tool_wrist_pitch" type="revolute">

File: surgical_sim/models/urdf/surgical_tool/tool_forceps/tool_t_forceps.links.xacro (robot description, xacro)
@@ -2,5 +2,5 @@
 <robot name="surgical_tool" xmlns:xacro="http://www.ros.org/wiki/xacro">
   <xacro:include filename="$(find surgical_sim)/models/urdf/surgical_tool/templates/gazebo.links.xacro"/>
-  <xacro:macro name="create_forceps_links" params="tool_id:=right">
+  <xacro:macro name="create_forceps_links" params="tool_id">
     <!-- link 5: tool_wrist_forceps_link -->
     <link name="${tool_id}_tool_wrist_forceps_link">

File: surgical_sim/models/urdf/surgical_tool/tool_forceps/tool_t_forceps.urdf.xacro (robot description, xacro)
@@ -3,5 +3,5 @@
   <xacro:include filename="$(find surgical_sim)/models/urdf/surgical_tool/tool_forceps/tool_t_forceps.links.xacro"/>
   <xacro:include filename="$(find surgical_sim)/models/urdf/surgical_tool/tool_forceps/tool_t_forceps.joints.xacro"/>
-  <xacro:macro name="create_forceps" params="tool_id:=right connected_to">
+  <xacro:macro name="create_forceps" params="tool_id connected_to">
     <xacro:create_forceps_links tool_id="${tool_id}"/>
     <xacro:create_forceps_joints tool_id="${tool_id}" connected_to="${connected_to}" />

File: surgical_sim/models/urdf/surgical_tool/tool_gripper/tool_t_gripper.urdf.xacro (robot description, xacro)
@@ -2,9 +2,9 @@
 <robot name="surgical_tool" xmlns:xacro="http://www.ros.org/wiki/xacro">
   <!-- gripper  -->
-  <xacro:macro name="create_gripper">
+  <xacro:macro name="create_gripper tool_id">
     <!-- joint 5: Outer wrist pitch joint -->
-    <joint name="outer_wrist_pitch" type="revolute">
-      <parent link="tool_wrist_shaft_link"/>
-      <child link="tool_wrist_gripper_link"/>
+    <joint name="${tool_id}_outer_wrist_pitch" type="revolute">
+      <parent link="${tool_id}_tool_wrist_shaft_link"/>
+      <child link="${tool_id}_tool_wrist_gripper_link"/>
       <axis xyz="0 0 1"/>
       <origin rpy="-1.5708 -1.5708 0" xyz="0 0 0"/>
@@ -22,7 +22,7 @@
     </link>
     <!-- joint 6: Outer wrist yaw joint -->
-    <joint name="outer_wrist_yaw" type="revolute">
-      <parent link="tool_wrist_gripper_link"/>
-      <child link="tool_wrist_gripper_shaft_link"/>
+    <joint name="${tool_id}_outer_wrist_yaw" type="revolute">
+      <parent link="${tool_id}_tool_wrist_gripper_link"/>
+      <child link="${tool_id}_tool_wrist_gripper_shaft_link"/>
       <axis xyz="0 0 1"/>
       <origin rpy="-1.5708 -1.5708 0" xyz="0.0091 0 0"/>
@@ -40,7 +40,7 @@
     </link>
     <!-- joint 7-1: Outer open angle 1  -->
-    <joint name="outer_wrist_open_angle" type="revolute">
-      <parent link="tool_wrist_gripper_shaft_link"/>
-      <child link="tool_wrist_gripper_ee_link_1"/>
+    <joint name="${tool_id}_outer_wrist_open_angle" type="revolute">
+      <parent link="${tool_id}_tool_wrist_gripper_shaft_link"/>
+      <child link="${tool_id}_tool_wrist_gripper_ee_link_1"/>
       <axis xyz="0 0 1"/>
       <origin rpy="0 0 0" xyz="0 0 0"/>
@@ -57,7 +57,7 @@
     </link>
     <!-- joint 7-2: Outer open angle 2   -->
-    <joint name="outer_wrist_open_angle_mimic" type="revolute">
-      <parent link="tool_wrist_gripper_shaft_link"/>
-      <child link="tool_wrist_gripper_ee_link_2"/>
+    <joint name="${tool_id}_outer_wrist_open_angle_mimic" type="revolute">
+      <parent link="${tool_id}_tool_wrist_gripper_shaft_link"/>
+      <child link="${tool_id}_tool_wrist_gripper_ee_link_2"/>
       <axis xyz="0 0 1"/>
       <origin rpy="0 0 0" xyz="0 0 0"/>
@@ -75,7 +75,7 @@
     </link>
     <!-- tool tip -->
-    <joint name="tool_tip_" type="fixed">
-      <parent link="tool_wrist_gripper_shaft_link"/>
-      <child link="tool_tip_link"/>
+    <joint name="${tool_id}_tool_tip_" type="fixed">
+      <parent link="${tool_id}_tool_wrist_gripper_shaft_link"/>
+      <child link="${tool_id}_tool_tip_link"/>
       <origin rpy="0 ${pi/2} ${pi/2}" xyz="0 0.0102 0"/>
     </joint>
