Commit message: now both tools have a position controller interface

File: surgical_sim/models/urdf/body/torso/torso.joints.xacro (robot description, xacro)
@@ -11,5 +11,5 @@
       <origin rpy="${rpy}" xyz="${xyz}"/>
     </joint>
-    <joint name="right_trocar_joint" type="fixed">
+    <!-- <joint name="right_trocar_joint" type="fixed">
       <parent link="torso_link"/>
       <child link="/right_trocar_link"/>
@@ -22,5 +22,5 @@
       <axis xyz="0 0 1"/>
       <origin rpy="0 0 ${pi/2}" xyz="0.0 0.0 0.2"/>
-    </joint>
+    </joint> -->
     <xacro:gazebo_joints name="torso_joint"/>
   </xacro:macro>

File: surgical_sim/models/urdf/body/torso/torso.links.xacro (robot description, xacro)
@@ -23,9 +23,10 @@
 			</inertial>
     </link>
-   <link name="/left_trocar_link"/>
-   <link name="/right_trocar_link"/>
+   <!-- <link name="/left_trocar_link"/>
+   <link name="/right_trocar_link"/> -->
    <xacro:gazebo_links name="torso_link"/>
-   <xacro:gazebo_links name="/left_trocar_link"/>
+   <!-- <xacro:gazebo_links name="/left_trocar_link"/>
    <xacro:gazebo_links name="/right_trocar_link"/>
+    -->
   </xacro:macro>
 </robot>

File: surgical_sim/models/urdf/surgical_tool/templates/gazebo.links.xacro (robot description, xacro)
@@ -12,5 +12,5 @@
 			<kp>${kpCollision}</kp>
 			<kd>${kdCollision}</kd>
-			<selfCollide>true</selfCollide>
+			<selfCollide>false</selfCollide>
 			<maxVel>0.01</maxVel>
 			<minDepth>0.003</minDepth>

File: surgical_sim/models/urdf/surgical_tool/tool.urdf (robot description, URDF)
Before this commit: robot surgical_tool, 14 links, 13 joints
Links:
- link right_tool_base_link: mass 0.001 -> 0.1
- link right_tool_main_link: mass 0.05 -> 0.1
- link right_tool_wrist_forceps_link: geometry visual mesh filename=package://surgical_sim/models/meshes/stl/tool/tool_wrist_fo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
- link right_tool_wrist_forceps_link_2_left: mass 0.1 -> 0.05
- link right_tool_wrist_forceps_link_2_right: mass 0.1 -> 0.05
- link right_tool_wrist_forceps_link_shaft: geometry visual mesh filename=package://surgical_sim/models/meshes/stl/tool/tool_wrist_fo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
Joints:
- removed joint right_tool_tip_
- removed joint right_tool_tip_ee
- removed joint right_tool_wrist_pitch
- removed joint right_tool_wrist_yaw
- added joint right_tool_tip_ee_fixed: type fixed, parent right_tool_tip_link, child right_tool_tip_link_ee, origin xyz=0 0 0 rpy=3.14159265359 0 -1.57079632679
- added joint right_tool_tip_fixed: type fixed, parent right_tool_wrist_forceps_link_shaft, child right_tool_tip_link, origin xyz=0 0.0202 0 rpy=0 1.57079632679 1.57079632679
- added joint right_tool_wrist_fixed_p: type fixed, parent right_tool_wrist_shaft_link, child right_tool_wrist_forceps_link, origin xyz=0 0 0 rpy=-1.5708 -1.5708 3.14159265359, axis 0 0 1
- added joint right_tool_wrist_fixed_yw: type fixed, parent right_tool_wrist_forceps_link, child right_tool_wrist_forceps_link_shaft, origin xyz=0.0091 0 0 rpy=0.00 -1.5708 -1.5708, axis 0 0 1
- joint right_tool_insertion: limit lower=0.0 upper=0.240 effort=1000 velocity=3 -> lower=0.0 upper=0.240 effort=30 velocity=100
- joint right_tool_pitch: limit lower=-1.5707 upper=1.5707 effort=1000 velocity=3 -> lower=-1.5707 upper=1.5707 effort=30 velocity=100
- joint right_tool_roll: limit lower=-1.5707 upper=1.5707 effort=1000 velocity=3 -> lower=-1.5707 upper=1.5707 effort=30 velocity=100
- joint right_tool_wrist_open_angle: limit lower=0 upper=0.523598775598 effort=1000 velocity=3.0 -> lower=0.0 upper=0.523598775598 effort=10 velocity=3.0
- joint right_tool_wrist_open_angle_mimic: limit lower=0 upper=0.523598775598 effort=1000 velocity=3.0 -> lower=0.0 upper=0.523598775598 effort=10 velocity=3.0
- joint right_tool_yaw: limit lower=-4.71238898038 upper=4.71238898038 effort=1000 velocity=3 -> lower=-4.71238898038 upper=4.71238898038 effort=30 velocity=100

File: surgical_sim/models/urdf/surgical_tool/tool_base/tool_base.joints.xacro (robot description, xacro)
@@ -6,35 +6,41 @@
     <!-- joint 1: tool_yaw -->
     <joint name="${tool_id}_tool_pitch" type="revolute">
+      <!-- <safety_controller k_position="100.0" k_velocity="40.0" soft_lower_limit="-1.5" soft_upper_limit="1.5"/> -->
       <parent link="${parent_link}"/>
       <child link="${tool_id}_tool_pitch_link"/>
       <axis xyz="0 0 1"/>
       <origin rpy="0 -${pi/2} ${pi}" xyz="0.0 0.0 0.0"/>
-      <limit lower="-1.5707" upper="1.5707" velocity="3" effort="1000"/>
+      <limit lower="-1.5707" upper="1.5707" velocity="100" effort="30"/>
     </joint>
     <!-- joint 2: tool_pitch -->
     <joint name="${tool_id}_tool_roll" type="revolute">
+      <!-- <safety_controller k_position="100.0" k_velocity="40.0" soft_lower_limit="-1.5" soft_upper_limit="1.5"/> -->
       <parent link="${tool_id}_tool_pitch_link"/>
       <child link="${tool_id}_tool_roll_link"/>
       <axis xyz="0 0 1"/>
       <origin rpy="-${pi/2} -${pi/2} 0" xyz="0 0 0"/>
-      <limit lower="-1.5707" upper="1.5707" velocity="3" effort="1000"/>
+      <limit lower="-1.5707" upper="1.5707" velocity="100" effort="30"/>
     </joint>
     <!-- joint : tool Roll -->
-    <joint name="${tool_id}_tool_yaw" type="revolute">
+    <joint name="${tool_id}_tool_yaw" type="continuous">
+      <!-- <safety_controller k_position="100.0" k_velocity="40.0" soft_lower_limit="-1.5" soft_upper_limit="1.5"/> -->
       <parent link="${tool_id}_tool_roll_link"/>
       <child link="${tool_id}_tool_yaw_link"/>
       <axis xyz="0 0 1"/>
       <origin rpy="${pi/2} 0 0" xyz="0 0 0"/>
-      <limit lower="-${1.5*pi}" upper="${1.5*pi}" velocity="3" effort="1000"/>
+      <limit velocity="2" effort="10"/>
+      <!-- <limit lower="-${1.5 * pi}" upper="${1.5 * pi}" velocity="2" effort="2"/> -->
     </joint>
     <!-- joint 3: insertion -->
     <joint name="${tool_id}_tool_insertion" type="prismatic">
+      <!-- <safety_controller k_position="100.0" k_velocity="40.0" soft_lower_limit="-1.5" soft_upper_limit="1.5"/> -->
       <parent link="${tool_id}_tool_yaw_link"/>
       <child link="${tool_id}_tool_main_link"/>
       <axis xyz="0 0 1"/>
       <origin rpy="0 0 0" xyz="0 0 -${0.4318-0.041}"/>
-      <limit lower="0.0" upper="0.240" velocity="3" effort="1000"/>
+      <limit lower="0.0" upper="0.240" velocity="100" effort="30"/>
     </joint>
     <joint name="${tool_id}_tool_wrist_fixed" type="fixed">
+      <!-- <safety_controller k_position="100.0" k_velocity="40.0" soft_lower_limit="-1.5" soft_upper_limit="1.5"/> -->
       <parent link="${tool_id}_tool_main_link"/>
       <child link="${tool_id}_tool_wrist_link"/>
@@ -44,4 +50,5 @@
     <!-- joint 4-1: tool roll shaft joint FIXED-->
     <joint name="${tool_id}_tool_wrist_shaft_fixed" type="fixed">
+      <!-- <safety_controller k_position="100.0" k_velocity="40.0" soft_lower_limit="-1.5" soft_upper_limit="1.5"/> -->
       <parent link="${tool_id}_tool_wrist_link"/>
       <child link="${tool_id}_tool_wrist_shaft_link"/>

File: surgical_sim/models/urdf/surgical_tool/tool_base/tool_base.links.xacro (robot description, xacro)
@@ -2,4 +2,7 @@
 <robot name="surgical_tool" xmlns:xacro="http://www.ros.org/wiki/xacro">
 <xacro:include filename="$(find surgical_sim)/models/urdf/surgical_tool/templates/gazebo.links.xacro"/>
+  <xacro:property name="toolMass" value="0.1"/>
+  <xacro:property name="toolLength" value="0.4"/>
+  <xacro:property name="toolRadius" value="0.005"/>
   <xacro:macro name="create_tool_base_links" params="parent_link xyz rpy tool_id">
     <!-- link 1: tool_yaw -->
@@ -42,6 +45,6 @@
       <inertial>
 				<origin xyz="0 0 0" rpy="0 0 0"/>
-				<mass value="0.05"/>
-				<inertia ixx="0.01" ixy="0.0" ixz="0.0" iyy="0.01" iyz="0.0" izz="0.005"/>
+			<mass value="${toolMass}"/>
+        <inertia ixx="${toolMass*(3*toolRadius*toolRadius+toolLength*toolLength)/12}" ixy="0" ixz="0" iyy="${toolMass*(3*toolRadius*toolRadius+toolLength*toolLength)/12}" iyz="0" izz="${toolMass*toolRadius*toolRadius/2}"/>
 			</inertial>
     </link>
@@ -86,10 +89,10 @@
 			</inertial>
     </link>
-    <xacro:gazebo_links name="tool_yaw_link"/>
-    <xacro:gazebo_links name="tool_pitch_link"/>
-    <xacro:gazebo_links name="tool_roll_link"/>
-    <xacro:gazebo_links name="tool_main_link"/>
-    <xacro:gazebo_links name="tool_wrist_link"/>
-    <xacro:gazebo_links name="tool_wrist_shaft_link"/>
+    <xacro:gazebo_links name="${tool_id}_tool_yaw_link"/>
+    <xacro:gazebo_links name="${tool_id}_tool_pitch_link"/>
+    <xacro:gazebo_links name="${tool_id}_tool_roll_link"/>
+    <xacro:gazebo_links name="${tool_id}_tool_main_link"/>
+    <xacro:gazebo_links name="${tool_id}_tool_wrist_link"/>
+    <xacro:gazebo_links name="${tool_id}_tool_wrist_shaft_link"/>
   </xacro:macro>
 </robot>

File: surgical_sim/models/urdf/surgical_tool/tool_create.urdf.xacro (robot description, xacro)
@@ -29,6 +29,6 @@
     <inertial>
       <origin xyz="0.0 0.0 0.0" rpy="0.0 0.0 0.0"/>
-      <mass value="0.001"/>
-      <inertia ixx="0.001" ixy="0.0" ixz="0.0" iyy="0.0001" iyz="0.0" izz="0.0001"/>
+      <mass value="0.1"/>
+      <inertia ixx="0.01" ixy="0.0" ixz="0.0" iyy="0.01" iyz="0.0" izz="0.001"/>
     </inertial>
   </link>

File: surgical_sim/models/urdf/surgical_tool/tool_forceps/tool_t_forceps.joints.xacro (robot description, xacro)
@@ -5,5 +5,5 @@
   <xacro:macro name="create_forceps_joints" params="tool_id connected_to">
     <!-- joint 5: tool wrist pitch joint -->
-    <joint name="${tool_id}_tool_wrist_pitch" type="revolute">
+    <joint name="${tool_id}_tool_wrist_pitch" type="fixed">
       <parent link="${connected_to}"/>
       <!-- <parent link="${tool_id}_world"/> -->
@@ -11,13 +11,13 @@
       <axis xyz="0 0 1"/>
       <origin rpy="-1.5708 -1.5708 ${pi}" xyz="0 0 0"/>
-      <limit lower="-${pi/2}" upper="${pi/2}" velocity="3.0" effort="1000"/>
+      <limit lower="-${pi/2}" upper="${pi/2}" velocity="3.0" effort="2"/>
     </joint>
     <!-- joint 6: Tool wrist yaw joint -->
-    <joint name="${tool_id}_tool_wrist_yaw" type="revolute">
+    <joint name="${tool_id}_tool_wrist_yaw" type="fixed">
       <parent link="${tool_id}_tool_wrist_forceps_link"/>
       <child link="${tool_id}_tool_wrist_forceps_link_shaft"/>
       <axis xyz="0 0 1"/>
       <origin rpy="0.00 -1.5708 -1.5708" xyz="0.0091 0 0"/>
-      <limit lower="-${pi/2}" upper="${pi/2}" velocity="3.0" effort="1000"/>
+      <limit lower="-${pi/2}" upper="${pi/2}" velocity="3.0" effort="2"/>
     </joint>
     <!-- joint 6-1: tool open angle 1 -->
@@ -27,5 +27,5 @@
       <axis xyz="0 0 1"/>
       <origin rpy="0 0 0" xyz="0 0 0"/>
-      <limit lower="0" upper="${radians(30.0)}" velocity="3.0" effort="1000"/>
+      <limit lower="${radians(0.0)}" upper="${radians(30.0)}" velocity="3.0" effort="10"/>
     </joint>
   <!-- joint 6-2: tool open angle 2  -->
@@ -35,5 +35,5 @@
       <axis xyz="0 0 1"/>
       <origin rpy="3.1415926 0 0" xyz="0 0 0"/>
-      <limit lower="0" upper="${radians(30.0)}" velocity="3.0" effort="1000"/>
+      <limit lower="${radians(0.0)}" upper="${radians(30.0)}" velocity="3.0" effort="10"/>
       <mimic joint="${tool_id}_tool_wrist_open_angle" multiplier="1"/>
     </joint>
@@ -49,6 +49,6 @@
       <origin rpy="${pi} 0 ${-pi/2}" xyz="0 0 0"/>
     </joint>
-    <xacro:joint_trans name="${tool_id}_tool_wrist_pitch" reduction="1"/>
-    <xacro:joint_trans name="${tool_id}_tool_wrist_yaw" reduction="1"/>
+    <!-- <xacro:joint_trans name="${tool_id}_tool_wrist_pitch" reduction="1"/>
+    <xacro:joint_trans name="${tool_id}_tool_wrist_yaw" reduction="1"/> -->
     <xacro:joint_trans name="${tool_id}_tool_wrist_open_angle" reduction="1"/>
     <xacro:joint_trans name="${tool_id}_tool_wrist_open_angle_mimic" reduction="1"/>

File: surgical_sim/models/urdf/surgical_tool/tool_forceps/tool_t_forceps.links.xacro (robot description, xacro)
@@ -12,10 +12,4 @@
         <material name="gray"><color rgba="0.5 0.5 0.9 1.0"/></material>
       </visual>
-      <collision>
-        <origin rpy="0.00 -1.5708 0.0" xyz="-0.0024 0.00 0.000"/>
-        <geometry>
-          <mesh filename="package://surgical_sim/models/meshes/stl/tool/tool_wrist_forceps_link_1.stl"/>
-        </geometry>
-      </collision>
       <inertial>
           <origin xyz="0 0 0" rpy="0 0 0"/>
@@ -33,14 +27,8 @@
         <material name="gray"><color rgba="0.5 0.5 0.9 1.0"/></material>
       </visual>
-      <collision>
-        <origin rpy="0.00 1.5708 0.0" xyz="0.0 0.00 0.000"/>
-        <geometry>
-          <mesh filename="package://surgical_sim/models/meshes/stl/tool/tool_wrist_forceps_link_1_shaft.stl"/>
-        </geometry>
-      </collision>
       <inertial>
 				<origin xyz="0 0 0" rpy="0 0 0"/>
 				<mass value="0.1"/>
-        <inertia ixx="1" ixy="0.0" ixz="0.0" iyy="1" iyz="0.0" izz="0.05"/>
+        <inertia ixx="0.1" ixy="0.0" ixz="0.0" iyy="0.1" iyz="0.0" izz="0.005"/>
 			</inertial>
     </link>
@@ -61,6 +49,6 @@
       <inertial>
 				<origin xyz="0 0 0" rpy="0 0 0"/>
-        <mass value="0.1"/>
-        <inertia ixx="1" ixy="0.0" ixz="0.0" iyy="1" iyz="0.0" izz="0.05"/>
+        <mass value="0.05"/>
+        <inertia ixx="0.01" ixy="0.0" ixz="0.0" iyy="0.01" iyz="0.0" izz="0.005"/>
 			</inertial>
     </link>
@@ -81,6 +69,6 @@
       <inertial>
 				<origin xyz="0 0 0" rpy="0 0 0"/>
-				<mass value="0.1"/>
-        <inertia ixx="1" ixy="0.0" ixz="0.0" iyy="1" iyz="0.0" izz="0.05"/>
+				<mass value="0.05"/>
+        <inertia ixx="0.01" ixy="0.0" ixz="0.0" iyy="0.01" iyz="0.0" izz="0.005"/>
 			</inertial>
     </link>
@@ -91,5 +79,5 @@
     <xacro:gazebo_links name="${tool_id}_tool_wrist_forceps_link_2_left"/>
     <xacro:gazebo_links name="${tool_id}_tool_wrist_forceps_link_2_right"/>
-      <xacro:gazebo_links name="${tool_id}_tool_tip_link"/>
+    <xacro:gazebo_links name="${tool_id}_tool_tip_link"/>
     <xacro:gazebo_links name="${tool_id}_tool_tip_link_ee"/>
   </xacro:macro>
