Commit message: integrate frankas with tool (separately controlled)

File: surgical_sim/models/urdf/franka/panda.urdf (robot description, URDF)
Before this commit: robot panda, 20 links, 19 joints
Links:
- removed link panda_tool_base_link
- removed link panda_tool_main_link
- removed link panda_tool_tip_link
- removed link panda_tool_tip_link_ee
- removed link panda_tool_wrist_forceps_link
- removed link panda_tool_wrist_forceps_link_2_left
- removed link panda_tool_wrist_forceps_link_2_right
- removed link panda_tool_wrist_forceps_link_shaft
- removed link panda_tool_wrist_link
- removed link panda_tool_wrist_shaft_link
Joints:
- removed joint panda_base_fixed
- removed joint panda_tool_main_fixed
- removed joint panda_tool_tip_
- removed joint panda_tool_tip_ee
- removed joint panda_tool_wrist_fixed
- removed joint panda_tool_wrist_open_angle
- removed joint panda_tool_wrist_open_angle_mimic
- removed joint panda_tool_wrist_pitch
- removed joint panda_tool_wrist_shaft_fixed
- removed joint panda_tool_wrist_yaw

File: surgical_sim/models/urdf/franka/panda_arm.gazebo.xacro (robot description, xacro)
@@ -3,84 +3,84 @@
   <gazebo>
     <plugin name="gazebo_ros_control" filename="libgazebo_ros_control.so">
-      <robotNamespace>${arm_id}</robotNamespace>
+      <robotNamespace>/${arm_id}_panda</robotNamespace>
       <legacyModeNS>true</legacyModeNS>
     </plugin>
   </gazebo>
-  <gazebo reference="${arm_id}_link0"/>
-  <gazebo reference="${arm_id}_link1"/>
-  <gazebo reference="${arm_id}_link2"/>
-  <gazebo reference="${arm_id}_link3"/>
-  <gazebo reference="${arm_id}_link4"/>
-  <gazebo reference="${arm_id}_link5"/>
-  <gazebo reference="${arm_id}_link6"/>
-  <gazebo reference="${arm_id}_link7"/>
-  <gazebo reference="${arm_id}_link8"/>
-   <transmission name="${arm_id}_joint1_trans">
+  <gazebo reference="${arm_id}_panda_link0"/>
+  <gazebo reference="${arm_id}_panda_link1"/>
+  <gazebo reference="${arm_id}_panda_link2"/>
+  <gazebo reference="${arm_id}_panda_link3"/>
+  <gazebo reference="${arm_id}_panda_link4"/>
+  <gazebo reference="${arm_id}_panda_link5"/>
+  <gazebo reference="${arm_id}_panda_link6"/>
+  <gazebo reference="${arm_id}_panda_link7"/>
+  <gazebo reference="${arm_id}_panda_link8"/>
+   <transmission name="${arm_id}_panda_joint1_trans">
     <type>transmission_interface/SimpleTransmission</type>
-    <joint name="${arm_id}_joint1">
+    <joint name="${arm_id}_panda_joint1">
       <hardwareInterface>hardware_interface/PositionJointInterface</hardwareInterface>
       <!-- <hardwareInterface>PositionJointInterface</hardwareInterface> -->
     </joint>
-    <actuator name="${arm_id}_joint1_motor">
+    <actuator name="${arm_id}_panda_joint1_motor">
       <mechanicalReduction>1</mechanicalReduction>
     </actuator>
   </transmission>
-  <transmission name="${arm_id}_joint2_trans">
+  <transmission name="${arm_id}_panda_joint2_trans">
     <type>transmission_interface/SimpleTransmission</type>
-    <joint name="${arm_id}_joint2">
+    <joint name="${arm_id}_panda_joint2">
       <hardwareInterface>hardware_interface/PositionJointInterface</hardwareInterface>
       <!-- <hardwareInterface>PositionJointInterface</hardwareInterface> -->
     </joint>
-    <actuator name="${arm_id}_joint2_motor">
+    <actuator name="${arm_id}_panda_joint2_motor">
       <mechanicalReduction>1</mechanicalReduction>
     </actuator>
   </transmission>
-  <transmission name="${arm_id}_joint3_trans">
+  <transmission name="${arm_id}_panda_joint3_trans">
     <type>transmission_interface/SimpleTransmission</type>
-    <joint name="${arm_id}_joint3">
+    <joint name="${arm_id}_panda_joint3">
       <hardwareInterface>hardware_interface/PositionJointInterface</hardwareInterface>
       <!-- <hardwareInterface>PositionJointInterface</hardwareInterface> -->
     </joint>
-    <actuator name="${arm_id}_joint3_motor">
+    <actuator name="${arm_id}_panda_joint3_motor">
       <mechanicalReduction>1</mechanicalReduction>
     </actuator>
   </transmission>
-  <transmission name="${arm_id}_joint4_trans">
+  <transmission name="${arm_id}_panda_joint4_trans">
     <type>transmission_interface/SimpleTransmission</type>
-    <joint name="${arm_id}_joint4">
+    <joint name="${arm_id}_panda_joint4">
       <hardwareInterface>hardware_interface/PositionJointInterface</hardwareInterface>
       <!-- <hardwareInterface>PositionJointInterface</hardwareInterface> -->
     </joint>
-    <actuator name="${arm_id}_joint4_motor">
+    <actuator name="${arm_id}_panda_joint4_motor">
       <mechanicalReduction>1</mechanicalReduction>
     </actuator>
   </transmission>
-  <transmission name="${arm_id}_joint5_trans">
+  <transmission name="${arm_id}_panda_joint5_trans">
     <type>transmission_interface/SimpleTransmission</type>
-    <joint name="${arm_id}_joint5">
+    <joint name="${arm_id}_panda_joint5">
       <hardwareInterface>hardware_interface/PositionJointInterface</hardwareInterface>
       <!-- <hardwareInterface>PositionJointInterface</hardwareInterface> -->
     </joint>
-    <actuator name="${arm_id}_joint5_motor">
+    <actuator name="${arm_id}_panda_joint5_motor">
       <mechanicalReduction>1</mechanicalReduction>
     </actuator>
   </transmission>
-  <transmission name="${arm_id}_joint6_trans">
+  <transmission name="${arm_id}_panda_joint6_trans">
     <type>transmission_interface/SimpleTransmission</type>
-    <joint name="${arm_id}_joint6">
+    <joint name="${arm_id}_panda_joint6">
       <hardwareInterface>hardware_interface/PositionJointInterface</hardwareInterface>
       <!-- <hardwareInterface>PositionJointInterface</hardwareInterface> -->
     </joint>
-    <actuator name="${arm_id}_joint6_motor">
+    <actuator name="${arm_id}_panda_joint6_motor">
       <mechanicalReduction>1</mechanicalReduction>
     </actuator>
   </transmission>
-  <transmission name="${arm_id}_joint7_trans">
+  <transmission name="${arm_id}_panda_joint7_trans">
     <type>transmission_interface/SimpleTransmission</type>
-    <joint name="${arm_id}_joint7">
+    <joint name="${arm_id}_panda_joint7">
       <hardwareInterface>hardware_interface/PositionJointInterface</hardwareInterface>
       <!-- <hardwareInterface>PositionJointInterface</hardwareInterface> -->
     </joint>
-    <actuator name="${arm_id}_joint7_motor">
+    <actuator name="${arm_id}_panda_joint7_motor">
       <mechanicalReduction>1</mechanicalReduction>
     </actuator>

File: surgical_sim/models/urdf/franka/panda_arm.urdf.xacro (robot description, xacro)
@@ -2,5 +2,5 @@
 <robot xmlns:xacro="http://www.ros.org/wiki/xacro" name="panda">
 	<xacro:arg name="gazebo" default="true"/>
-	<xacro:arg name="robotName" default="panda"/>
+	<xacro:arg name="arm_id" default="right"/>
   <xacro:arg name="origin.x" default="0"/>
   <xacro:arg name="origin.y" default="0"/>
@@ -9,116 +9,9 @@
   <xacro:arg name="origin.ay" default="0"/>
   <xacro:arg name="origin.az" default="0"/>
-  <xacro:arg name="addFrame" default="0"/>
-  <xacro:arg name="addCamera" default="0"/>
-  <xacro:arg name="useInstrument" default="1"/>
-  <xacro:property name="toolMass" value="0.1"/>
-  <xacro:property name="toolLength" value="0.4"/>
-  <xacro:property name="toolRadius" value="0.005"/>
-  <xacro:property name="M_PI" value="3.14159265359" />
   <gazebo reference="world">
-<!--     <static>true</static>
-    <turnGravityOff>true</turnGravityOff> -->
   </gazebo>
-  <xacro:include filename="$(find surgical_sim)/models/urdf/surgical_tool_panda/tool_create.urdf.xacro">
-  	<xacro:arg name="bringup_solo" value="false"/>
-    <xacro:arg name="toolID" value="$(arg robotName)"/>
-  </xacro:include>
   <xacro:include filename="$(find surgical_sim)/models/urdf/franka/panda_arm.xacro" >
   	<xacro:arg name="gazebo" value="${gazebo}"/>
   </xacro:include>
-  <xacro:panda_arm connected_to='world' arm_id="$(arg robotName)" xyz='$(arg origin.x) $(arg origin.y) $(arg origin.z)' rpy='$(arg origin.ax) $(arg origin.ay) $(arg origin.az)'/>
- <xacro:if value="${$(arg useInstrument)==0}">
-    <link name='$(arg robotName)_tool'>
-      <inertial>
-        <origin xyz="0 0 ${toolLength/2}" rpy="0 0 0"/>
-        <mass value="${toolMass}"/>
-        <inertia ixx="${toolMass*(3*toolRadius*toolRadius+toolLength*toolLength)/12}" ixy="0" ixz="0" iyy="${toolMass*(3*toolRadius*toolRadius+toolLength*toolLength)/12}" iyz="0" izz="${toolMass*toolRadius*toolRadius/2}"/>
-      </inertial>
-      <collision name='collision'>
-        <origin xyz="0 0 ${toolLength/2}" rpy="0 0 0" />
-        <geometry>
-          <cylinder length="${toolLength}" radius="${toolRadius}"/>
-        </geometry>
-      </collision>
-      <visual name='visual'>
-        <origin xyz="0 0 ${toolLength/2}" rpy="0 0 0" />
-        <geometry>
-          <cylinder length="${toolLength}" radius="${toolRadius}"/>
-        </geometry>
-        <material name="white">
-        <color rgba="1.0 1.0 1.0 1.0"/>
-      </material>
-      </visual>
-    </link>
-    <joint name="$(arg robotName)_tool_joint" type="fixed">
-      <origin xyz="0 0 0" rpy="0 0 0"/>
-      <parent link="$(arg robotName)_link8"/>
-      <child link="$(arg robotName)_tool"/>
-    </joint>
-  </xacro:if>
-  <xacro:if value="${$(arg useInstrument)==1}">
-    <xacro:add_tool connected_to="$(arg robotName)_link8" tool_name="$(arg robotName)"/>
-  </xacro:if>
-<xacro:if value="${$(arg addFrame)==1}">
-  <link name='$(arg robotName)_tipframe'>
-      <visual name='visual'>
-        <origin xyz="0 0 ${toolLength}" rpy="0 0 0" />
-          <geometry>
-           <mesh filename="package://surgical_simulator/models/meshes/dae/franka/frame.dae" scale="0.035 0.035 0.035"/>
-         </geometry>
-       </visual>
-  </link>
-  <joint name="$(arg robotName)_frame_joint" type="fixed">
-      <origin xyz="0 0 0" rpy="0 0 0"/>
-      <parent link="$(arg robotName)_tool"/>
-      <child link="$(arg robotName)_tipframe"/>
-  </joint>
- </xacro:if>
-<xacro:if value="${$(arg addCamera)==1}">
-  <link name="$(arg robotName)_camera_link">
-    <inertial>
-      <mass value="0.001" />
-      <origin xyz="0 0 0" />
-      <inertia ixx="0.0001" ixy="0.0" ixz="0.0" iyy="0.0001" iyz="0.0" izz="0.0001" />
-    </inertial>
-  </link>
-  <joint name="$(arg robotName)_camera_joint" type="fixed">
-        <parent link="$(arg robotName)_tool"/>
-        <child link="$(arg robotName)_camera_link"/>
-        <origin xyz="0 0 ${toolLength}" rpy="0 0 0"/>
-  </joint>
-  <gazebo reference='$(arg robotName)_camera_link'>
-    <sensor type="camera" name="camera_camera_sensor">
-      <!-- <alwaysOn>true</alwaysOn> -->
-      <update_rate>30.0</update_rate>
-    <camera>
-        <pose>0 0 0 0 ${-M_PI/2} ${M_PI}</pose>
-        <horizontal_fov>${85 * M_PI/180.0}</horizontal_fov>
-        <image>
-          <format>R8G8B8</format>
-          <width>1020</width>
-          <height>1020</height>
-        </image>
-        <clip>
-          <near>0.01</near>
-          <far>100</far>
-        </clip>
-      </camera>
-      <plugin name="camera_camera_controller" filename="libgazebo_ros_camera.so">
-        <alwaysOn>true</alwaysOn>
-        <updateRate>30.0</updateRate>
-        <cameraName>camera</cameraName>
-        <imageTopicName>image_raw</imageTopicName>
-        <cameraInfoTopicName>camera_info</cameraInfoTopicName>
-        <frameName>camera_link</frameName>
-        <hackBaseline>0.07</hackBaseline>
-        <distortionK1>0.0</distortionK1>
-        <distortionK2>0.0</distortionK2>
-        <distortionK3>0.0</distortionK3>
-        <distortionT1>0.0</distortionT1>
-        <distortionT2>0.0</distortionT2>
-      </plugin>
-    </sensor>
-  </gazebo>
-</xacro:if>
+  <xacro:panda_arm connected_to='world' arm_id="$(arg arm_id)" xyz='$(arg origin.x) $(arg origin.y) $(arg origin.z)' rpy='$(arg origin.ax) $(arg origin.ay) $(arg origin.az)'/>
 </robot>

File: surgical_sim/models/urdf/franka/panda_arm.xacro (robot description, xacro)
@@ -1,10 +1,10 @@
 <?xml version='1.0' encoding='utf-8'?>
 <robot xmlns:xacro="http://www.ros.org/wiki/xacro" name="panda">
-  <xacro:macro name="panda_arm" params="arm_id:='panda' package_name:='surgical_sim' connected_to:='' xyz:='0 0 0' rpy:='0 0 0'">
+  <xacro:macro name="panda_arm" params="arm_id package_name:='surgical_sim' connected_to:='' xyz:='0 0 0' rpy:='0 0 0'">
     <xacro:unless value="${not connected_to}">
       <link name="${connected_to}"/>
-      <joint name="${arm_id}_joint_${connected_to}" type="fixed">
+      <joint name="${arm_id}_panda_joint_${connected_to}" type="fixed">
         <parent link="${connected_to}"/>
-        <child link="${arm_id}_link0"/>
+        <child link="${arm_id}_panda_link0"/>
         <origin rpy="${rpy}" xyz="${xyz}"/>
       </joint>
@@ -15,5 +15,5 @@
       <xacro:include filename="$(find surgical_sim)/models/urdf/franka/panda_arm.gazebo.xacro"/>
     </xacro:if>
-    <link name="${arm_id}_link0">
+    <link name="${arm_id}_panda_link0">
       <inertial>
         <mass value="2.92" />
@@ -35,5 +35,5 @@
       </collision>
     </link>
-    <link name="${arm_id}_link1">
+    <link name="${arm_id}_panda_link1">
       <inertial>
         <mass value="2.74" />
@@ -55,13 +55,13 @@
       </collision>
     </link>
-    <joint name="${arm_id}_joint1" type="revolute">
+    <joint name="${arm_id}_panda_joint1" type="revolute">
       <safety_controller k_position="100.0" k_velocity="40.0" soft_lower_limit="-2.8973" soft_upper_limit="2.8973"/>
       <origin rpy="0 0 0" xyz="0 0 0.333"/>
-      <parent link="${arm_id}_link0"/>
-      <child link="${arm_id}_link1"/>
+      <parent link="${arm_id}_panda_link0"/>
+      <child link="${arm_id}_panda_link1"/>
       <axis xyz="0 0 1"/>
       <limit effort="87" lower="-2.8973" upper="2.8973" velocity="2.1750"/>
     </joint>
-    <link name="${arm_id}_link2">
+    <link name="${arm_id}_panda_link2">
       <inertial>
         <mass value="2.74" />
@@ -83,13 +83,13 @@
       </collision>
     </link>
-    <joint name="${arm_id}_joint2" type="revolute">
+    <joint name="${arm_id}_panda_joint2" type="revolute">
       <safety_controller k_position="100.0" k_velocity="40.0" soft_lower_limit="-1.7628" soft_upper_limit="1.7628"/>
       <origin rpy="${-pi/2} 0 0" xyz="0 0 0"/>
-      <parent link="${arm_id}_link1"/>
-      <child link="${arm_id}_link2"/>
+      <parent link="${arm_id}_panda_link1"/>
+      <child link="${arm_id}_panda_link2"/>
       <axis xyz="0 0 1"/>
       <limit effort="87" lower="-1.7628" upper="1.7628" velocity="2.1750"/>
     </joint>
-    <link name="${arm_id}_link3">
+    <link name="${arm_id}_panda_link3">
       <inertial>
         <mass value="2.38" />
@@ -111,13 +111,13 @@
       </collision>
     </link>
-    <joint name="${arm_id}_joint3" type="revolute">
+    <joint name="${arm_id}_panda_joint3" type="revolute">
       <safety_controller k_position="100.0" k_velocity="40.0" soft_lower_limit="-2.8973" soft_upper_limit="2.8973"/>
       <origin rpy="${pi/2} 0 0" xyz="0 -0.316 0"/>
-      <parent link="${arm_id}_link2"/>
-      <child link="${arm_id}_link3"/>
+      <parent link="${arm_id}_panda_link2"/>
+      <child link="${arm_id}_panda_link3"/>
       <axis xyz="0 0 1"/>
       <limit effort="87" lower="-2.8973" upper="2.8973" velocity="2.1750"/>
     </joint>
-    <link name="${arm_id}_link4">
+    <link name="${arm_id}_panda_link4">
       <inertial>
         <mass value="2.38" />
@@ -139,15 +139,15 @@
       </collision>
     </link>
-    <joint name="${arm_id}_joint4" type="revolute">
+    <joint name="${arm_id}_panda_joint4" type="revolute">
       <safety_controller k_position="100.0" k_velocity="40.0" soft_lower_limit="-3.0718" soft_upper_limit="0.0698"/>
       <!-- soft_upper_limitr should be -0.0698, but that brakes simulation when initial position for this joint is 0.0 -->
       <origin rpy="${pi/2} 0 0" xyz="0.0825 0 0"/>
-      <parent link="${arm_id}_link3"/>
-      <child link="${arm_id}_link4"/>
+      <parent link="${arm_id}_panda_link3"/>
+      <child link="${arm_id}_panda_link4"/>
       <axis xyz="0 0 1"/>
       <limit effort="87" lower="-3.0718" upper="0.0698" velocity="2.1750"/>
       <!-- upper should be -0.0698, but that brakes simulation when initial position for this joint is 0.0 -->
     </joint>
-    <link name="${arm_id}_link5">
+    <link name="${arm_id}_panda_link5">
       <inertial>
         <mass value="2.74" />
@@ -169,13 +169,13 @@
       </collision>
     </link>
-    <joint name="${arm_id}_joint5" type="revolute">
+    <joint name="${arm_id}_panda_joint5" type="revolute">
       <safety_controller k_position="100.0" k_velocity="40.0" soft_lower_limit="-2.8973" soft_upper_limit="2.8973"/>
       <origin rpy="${-pi/2} 0 0" xyz="-0.0825 0.384 0"/>
-      <parent link="${arm_id}_link4"/>
-      <child link="${arm_id}_link5"/>
+      <parent link="${arm_id}_panda_link4"/>
+      <child link="${arm_id}_panda_link5"/>
       <axis xyz="0 0 1"/>
       <limit effort="12" lower="-2.8973" upper="2.8973" velocity="2.6100"/>
     </joint>
-    <link name="${arm_id}_link6">
+    <link name="${arm_id}_panda_link6">
       <inertial>
         <mass value="1.55" />
@@ -197,13 +197,13 @@
       </collision>
     </link>
-    <joint name="${arm_id}_joint6" type="revolute">
+    <joint name="${arm_id}_panda_joint6" type="revolute">
       <safety_controller k_position="100.0" k_velocity="40.0" soft_lower_limit="-0.0175" soft_upper_limit="3.7525"/>
       <origin rpy="${pi/2} 0 0" xyz="0 0 0"/>
-      <parent link="${arm_id}_link5"/>
-      <child link="${arm_id}_link6"/>
+      <parent link="${arm_id}_panda_link5"/>
+      <child link="${arm_id}_panda_link6"/>
       <axis xyz="0 0 1"/>
       <limit effort="12" lower="-0.0175" upper="3.7525" velocity="2.6100"/>
     </joint>
-    <link name="${arm_id}_link7">
+    <link name="${arm_id}_panda_link7">
       <inertial>
         <mass value="0.54" />
@@ -225,17 +225,17 @@
       </collision>
     </link>
-    <joint name="${arm_id}_joint7" type="revolute">
+    <joint name="${arm_id}_panda_joint7" type="revolute">
       <safety_controller k_position="100.0" k_velocity="40.0" soft_lower_limit="-2.8973" soft_upper_limit="2.8973"/>
       <origin rpy="${pi/2} 0 0" xyz="0.088 0 0"/>
-      <parent link="${arm_id}_link6"/>
-      <child link="${arm_id}_link7"/>
+      <parent link="${arm_id}_panda_link6"/>
+      <child link="${arm_id}_panda_link7"/>
       <axis xyz="0 0 1"/>
       <limit effort="12" lower="-2.8973" upper="2.8973" velocity="2.6100"/>
     </joint>
-    <link name="${arm_id}_link8"/>
-    <joint name="${arm_id}_joint8" type="fixed">
+    <link name="${arm_id}_panda_link8"/>
+    <joint name="${arm_id}_panda_joint8" type="fixed">
       <origin rpy="0 0 0" xyz="0 0 0.107"/>
-      <parent link="${arm_id}_link7"/>
-      <child link="${arm_id}_link8"/>
+      <parent link="${arm_id}_panda_link7"/>
+      <child link="${arm_id}_panda_link8"/>
       <axis xyz="0 0 0"/>
     </joint>

File: surgical_sim/models/urdf/surgical_tool/tool_forceps/tool_t_forceps.links.xacro (robot description, xacro)
@@ -84,6 +84,6 @@
     <xacro:gazebo_links name="${tool_id}_tool_wrist_forceps_link"/>
     <xacro:gazebo_links name="${tool_id}_tool_wrist_forceps_link_shaft"/>
-    <xacro:gazebo_links name="${tool_id}_tool_wrist_forceps_link_2_left" frictCoeff="10.0"/>
-    <xacro:gazebo_links name="${tool_id}_tool_wrist_forceps_link_2_right" frictCoeff="10.0"/>
+    <xacro:gazebo_links name="${tool_id}_tool_wrist_forceps_link_2_left" frictCoeff="0.2"/>
+    <xacro:gazebo_links name="${tool_id}_tool_wrist_forceps_link_2_right" frictCoeff="0.2"/>
     <xacro:gazebo_links name="${tool_id}_tool_tip_link"/>
     <xacro:gazebo_links name="${tool_id}_tool_tip_link_ee"/>

File: surgical_sim/models/urdf/target_object/templates/gazebo.joints.xacro (robot description, xacro)
@@ -3,6 +3,6 @@
 	<xacro:macro name="gazebo_joints" params="name">
 		<gazebo reference="${name}">
-			<!-- <implicitSpringDamper>0</implicitSpringDamper>
-			<provideFeedback>1</provideFeedback> -->
+			<implicitSpringDamper>0</implicitSpringDamper>
+			<!--provideFeedback>1</provideFeedback> -->
 		</gazebo>
 	</xacro:macro>

File: surgical_sim/models/urdf/target_object/templates/gazebo.links.xacro (robot description, xacro)
@@ -1,7 +1,7 @@
 <?xml version="1.0"?>
 <robot xmlns:xacro="http://www.ros.org/wiki/xacro">
-	<xacro:property name="fricCoeff1" value="100.0"/>
-	<xacro:property name="fricCoeff2" value="100.0"/>
-	<xacro:property name="kpCollision" value="100000000.0"/>
+	<xacro:property name="fricCoeff1" value="10.0"/>
+	<xacro:property name="fricCoeff2" value="10.0"/>
+	<xacro:property name="kpCollision" value="10000.0"/>
 	<xacro:property name="kdCollision" value="100000000.0"/>
 	<xacro:macro name="gazebo_links" params="name">
@@ -10,10 +10,10 @@
 			<mu1>${fricCoeff1}</mu1>
 			<mu2>${fricCoeff2}</mu2>
-			<!-- <kp>${kpCollision}</kp> -->
-			<!-- <kd>${kdCollision}</kd> -->
+			<kp>${kpCollision}</kp>
+			<kd>${kdCollision}</kd>
 			<selfCollide>true</selfCollide>
-			<!-- <maxVel>0.01</maxVel> -->
-			<minDepth>0.001</minDepth>
-			<dampingFactor>0.05</dampingFactor>
+			<maxVel>0.00001</maxVel>
+			<minDepth>0.00001</minDepth>
+			<dampingFactor>0.1</dampingFactor>
 		</gazebo>
 	</xacro:macro>
