Commit message: change the way to self rotation of the tool (speed, position) expand the controller for a camera.

File: surgical_sim/models/urdf/surgical_tool/camera_base/camera_base.joints.xacro (robot description, xacro)
@@ -3,5 +3,5 @@
   <xacro:include filename="$(find surgical_sim)/models/urdf/surgical_tool/templates/joint.transmissions.xacro"/>
   <xacro:include filename="$(find surgical_sim)/models/urdf/surgical_tool/templates/gazebo.joints.xacro"/>
-  <xacro:macro name="create_tool_base_joints" params="parent_link xyz rpy tool_id">
+  <xacro:macro name="create_camera_base_joints" params="parent_link xyz rpy tool_id">
     <!-- joint 1: tool_yaw -->
     <joint name="${tool_id}_tool_joint1_pitch" type="revolute">
@@ -38,32 +38,28 @@
       <child link="${tool_id}_tool_main_link"/>
       <axis xyz="0 0 1"/>
-      <origin rpy="0 0 0" xyz="0 0 -${0.4318-0.041}"/>
+      <origin rpy="0 0 0" xyz="0 0 -${0.365}"/>
       <limit lower="0.0" upper="0.240" velocity="10" effort="1000"/>
     </joint>
-    <joint name="${tool_id}_tool_jointf_wrist_fixed" type="fixed">
-      <!-- <safety_controller k_position="100.0" k_velocity="40.0" soft_lower_limit="-1.5" soft_upper_limit="1.5"/> -->
+    <joint name="${tool_id}_tool_wrist_fixed" type="fixed">
       <parent link="${tool_id}_tool_main_link"/>
       <child link="${tool_id}_tool_wrist_link"/>
       <axis xyz="0 0 1"/>
-      <origin rpy="0 0 0" xyz="0 0 ${0.4162-0.041}"/>
+      <origin rpy="0 0 0" xyz="0 0 ${0.365}"/>
     </joint>
     <!-- joint 4-1: tool roll shaft joint FIXED-->
-    <joint name="${tool_id}_tool_jointf_wrist_shaft_fixed" type="fixed">
-      <!-- <safety_controller k_position="100.0" k_velocity="40.0" soft_lower_limit="-1.5" soft_upper_limit="1.5"/> -->
+    <joint name="${tool_id}_tool_tip_link_ee" type="fixed">
       <parent link="${tool_id}_tool_wrist_link"/>
-      <child link="${tool_id}_tool_wrist_shaft_link"/>
+      <child link="${tool_id}_tool_tip_link_ee"/>
       <axis xyz="0 0 1"/>
       <origin rpy="0 0 0" xyz="0 0 0.0"/>
     </joint>
-    <xacro:joint_trans name="${tool_id}_tool_joint1_pitch" reduction="1"/>
-    <xacro:joint_trans name="${tool_id}_tool_joint2_roll" reduction="1"/>
-    <xacro:joint_trans name="${tool_id}_tool_joint3_yaw" reduction="1"/>
-    <xacro:joint_trans name="${tool_id}_tool_joint4_insertion" reduction="1"/>
+    <xacro:joint_trans name="${tool_id}_tool_joint1_pitch" reduction="1" type="PositionJointInterface"/>
+    <xacro:joint_trans name="${tool_id}_tool_joint2_roll" reduction="1" type="PositionJointInterface"/>
+    <xacro:joint_trans name="${tool_id}_tool_joint3_yaw" reduction="1" type="PositionJointInterface"/>
+    <xacro:joint_trans name="${tool_id}_tool_joint4_insertion" reduction="1" type="PositionJointInterface"/>
     <xacro:gazebo_joints name="${tool_id}_tool_joint1_pitch"/>
     <xacro:gazebo_joints name="${tool_id}_tool_joint2_roll"/>
     <xacro:gazebo_joints name="${tool_id}_tool_joint3_yaw"/>
     <xacro:gazebo_joints name="${tool_id}_tool_joint4_insertion"/>
-    <xacro:gazebo_joints name="${tool_id}_tool_jointf_wrist_fixed"/>
-    <xacro:gazebo_joints name="${tool_id}_tool_jointf_wrist_shaft_fixed"/>
   </xacro:macro>
 </robot>

File: surgical_sim/models/urdf/surgical_tool/templates/gazebo.joints.xacro (robot description, xacro)
@@ -4,5 +4,5 @@
 		<gazebo reference="${name}">
 			<!-- <implicitSpringDamper>1</implicitSpringDamper> -->
-			<provideFeedback>1</provideFeedback>
+			<!-- <provideFeedback>1</provideFeedback> -->
 		</gazebo>
 	</xacro:macro>

File: surgical_sim/models/urdf/surgical_tool/templates/gazebo.links.xacro (robot description, xacro)
@@ -12,5 +12,5 @@
 			<!-- <kp>${kpCollision}</kp> -->
 			<!-- <kd>${kdCollision}</kd> -->
-			<!-- <selfCollide>false</selfCollide> -->
+			<selfCollide>false</selfCollide>
 			<maxVel>0.01</maxVel>
 			<minDepth>0.001</minDepth>

File: surgical_sim/models/urdf/surgical_tool/templates/joint.transmissions.xacro (robot description, xacro)
@@ -1,12 +1,12 @@
 <?xml version="1.0"?>
 <robot xmlns:xacro="http://www.ros.org/wiki/xacro">
-	<xacro:macro name="joint_trans" params="name reduction">
+	<xacro:macro name="joint_trans" params="name reduction type:='EffortJointInterface'">
 		<transmission name="${name}_trans">
 			<type>transmission_interface/SimpleTransmission</type>
 			<joint name="${name}">
-				<hardwareInterface>hardware_interface/EffortJointInterface</hardwareInterface>
+				<hardwareInterface>hardware_interface/${type}</hardwareInterface>
 			</joint>
 			<actuator name="${name}_motor">
-				<hardwareInterface>hardware_interface/EffortJointInterface</hardwareInterface>
+				<hardwareInterface>hardware_interface/${type}</hardwareInterface>
 				<mechanicalReduction>${reduction}</mechanicalReduction>
 			</actuator>

File: surgical_sim/models/urdf/surgical_tool/tool.urdf (robot description, URDF)
Before this commit: robot surgical_tool, 14 links, 13 joints
Links:
- removed link right_tool_tip_link
- removed link right_tool_wrist_forceps_link
- removed link right_tool_wrist_forceps_link_2_left
- removed link right_tool_wrist_forceps_link_2_right
- removed link right_tool_wrist_forceps_link_shaft
- removed link right_tool_wrist_shaft_link
- link right_tool_roll_link: mass 0.151 -> 0.05
- link right_tool_tip_link_ee: mass None -> 0.001
- link right_tool_wrist_link: mass 0.05 -> 0.001; geometry 
Joints:
- removed joint right_tool_tip_ee_fixed
- removed joint right_tool_tip_fixed
- removed joint right_tool_wrist_fixed_p
- removed joint right_tool_wrist_fixed_yw
- removed joint right_tool_wrist_open_angle
- removed joint right_tool_wrist_open_angle_mimic
- removed joint right_tool_wrist_shaft_fixed
- added joint right_tool_tip_link_ee: type fixed, parent right_tool_wrist_link, child right_tool_tip_link_ee, origin xyz=0 0 0.0 rpy=0 0 0, axis 0 0 1
- joint right_tool_insertion: limit lower=0.0 upper=0.240 effort=30 velocity=100 -> lower=0.0 upper=0.240 effort=1000 velocity=10; origin xyz=0 0 -0.3908 rpy=0 0 0 -> xyz=0 0 -0.365 rpy=0 0 0
- joint right_tool_pitch: limit lower=-1.5707 upper=1.5707 effort=30 velocity=100 -> lower=-1.5707 upper=1.5707 effort=1000 velocity=10
- joint right_tool_roll: limit lower=-1.5707 upper=1.5707 effort=30 velocity=100 -> lower=-1.5707 upper=1.5707 effort=1000 velocity=10
- joint right_tool_wrist_fixed: origin xyz=0 0 0.3752 rpy=0 0 0 -> xyz=0 0 0.365 rpy=0 0 0
- joint right_tool_yaw: limit lower=-4.71238898038 upper=4.71238898038 effort=30 velocity=100 -> effort=1000 velocity=10; type revolute -> continuous

File: surgical_sim/models/urdf/surgical_tool/tool_create.urdf.xacro (robot description, xacro)
@@ -3,25 +3,13 @@
   <!-- Macros -->
   <!-- Macros -->
+  <xacro:include filename="$(find surgical_sim)/models/urdf/surgical_tool/camera_base/camera_base.urdf.xacro"/>
   <xacro:include filename="$(find surgical_sim)/models/urdf/surgical_tool/tool_base/tool_base.urdf.xacro"/>
   <xacro:include filename="$(find surgical_sim)/models/urdf/surgical_tool/tool_gripper/tool_t_gripper.urdf.xacro"/>
   <xacro:include filename="$(find surgical_sim)/models/urdf/surgical_tool/tool_forceps/tool_t_forceps.urdf.xacro"/>
   <xacro:arg name="with_forceps" default="true"/>
-  <xacro:arg name="with_gripper" default="false"/>
   <xacro:arg name="toolID" default="right"/>
   <xacro:arg name="originTrocar.x" default="0.015"/>
   <xacro:arg name="originTrocar.y" default="0.515"/>
   <xacro:arg name="originTrocar.z" default="1.3"/>
-  <xacro:macro name="attach_gripper" params="parent_link xyz rpy tool_id">
-    <xacro:create_tool_base
-        parent_link="${parent_link}"
-        xyz="${xyz}" rpy="${rpy}" tool_id="${tool_id}"/>
-    <xacro:create_gripper/>
-  </xacro:macro>
-  <xacro:macro name="attach_forceps" params="parent_link xyz rpy tool_id">
-    <xacro:create_tool_base
-        parent_link="${parent_link}"
-        xyz="${xyz}" rpy="${rpy}" tool_id="${tool_id}"/>
-     <xacro:create_forceps tool_id="${tool_id}" connected_to="$(arg toolID)_tool_wrist_shaft_link"/>
-  </xacro:macro>
  <!--  -->
   <link name="world"/>
@@ -34,14 +22,13 @@
   </link>
   <xacro:if value="$(arg with_forceps)">
-    <xacro:attach_forceps
-        parent_link="$(arg toolID)_tool_base_link"
-        xyz="-0.25 0.0 0.5" rpy="0.0 0.0 3.1415926" tool_id="$(arg toolID)"/>
+    <xacro:create_tool_base
+          parent_link="$(arg toolID)_tool_base_link"
+          xyz="-0.25 0.0 0.5" rpy="0.0 0.0 3.1415926" tool_id="$(arg toolID)"/>
+    <xacro:create_forceps tool_id="$(arg toolID)" connected_to="$(arg toolID)_tool_wrist_shaft_link"/>
   </xacro:if>
   <xacro:unless value="$(arg with_forceps)">
-    <xacro:if value="$(arg with_gripper)">
-        <xacro:attach_gripper
-        parent_link="$(arg toolID)_tool_base_link"
-        xyz="-0.25 0.0 0.5" rpy="0.0 0.0 3.1415926" tool_id="$(arg toolID)"/>
-    </xacro:if>
+    <xacro:create_camera_base
+          parent_link="$(arg toolID)_tool_base_link"
+          xyz="-0.25 0.0 0.5" rpy="0.0 0.0 3.1415926" tool_id="$(arg toolID)"/>
   </xacro:unless>
   <joint name="world_fixed" type="fixed">

File: surgical_sim/models/urdf/surgical_tool/tool_forceps/tool_t_forceps.joints.xacro (robot description, xacro)
@@ -5,5 +5,5 @@
   <xacro:macro name="create_forceps_joints" params="tool_id connected_to">
     <!-- joint 5: tool wrist pitch joint -->
-    <joint name="${tool_id}_tool_wrist_pitch" type="fixed">
+    <joint name="${tool_id}_tool_jointf_wrist_pitch" type="fixed">
       <parent link="${connected_to}"/>
       <!-- <parent link="${tool_id}_world"/> -->
@@ -14,5 +14,5 @@
     </joint>
     <!-- joint 6: Tool wrist yaw joint -->
-    <joint name="${tool_id}_tool_wrist_yaw" type="fixed">
+    <joint name="${tool_id}_tool_jointf_wrist_yaw" type="fixed">
       <parent link="${tool_id}_tool_wrist_forceps_link"/>
       <child link="${tool_id}_tool_wrist_forceps_link_shaft"/>
@@ -22,5 +22,5 @@
     </joint>
     <!-- joint 6-1: tool open angle 1 -->
-    <joint name="${tool_id}_tool_wrist_open_angle" type="revolute">
+    <joint name="${tool_id}_tool_joint5_wrist_open_angle" type="revolute">
       <parent link="${tool_id}_tool_wrist_forceps_link_shaft"/>
       <child link="${tool_id}_tool_wrist_forceps_link_2_left"/>
@@ -30,5 +30,5 @@
     </joint>
   <!-- joint 6-2: tool open angle 2  -->
-    <joint name="${tool_id}_tool_wrist_open_angle_mimic" type="revolute">
+    <joint name="${tool_id}_tool_joint5_wrist_open_angle_mimic" type="revolute">
       <parent link="${tool_id}_tool_wrist_forceps_link_shaft"/>
       <child link="${tool_id}_tool_wrist_forceps_link_2_right"/>
@@ -39,10 +39,10 @@
     </joint>
          <!-- tool tip -->
-    <joint name="${tool_id}_tool_tip_" type="fixed">
+    <joint name="${tool_id}_tool_jointf_tip_" type="fixed">
       <parent link="${tool_id}_tool_wrist_forceps_link_shaft"/>
       <child link="${tool_id}_tool_tip_link"/>
       <origin rpy="0 ${pi/2} ${pi/2}" xyz="0 0.0202 0"/>
     </joint>
-    <joint name="${tool_id}_tool_tip_ee" type="fixed">
+    <joint name="${tool_id}_tool_jointf_tip_ee" type="fixed">
       <parent link="${tool_id}_tool_tip_link"/>
       <child link="${tool_id}_tool_tip_link_ee"/>
@@ -51,12 +51,12 @@
     <!-- <xacro:joint_trans name="${tool_id}_tool_wrist_pitch" reduction="1"/>
     <xacro:joint_trans name="${tool_id}_tool_wrist_yaw" reduction="1"/> -->
-    <xacro:joint_trans name="${tool_id}_tool_wrist_open_angle" reduction="1"/>
-    <xacro:joint_trans name="${tool_id}_tool_wrist_open_angle_mimic" reduction="1"/>
-    <xacro:gazebo_joints name="${tool_id}_tool_wrist_pitch"/>
-    <xacro:gazebo_joints name="${tool_id}_tool_wrist_yaw"/>
-    <xacro:gazebo_joints name="${tool_id}_tool_wrist_open_angle"/>
-    <xacro:gazebo_joints name="${tool_id}_tool_wrist_open_angle_mimic"/>
-    <xacro:gazebo_joints name="${tool_id}_tool_tip_"/>
-    <xacro:gazebo_joints name="${tool_id}_tool_tip_ee"/>
+    <xacro:joint_trans name="${tool_id}_tool_joint5_wrist_open_angle" reduction="1"/>
+    <xacro:joint_trans name="${tool_id}_tool_joint5_wrist_open_angle_mimic" reduction="1"/>
+    <xacro:gazebo_joints name="${tool_id}_tool_jointf_wrist_pitch"/>
+    <xacro:gazebo_joints name="${tool_id}_tool_jointf_wrist_yaw"/>
+    <xacro:gazebo_joints name="${tool_id}_tool_joint5_wrist_open_angle"/>
+    <xacro:gazebo_joints name="${tool_id}_tool_joint5_wrist_open_angle_mimic"/>
+    <xacro:gazebo_joints name="${tool_id}_tool_jointf_tip_"/>
+    <xacro:gazebo_joints name="${tool_id}_tool_jointf_tip_ee"/>
   </xacro:macro>
 </robot>

File: surgical_sim/models/urdf/surgical_tool/tool_forceps/tool_t_forceps.links.xacro (robot description, xacro)
@@ -51,5 +51,5 @@
         <origin rpy="0.0 0 0.0" xyz="0 0 0.00195"/>
         <geometry>
-          <mesh filename="package://surgical_sim/models/meshes/stl/tool/tool_wrist_forceps_link_2_left.stl"/>
+          <mesh filename="package://surgical_sim/models/meshes/stl/tool/tool_wrist_forceps_link_fill.stl"/>
         </geometry>
       </collision>
@@ -71,5 +71,5 @@
         <origin rpy="0 0 -3.1415926" xyz="0 0 0.00195"/>
         <geometry>
-          <mesh filename="package://surgical_sim/models/meshes/stl/tool/tool_wrist_forceps_link_2_right.stl"/>
+          <mesh filename="package://surgical_sim/models/meshes/stl/tool/tool_wrist_forceps_link_fill.stl"/>
         </geometry>
       </collision>

File: surgical_sim/models/urdf/target_object/target_object.urdf.xacro (robot description, xacro)
@@ -65,17 +65,17 @@
   <link name="$(arg targetID)_target_main_link">
     <visual>
-      <origin rpy="0 0 0" xyz="0 0 0"/>
+      <origin rpy="0 0 0" xyz="0.0 0.0 0.0"/>
         <geometry>
           <!-- <box size="${sphere_radius} ${2*sphere_radius} ${2*sphere_radius}"/> -->
           <!-- <sphere radius="${sphere_radius}"/> -->
-          <mesh filename="package://surgical_sim/models/meshes/stl/target/target.STL"/>
+          <mesh filename="package://surgical_sim/models/meshes/stl/target/target_translated.STL"/>
         </geometry>
     </visual>
     <collision>
-        <origin rpy="0 0 0" xyz="0 0 0"/>
+        <origin rpy="0 0 0" xyz="0.0 0.0 0.0"/>
         <geometry>
           <!-- <box size="${2*sphere_radius} ${2*sphere_radius} ${2*sphere_radius}"/> -->
           <!-- <sphere radius="${sphere_radius}"/> -->
-          <mesh filename="package://surgical_sim/models/meshes/stl/target/target_2.STL" scale="1.0 1.2 1.0"/>
+          <mesh filename="package://surgical_sim/models/meshes/stl/target/target_translated_collision.STL" scale="1.1 1.1 1.1"/>
         </geometry>
     </collision>

File: surgical_sim/models/urdf/target_object/templates/gazebo.links.xacro (robot description, xacro)
@@ -3,6 +3,6 @@
 	<xacro:property name="fricCoeff1" value="10.0"/>
 	<xacro:property name="fricCoeff2" value="10.0"/>
-	<xacro:property name="kpCollision" value="10000.0"/>
-	<xacro:property name="kdCollision" value="100000000.0"/>
+	<xacro:property name="kpCollision" value="10000000.0"/>
+	<xacro:property name="kdCollision" value="1000000000000.0"/>
 	<xacro:macro name="gazebo_links" params="name">
 		<gazebo reference="${name}">
@@ -10,10 +10,10 @@
 			<mu1>${fricCoeff1}</mu1>
 			<mu2>${fricCoeff2}</mu2>
-			<kp>${kpCollision}</kp>
+			<!-- <kp>${kpCollision}</kp>  -->
 			<kd>${kdCollision}</kd>
 			<selfCollide>true</selfCollide>
-			<maxVel>0.00001</maxVel>
-			<minDepth>0.00001</minDepth>
-			<dampingFactor>0.1</dampingFactor>
+			<maxVel>0.00000001</maxVel>
+			<minDepth>0.0000001</minDepth>
+			<dampingFactor>0.05</dampingFactor>
 		</gazebo>
 	</xacro:macro>

Commit message: fix the relative target for speed control, the limits of the map have to be symmetric if a deadzone in the input is to be used

File: surgical_sim/models/urdf/surgical_tool/camera_base/camera_base.joints.xacro (robot description, xacro)
@@ -11,5 +11,5 @@
       <axis xyz="0 0 1"/>
       <origin rpy="0 -${pi/2} ${pi}" xyz="0.0 0.0 0.0"/>
-      <limit lower="-1.5707" upper="1.5707" velocity="10" effort="1000"/>
+      <limit lower="-${1.0*pi/2}" upper="${1.0*pi/2}" velocity="10" effort="1000"/>
     </joint>
     <!-- joint 2: tool_pitch -->
@@ -20,5 +20,5 @@
       <axis xyz="0 0 1"/>
       <origin rpy="-${pi/2} -${pi/2} 0" xyz="0 0 0"/>
-      <limit lower="-1.5707" upper="1.5707" velocity="10" effort="1000"/>
+      <limit lower="-${1.0*pi/2}" upper="${1.0*pi/2}" velocity="10" effort="1000"/>
     </joint>
     <!-- joint : tool Roll -->
@@ -39,5 +39,5 @@
       <axis xyz="0 0 1"/>
       <origin rpy="0 0 0" xyz="0 0 -${0.365}"/>
-      <limit lower="0.0" upper="0.240" velocity="10" effort="1000"/>
+      <limit lower="0.0" upper="0.260" velocity="10" effort="1000"/>
     </joint>
     <joint name="${tool_id}_tool_wrist_fixed" type="fixed">

File: surgical_sim/models/urdf/surgical_tool/tool_base/tool_base.joints.xacro (robot description, xacro)
@@ -11,5 +11,5 @@
       <axis xyz="0 0 1"/>
       <origin rpy="0 -${pi/2} ${pi}" xyz="0.0 0.0 0.0"/>
-      <limit lower="-1.5707" upper="1.5707" velocity="10" effort="1000"/>
+      <limit lower="-${1.0*pi/2}" upper="${1.0*pi/2}" velocity="10" effort="1000"/>
     </joint>
     <!-- joint 2: tool_pitch -->
@@ -20,5 +20,5 @@
       <axis xyz="0 0 1"/>
       <origin rpy="-${pi/2} -${pi/2} 0" xyz="0 0 0"/>
-      <limit lower="-1.5707" upper="1.5707" velocity="10" effort="1000"/>
+      <limit lower="-${1.0*pi/2}" upper="${1.0*pi/2}" velocity="10" effort="1000"/>
     </joint>
     <!-- joint : tool Roll -->
@@ -39,5 +39,5 @@
       <axis xyz="0 0 1"/>
       <origin rpy="0 0 0" xyz="0 0 -${0.4318-0.041}"/>
-      <limit lower="0.0" upper="0.240" velocity="10" effort="1000"/>
+      <limit lower="0.0" upper="0.26" velocity="10" effort="1000"/>
     </joint>
     <joint name="${tool_id}_tool_jointf_wrist_fixed" type="fixed">
