Commit message: backup 12.11.2021

File: surgical_sim/models/urdf/body/templates/gazebo.links.xacro (robot description, xacro)
@@ -1,6 +1,6 @@
 <?xml version="1.0"?>
 <robot xmlns:xacro="http://www.ros.org/wiki/xacro">
-	<xacro:property name="fricCoeff1" value="0.112"/>
-	<xacro:property name="fricCoeff2" value="0.112"/>
+	<xacro:property name="fricCoeff1" value="1.0"/>
+	<xacro:property name="fricCoeff2" value="1.0"/>
 	<xacro:property name="kpCollision" value="1000000"/>
 	<xacro:property name="kdCollision" value="1"/>

File: surgical_sim/models/urdf/body/torso/torso.links.xacro (robot description, xacro)
@@ -14,5 +14,5 @@
         <origin rpy="${-pi/2} 0 0" xyz="0 0 0"/>
         <geometry>
-          <mesh filename="package://surgical_sim/models/meshes/stl/body/torso_simp.stl"/>
+          <mesh filename="package://surgical_sim/models/meshes/stl/body/torso_simp_2_3.stl"/>
         </geometry>
       </collision>

File: surgical_sim/models/urdf/surgical_tool/templates/gazebo.links.xacro (robot description, xacro)
@@ -1,6 +1,6 @@
 <?xml version="1.0"?>
 <robot xmlns:xacro="http://www.ros.org/wiki/xacro">
-	<xacro:property name="fricCoeff1" value="0.112"/>
-	<xacro:property name="fricCoeff2" value="0.112"/>
+	<xacro:property name="fricCoeff1" value="1000"/>
+	<xacro:property name="fricCoeff2" value="1000"/>
 	<xacro:property name="kpCollision" value="1000000"/>
 	<xacro:property name="kdCollision" value="1"/>

File: surgical_sim/models/urdf/surgical_tool/tool_forceps/tool_t_forceps.joints.xacro (robot description, xacro)
@@ -27,5 +27,5 @@
       <axis xyz="0 0 1"/>
       <origin rpy="0 0 0" xyz="0 0 0"/>
-      <limit lower="${radians(0.0)}" upper="${radians(30.0)}" velocity="3.0" effort="10"/>
+      <limit lower="${radians(0.0)}" upper="${radians(30.0)}" velocity="3.0" effort="20"/>
     </joint>
   <!-- joint 6-2: tool open angle 2  -->
@@ -35,5 +35,5 @@
       <axis xyz="0 0 1"/>
       <origin rpy="3.1415926 0 0" xyz="0 0 0"/>
-      <limit lower="${radians(0.0)}" upper="${radians(30.0)}" velocity="3.0" effort="10"/>
+      <limit lower="${radians(0.0)}" upper="${radians(30.0)}" velocity="3.0" effort="20"/>
       <mimic joint="${tool_id}_tool_wrist_open_angle" multiplier="1"/>
     </joint>

File: surgical_sim/models/urdf/target_object/base_object/base_object.links.xacro (robot description, xacro)
@@ -17,5 +17,5 @@
       <inertial>
 				<origin xyz="0 0 0" rpy="0 0 0"/>
-				<mass value="1"/>
+				<mass value="2"/>
 				<inertia ixx="${2/5 * 1 * 0.019 * 0.019 }" ixy="0.0" ixz="0.0" iyy="${2/5 * 1 * 0.019 * 0.019 }" iyz="0.0" izz="${2/5 * 1 * 0.019 * 0.019 }"/>
 			</inertial>

File: surgical_sim/models/urdf/target_object/target_object.urdf.xacro (robot description, xacro)
@@ -1,13 +1,43 @@
 <?xml version="1.0" ?>
 <robot name="target_object" xmlns:xacro="http://www.ros.org/wiki/xacro">
+  <xacro:include filename="$(find surgical_sim)/models/urdf/target_object/templates/gazebo.links.xacro"/>
+  <xacro:include filename="$(find surgical_sim)/models/urdf/target_object/templates/gazebo.joints.xacro"/>
   <xacro:arg name="parent_link" default="world"/>
-  <xacro:include filename="$(find surgical_sim)/models/urdf/target_object/base_object/base_object.urdf.xacro"/>
-  <link name="world"/>
-  <xacro:create_base_object
-        parent_link="world"
-        xyz="0.0 0.0 0.0" rpy="0.0 0.0 0.0" />
+  <xacro:property name="sphere_radius" value="0.005"/>
+  <xacro:arg name="targetID" default="right"/>
+  <link name="$(arg parent_link)"/>
+  <link name="$(arg targetID)_target_base_link">
+    <visual>
+        <origin rpy="${-pi/2} 0 0" xyz="0 0 0"/>
+        <geometry>
+          <sphere radius="0.007"/>
+        </geometry>
+      <material name="Cyan">
+       <color rgba="0 1.0 1.0 0.5"/>
+     </material>
+    </visual>
+    <collision>
+        <origin rpy="${-pi/2} 0 0" xyz="0 0 0"/>
+        <geometry>
+          <sphere radius="0.007"/>
+        </geometry>
+    </collision>
+      <inertial>
+        <origin xyz="0 0 0" rpy="0 0 0"/>
+        <mass value="10"/>
+        <inertia ixx="${2/5 * 1 * sphere_radius * sphere_radius }" ixy="0.0" ixz="0.0" iyy="${2/5 * 1 * sphere_radius * sphere_radius }" iyz="0.0" izz="${2/5 * 1 * sphere_radius * sphere_radius }"/>
+      </inertial>
+  </link>
+  <joint name="$(arg targetID)_target_base_joint" type="floating">
+     <origin xyz="0.0 0.0 0.0" rpy="0.0 0 0"/>
+     <parent link="$(arg parent_link)"/>
+     <child link="$(arg targetID)_target_base_link"/>
+  </joint>
+    <xacro:gazebo_links name="$(arg parent_link)"/>
+    <xacro:gazebo_links name="$(arg targetID)_base_link"/>
+    <xacro:gazebo_joints name="$(arg targetID)_base_joint"/>
     <gazebo>
         <plugin name="gazebo_ros_control" filename="libgazebo_ros_control.so">
-        <robotNamespace>/target_object</robotNamespace>
+        <robotNamespace>/$(arg targetID)_target</robotNamespace>
         <robotSimType>gazebo_ros_control/DefaultRobotHWSim</robotSimType>
         <legacyModeNS>true</legacyModeNS>

File: surgical_sim/models/urdf/target_object/templates/gazebo.links.xacro (robot description, xacro)
@@ -1,16 +1,16 @@
 <?xml version="1.0"?>
 <robot xmlns:xacro="http://www.ros.org/wiki/xacro">
-	<xacro:property name="fricCoeff1" value="0.112"/>
-	<xacro:property name="fricCoeff2" value="0.112"/>
-	<xacro:property name="kpCollision" value="1000000"/>
-	<xacro:property name="kdCollision" value="1"/>
+	<xacro:property name="fricCoeff1" value="1000"/>
+	<xacro:property name="fricCoeff2" value="1000"/>
+	<xacro:property name="kpCollision" value="10.0"/>
+	<xacro:property name="kdCollision" value="10.0"/>
 	<xacro:macro name="gazebo_links" params="name">
 		<gazebo reference="${name}">
-			<turnGravityOff>true</turnGravityOff>
+			<turnGravityOff>false</turnGravityOff>
 			<mu1>${fricCoeff1}</mu1>
 			<mu2>${fricCoeff2}</mu2>
 			<kp>${kpCollision}</kp>
 			<kd>${kdCollision}</kd>
-			<selfCollide>true</selfCollide>
+			<selfCollide>false</selfCollide>
 			<maxVel>0.01</maxVel>
 			<minDepth>0.003</minDepth>

Commit message: modified grasping needle simulation

File: surgical_sim/models/urdf/body/templates/gazebo.links.xacro (robot description, xacro)
@@ -1,7 +1,6 @@
 <?xml version="1.0"?>
 <robot xmlns:xacro="http://www.ros.org/wiki/xacro">
-	<xacro:property name="fricCoeff1" value="1.0"/>
-	<xacro:property name="fricCoeff2" value="1.0"/>
-	<xacro:property name="kpCollision" value="1000000"/>
+	<xacro:property name="fricCoeff1" value="0.1"/>
+	<xacro:property name="fricCoeff2" value="0.1"/>
 	<xacro:property name="kdCollision" value="1"/>
 	<xacro:macro name="gazebo_links" params="name">
@@ -10,9 +9,8 @@
 			<mu1>${fricCoeff1}</mu1>
 			<mu2>${fricCoeff2}</mu2>
-			<kp>${kpCollision}</kp>
 			<kd>${kdCollision}</kd>
 			<selfCollide>true</selfCollide>
 			<maxVel>0.01</maxVel>
-			<minDepth>0.003</minDepth>
+			<minDepth>0.001</minDepth>
 		</gazebo>
 	</xacro:macro>

File: surgical_sim/models/urdf/surgical_tool/templates/gazebo.links.xacro (robot description, xacro)
@@ -3,5 +3,5 @@
 	<xacro:property name="fricCoeff1" value="1000"/>
 	<xacro:property name="fricCoeff2" value="1000"/>
-	<xacro:property name="kpCollision" value="1000000"/>
+	<!-- <xacro:property name="kpCollision" value="100000000"/> -->
 	<xacro:property name="kdCollision" value="1"/>
 	<xacro:macro name="gazebo_links" params="name">
@@ -10,9 +10,9 @@
 			<mu1>${fricCoeff1}</mu1>
 			<mu2>${fricCoeff2}</mu2>
-			<kp>${kpCollision}</kp>
-			<kd>${kdCollision}</kd>
-			<selfCollide>false</selfCollide>
+			<!-- <kp>${kpCollision}</kp> -->
+			<!-- <kd>${kdCollision}</kd> -->
+			<!-- <selfCollide>false</selfCollide> -->
 			<maxVel>0.01</maxVel>
-			<minDepth>0.003</minDepth>
+			<minDepth>0.0001</minDepth>
 		</gazebo>
 	</xacro:macro>

File: surgical_sim/models/urdf/surgical_tool/templates/joint.transmissions.xacro (robot description, xacro)
@@ -5,8 +5,8 @@
 			<type>transmission_interface/SimpleTransmission</type>
 			<joint name="${name}">
-				<hardwareInterface>hardware_interface/PositionJointInterface</hardwareInterface>
+				<hardwareInterface>hardware_interface/EffortJointInterface</hardwareInterface>
 			</joint>
 			<actuator name="${name}_motor">
-				<hardwareInterface>hardware_interface/PositionJointInterface</hardwareInterface>
+				<hardwareInterface>hardware_interface/EffortJointInterface</hardwareInterface>
 				<mechanicalReduction>${reduction}</mechanicalReduction>
 			</actuator>

File: surgical_sim/models/urdf/surgical_tool/tool_base/tool_base.joints.xacro (robot description, xacro)
@@ -11,5 +11,5 @@
       <axis xyz="0 0 1"/>
       <origin rpy="0 -${pi/2} ${pi}" xyz="0.0 0.0 0.0"/>
-      <limit lower="-1.5707" upper="1.5707" velocity="100" effort="30"/>
+      <limit lower="-1.5707" upper="1.5707" velocity="10" effort="1000"/>
     </joint>
     <!-- joint 2: tool_pitch -->
@@ -20,5 +20,5 @@
       <axis xyz="0 0 1"/>
       <origin rpy="-${pi/2} -${pi/2} 0" xyz="0 0 0"/>
-      <limit lower="-1.5707" upper="1.5707" velocity="100" effort="30"/>
+      <limit lower="-1.5707" upper="1.5707" velocity="10" effort="1000"/>
     </joint>
     <!-- joint : tool Roll -->
@@ -29,5 +29,5 @@
       <axis xyz="0 0 1"/>
       <origin rpy="${pi/2} 0 0" xyz="0 0 0"/>
-      <limit velocity="2" effort="10"/>
+      <limit velocity="10" effort="1000"/>
       <!-- <limit lower="-${1.5 * pi}" upper="${1.5 * pi}" velocity="2" effort="2"/> -->
     </joint>
@@ -39,5 +39,5 @@
       <axis xyz="0 0 1"/>
       <origin rpy="0 0 0" xyz="0 0 -${0.4318-0.041}"/>
-      <limit lower="0.0" upper="0.240" velocity="100" effort="30"/>
+      <limit lower="0.0" upper="0.240" velocity="10" effort="1000"/>
     </joint>
     <joint name="${tool_id}_tool_wrist_fixed" type="fixed">

File: surgical_sim/models/urdf/surgical_tool/tool_base/tool_base.links.xacro (robot description, xacro)
@@ -10,6 +10,6 @@
       <inertial>
 				<origin xyz="0 0 0" rpy="0 0 0"/>
-				<mass value="0.05"/>
-				<inertia ixx="0.01" ixy="0.0" ixz="0.0" iyy="0.01" iyz="0.0" izz="0.005"/>
+				<mass value="0.005"/>
+				<inertia ixx="0.0001" ixy="0.0" ixz="0.0" iyy="0.0001" iyz="0.0" izz="0.0005"/>
 			</inertial>
     </link>
@@ -18,6 +18,6 @@
       <inertial>
 				<origin xyz="0 0 0" rpy="0 0 0"/>
-				<mass value="0.05"/>
-				<inertia ixx="0.01" ixy="0.0" ixz="0.0" iyy="0.01" iyz="0.0" izz="0.005"/>
+				<mass value="0.005"/>
+				<inertia ixx="0.0001" ixy="0.0" ixz="0.0" iyy="0.0001" iyz="0.0" izz="0.0005"/>
 			</inertial>
     </link>
@@ -25,6 +25,6 @@
       <inertial>
 				<origin xyz="0 0 0" rpy="0 0 0"/>
-				<mass value="0.151"/>
-				<inertia ixx="0.01" ixy="0.0" ixz="0.0" iyy="0.01" iyz="0.0" izz="0.005"/>
+				<mass value="0.005"/>
+				<inertia ixx="0.0001" ixy="0.0" ixz="0.0" iyy="0.0001" iyz="0.0" izz="0.0005"/>
 			</inertial>
     </link>

File: surgical_sim/models/urdf/surgical_tool/tool_create.urdf.xacro (robot description, xacro)
@@ -53,5 +53,5 @@
     <gazebo>
         <plugin name="gazebo_ros_control" filename="libgazebo_ros_control.so">
-        <robotNamespace>$(arg toolID)_tool</robotNamespace>
+        <robotNamespace>/$(arg toolID)_tool</robotNamespace>
         <robotParam>/$(arg toolID)_tool/robot_description</robotParam>
         <robotSimType>gazebo_ros_control/DefaultRobotHWSim</robotSimType>

File: surgical_sim/models/urdf/surgical_tool/tool_forceps/tool_t_forceps.joints.xacro (robot description, xacro)
@@ -11,5 +11,5 @@
       <axis xyz="0 0 1"/>
       <origin rpy="-1.5708 -1.5708 ${pi}" xyz="0 0 0"/>
-      <limit lower="-${pi/2}" upper="${pi/2}" velocity="3.0" effort="2"/>
+      <!-- <limit lower="-${pi/2}" upper="${pi/2}" velocity="3.0" effort="2"/> -->
     </joint>
     <!-- joint 6: Tool wrist yaw joint -->
@@ -19,5 +19,5 @@
       <axis xyz="0 0 1"/>
       <origin rpy="0.00 -1.5708 -1.5708" xyz="0.0091 0 0"/>
-      <limit lower="-${pi/2}" upper="${pi/2}" velocity="3.0" effort="2"/>
+      <!-- <limit lower="-${pi/2}" upper="${pi/2}" velocity="3.0" effort="2"/> -->
     </joint>
     <!-- joint 6-1: tool open angle 1 -->
@@ -27,5 +27,5 @@
       <axis xyz="0 0 1"/>
       <origin rpy="0 0 0" xyz="0 0 0"/>
-      <limit lower="${radians(0.0)}" upper="${radians(30.0)}" velocity="3.0" effort="20"/>
+      <limit lower="${radians(0.0)}" upper="${radians(30.0)}" velocity=".4" effort="1000"/>
     </joint>
   <!-- joint 6-2: tool open angle 2  -->
@@ -35,5 +35,5 @@
       <axis xyz="0 0 1"/>
       <origin rpy="3.1415926 0 0" xyz="0 0 0"/>
-      <limit lower="${radians(0.0)}" upper="${radians(30.0)}" velocity="3.0" effort="20"/>
+      <limit lower="${radians(0.0)}" upper="${radians(30.0)}" velocity=".4" effort="1000"/>
       <mimic joint="${tool_id}_tool_wrist_open_angle" multiplier="1"/>
     </joint>

File: surgical_sim/models/urdf/surgical_tool/tool_forceps/tool_t_forceps.links.xacro (robot description, xacro)
@@ -27,4 +27,11 @@
         <material name="gray"><color rgba="0.5 0.5 0.9 1.0"/></material>
       </visual>
+      <collision>
+        <origin rpy="0.00 1.5708 0.0" xyz="0.0 -0.0002 0.000"/>
+        <geometry>
+          <mesh filename="package://surgical_sim/models/meshes/stl/tool/tool_wrist_forceps_link_1_shaft.stl"/>
+        </geometry>
+        <material name="gray"><color rgba="0.5 0.5 0.9 1.0"/></material>
+      </collision>
       <inertial>
 				<origin xyz="0 0 0" rpy="0 0 0"/>

File: surgical_sim/models/urdf/target_object/target_object.urdf.xacro (robot description, xacro)
@@ -3,38 +3,116 @@
   <xacro:include filename="$(find surgical_sim)/models/urdf/target_object/templates/gazebo.links.xacro"/>
   <xacro:include filename="$(find surgical_sim)/models/urdf/target_object/templates/gazebo.joints.xacro"/>
+  <xacro:property name="sphere_radius" value="0.005"/>
+  <xacro:property name="linear_lim" value="0.02"/>
+  <xacro:property name="mass_x" value="0.0001"/>
+  <xacro:property name="mass_y" value="0.0001"/>
+  <xacro:property name="mass_z" value="0.001"/>
+  <xacro:property name="mass_main" value="0.001"/>
+  <xacro:arg name="targetID" default="right_t1"/>
   <xacro:arg name="parent_link" default="world"/>
-  <xacro:property name="sphere_radius" value="0.005"/>
-  <xacro:arg name="targetID" default="right"/>
   <link name="$(arg parent_link)"/>
   <link name="$(arg targetID)_target_base_link">
+      <inertial>
+        <origin xyz="0 0 0" rpy="0 0 0"/>
+        <mass value="${mass_x}"/>
+        <inertia ixx="${2/5 * mass_x * sphere_radius * sphere_radius }" ixy="0.0" ixz="0.0" iyy="${2/5 * mass_x * sphere_radius * sphere_radius }" iyz="0.0" izz="${2/5 * mass_x * sphere_radius * sphere_radius }"/>
+      </inertial>
+  </link>
+  <link name="$(arg targetID)_target_y_link">
+      <inertial>
+        <origin xyz="0 0 0" rpy="0 0 0"/>
+        <mass value="${mass_y}"/>
+        <inertia ixx="${2/5 * mass_y * sphere_radius * sphere_radius }" ixy="0.0" ixz="0.0" iyy="${2/5 * mass_y * sphere_radius * sphere_radius }" iyz="0.0" izz="${2/5 * mass_y * sphere_radius * sphere_radius }"/>
+      </inertial>
+  </link>
+  <link name="$(arg targetID)_target_z_link">
+      <inertial>
+        <origin xyz="0 0 0" rpy="0 0 0"/>
+        <mass value="${mass_z}"/>
+        <inertia ixx="${2/5 * mass_z * sphere_radius * sphere_radius }" ixy="0.0" ixz="0.0" iyy="${2/5 * mass_z * sphere_radius * sphere_radius }" iyz="0.0" izz="${2/5 * mass_z * sphere_radius * sphere_radius }"/>
+      </inertial>
+  </link>
+   <link name="$(arg targetID)_target_z2_link">
+      <inertial>
+        <origin xyz="0 0 0" rpy="0 0 0"/>
+        <mass value="${mass_z}"/>
+        <inertia ixx="${2/5 * mass_z * sphere_radius * sphere_radius }" ixy="0.0" ixz="0.0" iyy="${2/5 * mass_z * sphere_radius * sphere_radius }" iyz="0.0" izz="${2/5 * mass_z * sphere_radius * sphere_radius }"/>
+      </inertial>
+  </link>
+  <link name="$(arg targetID)_target_main_link">
     <visual>
-        <origin rpy="${-pi/2} 0 0" xyz="0 0 0"/>
+      <origin rpy="0 0 0" xyz="0 0 0"/>
         <geometry>
-          <sphere radius="0.007"/>
+          <!-- <box size="${sphere_radius} ${2*sphere_radius} ${2*sphere_radius}"/> -->
+          <!-- <sphere radius="${sphere_radius}"/> -->
+          <mesh filename="package://surgical_sim/models/meshes/stl/target/target.STL"/>
         </geometry>
-      <material name="Cyan">
-       <color rgba="0 1.0 1.0 0.5"/>
-     </material>
     </visual>
     <collision>
-        <origin rpy="${-pi/2} 0 0" xyz="0 0 0"/>
+        <origin rpy="0 0 0" xyz="0 0 0"/>
         <geometry>
-          <sphere radius="0.007"/>
+          <!-- <box size="${2*sphere_radius} ${2*sphere_radius} ${2*sphere_radius}"/> -->
+          <!-- <sphere radius="${sphere_radius}"/> -->
+          <mesh filename="package://surgical_sim/models/meshes/stl/target/target.STL"/>
         </geometry>
     </collision>
-      <inertial>
-        <origin xyz="0 0 0" rpy="0 0 0"/>
-        <mass value="10"/>
-        <inertia ixx="${2/5 * 1 * sphere_radius * sphere_radius }" ixy="0.0" ixz="0.0" iyy="${2/5 * 1 * sphere_radius * sphere_radius }" iyz="0.0" izz="${2/5 * 1 * sphere_radius * sphere_radius }"/>
-      </inertial>
+    <inertial>
+      <origin
+        xyz="-0.0027704 -0.00060187 -1.79059999999631E-08"
+        rpy="0 0 0" />
+      <mass
+        value="0.000037311" />
+      <inertia
+        ixx="2.99391393770835E-08"
+        ixy="-1.99518680567514E-09"
+        ixz="2.72589485952597E-15"
+        iyy="8.27991394391801E-09"
+        iyz="3.38023650313121E-14"
+        izz="3.77117809466761E-08" />
+    </inertial>
   </link>
-  <joint name="$(arg targetID)_target_base_joint" type="floating">
+  <joint name="$(arg targetID)_target_base_joint" type="fixed">
      <origin xyz="0.0 0.0 0.0" rpy="0.0 0 0"/>
      <parent link="$(arg parent_link)"/>
      <child link="$(arg targetID)_target_base_link"/>
   </joint>
-    <xacro:gazebo_links name="$(arg parent_link)"/>
-    <xacro:gazebo_links name="$(arg targetID)_base_link"/>
-    <xacro:gazebo_joints name="$(arg targetID)_base_joint"/>
+  <joint name="$(arg targetID)_target_x_joint" type="prismatic">
+     <origin xyz="0.0 0.0 0.0" rpy="0.0 0 0"/>
+     <axis xyz="1.0 0.0 0.0"/>
+     <parent link="$(arg targetID)_target_base_link"/>
+     <child link="$(arg targetID)_target_y_link"/>
+     <limit lower="-${linear_lim}" upper="${linear_lim}" effort="1000.0" velocity=".4"/>
+  </joint>
+  <joint name="$(arg targetID)_target_y_joint" type="prismatic">
+     <origin xyz="0.0 0.0 0.0" rpy="0.0 0 0"/>
+     <axis xyz="0.0 1.0 0.0"/>
+     <parent link="$(arg targetID)_target_y_link"/>
+     <child link="$(arg targetID)_target_z_link"/>
+     <limit lower="-${linear_lim}" upper="${linear_lim}" effort="1000.0" velocity=".4"/>
+  </joint>
+  <joint name="$(arg targetID)_target_z_joint" type="prismatic">
+     <origin xyz="0.0 0.0 0.0" rpy="0.0 0 0"/>
+     <axis xyz="0.0 0.0 1.0"/>
+     <parent link="$(arg targetID)_target_z_link"/>
+     <child link="$(arg targetID)_target_z2_link"/>
+     <limit lower="-${0.5*linear_lim}" upper="${2*linear_lim}" effort="1000.0" velocity=".4"/>
+  </joint>
+   <joint name="$(arg targetID)_target_z2_joint" type="continuous">
+     <origin xyz="0.0 0.0 0.0" rpy="0.0 0 0"/>
+     <axis xyz="0.0 0.0 1.0"/>
+     <parent link="$(arg targetID)_target_z2_link"/>
+     <child link="$(arg targetID)_target_main_link"/>
+     <limit effort="1000.0" velocity=".4"/>
+  </joint>
+  <xacro:gazebo_links name="$(arg parent_link)"/>
+  <xacro:gazebo_links name="$(arg targetID)_target_base_link"/>
+  <xacro:gazebo_links name="$(arg targetID)_target_y_link"/>
+  <xacro:gazebo_links name="$(arg targetID)_target_z_link"/>
+  <xacro:gazebo_links name="$(arg targetID)_target_main_link"/>
+  <xacro:gazebo_joints name="$(arg targetID)_base_joint"/>
+  <xacro:gazebo_joints name="$(arg targetID)_x_joint"/>
+  <xacro:gazebo_joints name="$(arg targetID)_y_joint"/>
+  <xacro:gazebo_joints name="$(arg targetID)_z_joint"/>
+  <xacro:gazebo_joints name="$(arg targetID)_z2_joint"/>
     <gazebo>
         <plugin name="gazebo_ros_control" filename="libgazebo_ros_control.so">

File: surgical_sim/models/urdf/target_object/templates/gazebo.joints.xacro (robot description, xacro)
@@ -3,9 +3,6 @@
 	<xacro:macro name="gazebo_joints" params="name">
 		<gazebo reference="${name}">
-			<implicitSpringDamper>0</implicitSpringDamper>
-			<provideFeedback>1</provideFeedback>
-			<!--stopCfm></stopCfm--> <!-- Force Mixing Error -->
-			<!--stopErp></stopErp--> <!-- Error Reduction Parameter -->
-			<!-- <fudgeFactor>0.5</fudgeFactor> -->
+			<!-- <implicitSpringDamper>0</implicitSpringDamper>
+			<provideFeedback>1</provideFeedback> -->
 		</gazebo>
 	</xacro:macro>

File: surgical_sim/models/urdf/target_object/templates/gazebo.links.xacro (robot description, xacro)
@@ -3,6 +3,6 @@
 	<xacro:property name="fricCoeff1" value="1000"/>
 	<xacro:property name="fricCoeff2" value="1000"/>
-	<xacro:property name="kpCollision" value="10.0"/>
-	<xacro:property name="kdCollision" value="10.0"/>
+	<xacro:property name="kpCollision" value="100000000.0"/>
+	<xacro:property name="kdCollision" value="1.0"/>
 	<xacro:macro name="gazebo_links" params="name">
 		<gazebo reference="${name}">
@@ -10,9 +10,9 @@
 			<mu1>${fricCoeff1}</mu1>
 			<mu2>${fricCoeff2}</mu2>
-			<kp>${kpCollision}</kp>
-			<kd>${kdCollision}</kd>
-			<selfCollide>false</selfCollide>
-			<maxVel>0.01</maxVel>
-			<minDepth>0.003</minDepth>
+			<!-- <kp>${kpCollision}</kp> -->
+			<!-- <kd>${kdCollision}</kd> -->
+			<selfCollide>true</selfCollide>
+			<!-- <maxVel>0.01</maxVel> -->
+			<!-- <minDepth>0.003</minDepth-->
 		</gazebo>
 	</xacro:macro>
