Commit message: fix bug. never use damping tag in joints

File: surgical_sim/models/urdf/body/templates/gazebo.links.xacro (robot description, xacro)
@@ -9,5 +9,5 @@
 			<mu1>${fricCoeff1}</mu1>
 			<mu2>${fricCoeff2}</mu2>
-			<kd>${kdCollision}</kd>
+			<!-- <kd>${kdCollision}</kd> -->
 			<selfCollide>true</selfCollide>
 			<maxVel>0.01</maxVel>

File: surgical_sim/models/urdf/surgical_tool/templates/gazebo.joints.xacro (robot description, xacro)
@@ -3,6 +3,6 @@
 	<xacro:macro name="gazebo_joints" params="name">
 		<gazebo reference="${name}">
-			<!-- <implicitSpringDamper>0</implicitSpringDamper>
-			<provideFeedback>1</provideFeedback> -->
+			<!-- <implicitSpringDamper>1</implicitSpringDamper> -->
+			<provideFeedback>1</provideFeedback>
 		</gazebo>
 	</xacro:macro>

File: surgical_sim/models/urdf/surgical_tool/templates/gazebo.links.xacro (robot description, xacro)
@@ -1,18 +1,18 @@
 <?xml version="1.0"?>
 <robot xmlns:xacro="http://www.ros.org/wiki/xacro">
-	<xacro:property name="fricCoeff1" value="1000"/>
-	<xacro:property name="fricCoeff2" value="1000"/>
+	<!-- <xacro:property name="fricCoeff1" value="10.0"/> -->
+	<!-- <xacro:property name="fricCoeff2" value="10.0"/> -->
 	<!-- <xacro:property name="kpCollision" value="100000000"/> -->
 	<xacro:property name="kdCollision" value="1"/>
-	<xacro:macro name="gazebo_links" params="name">
+	<xacro:macro name="gazebo_links" params="name frictCoeff:=0.12">
 		<gazebo reference="${name}">
 			<turnGravityOff>true</turnGravityOff>
-			<mu1>${fricCoeff1}</mu1>
-			<mu2>${fricCoeff2}</mu2>
+			<mu1>${frictCoeff}</mu1>
+			<mu2>${frictCoeff}</mu2>
 			<!-- <kp>${kpCollision}</kp> -->
 			<!-- <kd>${kdCollision}</kd> -->
 			<!-- <selfCollide>false</selfCollide> -->
 			<maxVel>0.01</maxVel>
-			<minDepth>0.0001</minDepth>
+			<minDepth>0.001</minDepth>
 		</gazebo>
 	</xacro:macro>

File: surgical_sim/models/urdf/surgical_tool/tool_base/tool_base.links.xacro (robot description, xacro)
@@ -10,6 +10,6 @@
       <inertial>
 				<origin xyz="0 0 0" rpy="0 0 0"/>
-				<mass value="0.005"/>
-				<inertia ixx="0.0001" ixy="0.0" ixz="0.0" iyy="0.0001" iyz="0.0" izz="0.0005"/>
+				<mass value="0.05"/>
+				<inertia ixx="0.01" ixy="0.0" ixz="0.0" iyy="0.01" iyz="0.0" izz="0.005"/>
 			</inertial>
     </link>
@@ -18,6 +18,6 @@
       <inertial>
 				<origin xyz="0 0 0" rpy="0 0 0"/>
-				<mass value="0.005"/>
-				<inertia ixx="0.0001" ixy="0.0" ixz="0.0" iyy="0.0001" iyz="0.0" izz="0.0005"/>
+				<mass value="0.05"/>
+				<inertia ixx="0.01" ixy="0.0" ixz="0.0" iyy="0.01" iyz="0.0" izz="0.005"/>
 			</inertial>
     </link>
@@ -25,6 +25,6 @@
       <inertial>
 				<origin xyz="0 0 0" rpy="0 0 0"/>
-				<mass value="0.005"/>
-				<inertia ixx="0.0001" ixy="0.0" ixz="0.0" iyy="0.0001" iyz="0.0" izz="0.0005"/>
+				<mass value="0.05"/>
+				<inertia ixx="0.01" ixy="0.0" ixz="0.0" iyy="0.01" iyz="0.0" izz="0.005"/>
 			</inertial>
     </link>

File: surgical_sim/models/urdf/surgical_tool/tool_forceps/tool_t_forceps.links.xacro (robot description, xacro)
@@ -14,6 +14,6 @@
       <inertial>
           <origin xyz="0 0 0" rpy="0 0 0"/>
-          <mass value="0.1"/>
-          <inertia ixx="1" ixy="0.0" ixz="0.0" iyy="1" iyz="0.0" izz="0.05"/>
+          <mass value="0.05"/>
+				  <inertia ixx="0.01" ixy="0.0" ixz="0.0" iyy="0.01" iyz="0.0" izz="0.005"/>
 			</inertial>
     </link>
@@ -36,6 +36,6 @@
       <inertial>
 				<origin xyz="0 0 0" rpy="0 0 0"/>
-				<mass value="0.1"/>
-        <inertia ixx="0.1" ixy="0.0" ixz="0.0" iyy="0.1" iyz="0.0" izz="0.005"/>
+				<mass value="0.05"/>
+				<inertia ixx="0.01" ixy="0.0" ixz="0.0" iyy="0.01" iyz="0.0" izz="0.005"/>
 			</inertial>
     </link>
@@ -84,6 +84,6 @@
     <xacro:gazebo_links name="${tool_id}_tool_wrist_forceps_link"/>
     <xacro:gazebo_links name="${tool_id}_tool_wrist_forceps_link_shaft"/>
-    <xacro:gazebo_links name="${tool_id}_tool_wrist_forceps_link_2_left"/>
-    <xacro:gazebo_links name="${tool_id}_tool_wrist_forceps_link_2_right"/>
+    <xacro:gazebo_links name="${tool_id}_tool_wrist_forceps_link_2_left" frictCoeff="10.0"/>
+    <xacro:gazebo_links name="${tool_id}_tool_wrist_forceps_link_2_right" frictCoeff="10.0"/>
     <xacro:gazebo_links name="${tool_id}_tool_tip_link"/>
     <xacro:gazebo_links name="${tool_id}_tool_tip_link_ee"/>

File: surgical_sim/models/urdf/target_object/target_object.urdf.xacro (robot description, xacro)
@@ -3,18 +3,23 @@
   <xacro:include filename="$(find surgical_sim)/models/urdf/target_object/templates/gazebo.links.xacro"/>
   <xacro:include filename="$(find surgical_sim)/models/urdf/target_object/templates/gazebo.joints.xacro"/>
-  <xacro:property name="sphere_radius" value="0.005"/>
   <xacro:property name="linear_lim" value="0.02"/>
   <xacro:property name="mass_x" value="0.0001"/>
   <xacro:property name="mass_y" value="0.0001"/>
   <xacro:property name="mass_z" value="0.001"/>
-  <xacro:property name="mass_main" value="0.001"/>
+  <xacro:property name="mass_main" value="0.00037311"/>
   <xacro:arg name="targetID" default="right_t1"/>
   <xacro:arg name="parent_link" default="world"/>
   <link name="$(arg parent_link)"/>
-  <link name="$(arg targetID)_target_base_link">
+ <link name="$(arg targetID)_target_base_link">
       <inertial>
         <origin xyz="0 0 0" rpy="0 0 0"/>
         <mass value="${mass_x}"/>
-        <inertia ixx="${2/5 * mass_x * sphere_radius * sphere_radius }" ixy="0.0" ixz="0.0" iyy="${2/5 * mass_x * sphere_radius * sphere_radius }" iyz="0.0" izz="${2/5 * mass_x * sphere_radius * sphere_radius }"/>
+        <inertia
+        ixx="${2.99391393770835E-08 * mass_x/mass_main}"
+        ixy="${-1.99518680567514E-09 * mass_x/mass_main}"
+        ixz="${2.72589485952597E-15 * mass_x/mass_main}"
+        iyy="${8.27991394391801E-09 * mass_x/mass_main}"
+        iyz="${3.38023650313121E-14 * mass_x/mass_main}"
+        izz="${3.77117809466761E-08 * mass_x/mass_main}" />
       </inertial>
   </link>
@@ -23,5 +28,11 @@
         <origin xyz="0 0 0" rpy="0 0 0"/>
         <mass value="${mass_y}"/>
-        <inertia ixx="${2/5 * mass_y * sphere_radius * sphere_radius }" ixy="0.0" ixz="0.0" iyy="${2/5 * mass_y * sphere_radius * sphere_radius }" iyz="0.0" izz="${2/5 * mass_y * sphere_radius * sphere_radius }"/>
+       <inertia
+        ixx="${2.99391393770835E-08 * mass_y/mass_main}"
+        ixy="${-1.99518680567514E-09 * mass_y/mass_main}"
+        ixz="${2.72589485952597E-15 * mass_y/mass_main}"
+        iyy="${8.27991394391801E-09 * mass_y/mass_main}"
+        iyz="${3.38023650313121E-14 * mass_y/mass_main}"
+        izz="${3.77117809466761E-08 * mass_y/mass_main}" />
       </inertial>
   </link>
@@ -30,5 +41,11 @@
         <origin xyz="0 0 0" rpy="0 0 0"/>
         <mass value="${mass_z}"/>
-        <inertia ixx="${2/5 * mass_z * sphere_radius * sphere_radius }" ixy="0.0" ixz="0.0" iyy="${2/5 * mass_z * sphere_radius * sphere_radius }" iyz="0.0" izz="${2/5 * mass_z * sphere_radius * sphere_radius }"/>
+        <inertia
+        ixx="${2.99391393770835E-08 * mass_z/mass_main}"
+        ixy="${-1.99518680567514E-09 * mass_z/mass_main}"
+        ixz="${2.72589485952597E-15 * mass_z/mass_main}"
+        iyy="${8.27991394391801E-09 * mass_z/mass_main}"
+        iyz="${3.38023650313121E-14 * mass_z/mass_main}"
+        izz="${3.77117809466761E-08 * mass_z/mass_main}" />
       </inertial>
   </link>
@@ -37,5 +54,11 @@
         <origin xyz="0 0 0" rpy="0 0 0"/>
         <mass value="${mass_z}"/>
-        <inertia ixx="${2/5 * mass_z * sphere_radius * sphere_radius }" ixy="0.0" ixz="0.0" iyy="${2/5 * mass_z * sphere_radius * sphere_radius }" iyz="0.0" izz="${2/5 * mass_z * sphere_radius * sphere_radius }"/>
+        <inertia
+        ixx="${2.99391393770835E-08 * mass_z/mass_main}"
+        ixy="${-1.99518680567514E-09 * mass_z/mass_main}"
+        ixz="${2.72589485952597E-15 * mass_z/mass_main}"
+        iyy="${8.27991394391801E-09 * mass_z/mass_main}"
+        iyz="${3.38023650313121E-14 * mass_z/mass_main}"
+        izz="${3.77117809466761E-08 * mass_z/mass_main}" />
       </inertial>
   </link>
@@ -54,5 +77,5 @@
           <!-- <box size="${2*sphere_radius} ${2*sphere_radius} ${2*sphere_radius}"/> -->
           <!-- <sphere radius="${sphere_radius}"/> -->
-          <mesh filename="package://surgical_sim/models/meshes/stl/target/target.STL"/>
+          <mesh filename="package://surgical_sim/models/meshes/stl/target/target_2.STL" scale="1.0 1.2 1.0"/>
         </geometry>
     </collision>
@@ -62,5 +85,5 @@
         rpy="0 0 0" />
       <mass
-        value="0.000037311" />
+        value="${mass_main}" />
       <inertia
         ixx="2.99391393770835E-08"
@@ -110,9 +133,9 @@
   <xacro:gazebo_links name="$(arg targetID)_target_z_link"/>
   <xacro:gazebo_links name="$(arg targetID)_target_main_link"/>
-  <xacro:gazebo_joints name="$(arg targetID)_base_joint"/>
-  <xacro:gazebo_joints name="$(arg targetID)_x_joint"/>
-  <xacro:gazebo_joints name="$(arg targetID)_y_joint"/>
-  <xacro:gazebo_joints name="$(arg targetID)_z_joint"/>
-  <xacro:gazebo_joints name="$(arg targetID)_z2_joint"/>
+  <xacro:gazebo_joints name="$(arg targetID)_target_base_joint"/>
+  <xacro:gazebo_joints name="$(arg targetID)_target_x_joint"/>
+  <xacro:gazebo_joints name="$(arg targetID)_target_y_joint"/>
+  <xacro:gazebo_joints name="$(arg targetID)_target_z_joint"/>
+  <xacro:gazebo_joints name="$(arg targetID)_target_z2_joint"/>
     <gazebo>
         <plugin name="gazebo_ros_control" filename="libgazebo_ros_control.so">

File: surgical_sim/models/urdf/target_object/templates/gazebo.links.xacro (robot description, xacro)
@@ -1,8 +1,8 @@
 <?xml version="1.0"?>
 <robot xmlns:xacro="http://www.ros.org/wiki/xacro">
-	<xacro:property name="fricCoeff1" value="1000"/>
-	<xacro:property name="fricCoeff2" value="1000"/>
+	<xacro:property name="fricCoeff1" value="2.0"/>
+	<xacro:property name="fricCoeff2" value="2.0"/>
 	<xacro:property name="kpCollision" value="100000000.0"/>
-	<xacro:property name="kdCollision" value="1.0"/>
+	<xacro:property name="kdCollision" value="100000000.0"/>
 	<xacro:macro name="gazebo_links" params="name">
 		<gazebo reference="${name}">
@@ -10,9 +10,10 @@
 			<mu1>${fricCoeff1}</mu1>
 			<mu2>${fricCoeff2}</mu2>
-			<!-- <kp>${kpCollision}</kp> -->
-			<!-- <kd>${kdCollision}</kd> -->
+			<kp>${kpCollision}</kp>
+			<kd>${kdCollision}</kd>
 			<selfCollide>true</selfCollide>
 			<!-- <maxVel>0.01</maxVel> -->
-			<!-- <minDepth>0.003</minDepth-->
+			<minDepth>0.001</minDepth>
+			<dampingFactor>0.05</dampingFactor>
 		</gazebo>
 	</xacro:macro>

Commit message: now grasping is easier. changed the collision of tip of the tool. Introduced torsional friction....

File: surgical_sim/models/urdf/body/templates/gazebo.links.xacro (robot description, xacro)
@@ -1,6 +1,6 @@
 <?xml version="1.0"?>
 <robot xmlns:xacro="http://www.ros.org/wiki/xacro">
-	<xacro:property name="fricCoeff1" value="0.1"/>
-	<xacro:property name="fricCoeff2" value="0.1"/>
+	<xacro:property name="fricCoeff1" value="0.0"/>
+	<xacro:property name="fricCoeff2" value="0.0"/>
 	<xacro:property name="kdCollision" value="1"/>
 	<xacro:macro name="gazebo_links" params="name">
@@ -9,8 +9,9 @@
 			<mu1>${fricCoeff1}</mu1>
 			<mu2>${fricCoeff2}</mu2>
+			<!-- <kinematic>1</kinematic> -->
 			<!-- <kd>${kdCollision}</kd> -->
 			<selfCollide>true</selfCollide>
-			<maxVel>0.01</maxVel>
-			<minDepth>0.001</minDepth>
+			<maxVel>1</maxVel>
+			<minDepth>0.000000001</minDepth>
 		</gazebo>
 	</xacro:macro>

File: surgical_sim/models/urdf/body/torso/torso.links.xacro (robot description, xacro)
@@ -14,5 +14,5 @@
         <origin rpy="${-pi/2} 0 0" xyz="0 0 0"/>
         <geometry>
-          <mesh filename="package://surgical_sim/models/meshes/stl/body/torso_simp_2_3.stl"/>
+          <mesh filename="package://surgical_sim/models/meshes/stl/body/torso_simp_2_3.stl" scale="1.0 1.0 1.0"/>
         </geometry>
       </collision>

File: surgical_sim/models/urdf/surgical_tool/templates/gazebo.links.xacro (robot description, xacro)
@@ -14,5 +14,5 @@
 			<selfCollide>false</selfCollide>
 			<maxVel>0.01</maxVel>
-			<minDepth>0.001</minDepth>
+			<minDepth>0.0000001</minDepth>
 		</gazebo>
 	</xacro:macro>

File: surgical_sim/models/urdf/surgical_tool/tool_base/tool_base.joints.xacro (robot description, xacro)
@@ -39,5 +39,5 @@
       <axis xyz="0 0 1"/>
       <origin rpy="0 0 0" xyz="0 0 -${0.4318-0.041}"/>
-      <limit lower="0.0" upper="0.26" velocity="10" effort="1000"/>
+      <limit lower="0.0" upper="0.36" velocity="10" effort="1000"/>
     </joint>
     <joint name="${tool_id}_tool_jointf_wrist_fixed" type="fixed">

File: surgical_sim/models/urdf/surgical_tool/tool_forceps/tool_t_forceps.links.xacro (robot description, xacro)
@@ -51,5 +51,5 @@
         <origin rpy="0.0 0 0.0" xyz="0 0 0.00195"/>
         <geometry>
-          <mesh filename="package://surgical_sim/models/meshes/stl/tool/tool_wrist_forceps_link_fill.stl"/>
+          <mesh filename="package://surgical_sim/models/meshes/stl/tool/tool_wrist_forceps_link_fill_cube_3.stl"/>
         </geometry>
       </collision>
@@ -60,5 +60,5 @@
 			</inertial>
     </link>
-  <!-- link 6-2: Outer open angle link 2 -->
+  <!-- link 3-2: Outer open angle link 2 -->
     <link name="${tool_id}_tool_wrist_forceps_link_2_right">
       <visual>
@@ -71,5 +71,5 @@
         <origin rpy="0 0 -3.1415926" xyz="0 0 0.00195"/>
         <geometry>
-          <mesh filename="package://surgical_sim/models/meshes/stl/tool/tool_wrist_forceps_link_fill.stl"/>
+          <mesh filename="package://surgical_sim/models/meshes/stl/tool/tool_wrist_forceps_link_fill_cube_6.stl"/>
         </geometry>
       </collision>
@@ -83,7 +83,7 @@
     <link name="${tool_id}_tool_tip_link_ee"/>
     <xacro:gazebo_links name="${tool_id}_tool_wrist_forceps_link"/>
-    <xacro:gazebo_links name="${tool_id}_tool_wrist_forceps_link_shaft"/>
-    <xacro:gazebo_links name="${tool_id}_tool_wrist_forceps_link_2_left" frictCoeff="0.2"/>
-    <xacro:gazebo_links name="${tool_id}_tool_wrist_forceps_link_2_right" frictCoeff="0.2"/>
+    <xacro:gazebo_links name="${tool_id}_tool_wrist_forceps_link_shaft" frictCoeff="10.0"/>
+    <xacro:gazebo_links name="${tool_id}_tool_wrist_forceps_link_2_left" frictCoeff="5.0"/>
+    <xacro:gazebo_links name="${tool_id}_tool_wrist_forceps_link_2_right" frictCoeff="5.0"/>
     <xacro:gazebo_links name="${tool_id}_tool_tip_link"/>
     <xacro:gazebo_links name="${tool_id}_tool_tip_link_ee"/>

File: surgical_sim/models/urdf/target_object/target_object.urdf.xacro (robot description, xacro)
@@ -4,8 +4,9 @@
   <xacro:include filename="$(find surgical_sim)/models/urdf/target_object/templates/gazebo.joints.xacro"/>
   <xacro:property name="linear_lim" value="0.02"/>
-  <xacro:property name="mass_x" value="0.0001"/>
-  <xacro:property name="mass_y" value="0.0001"/>
+  <xacro:property name="mass_x" value="0.001"/>
+  <xacro:property name="mass_y" value="0.001"/>
   <xacro:property name="mass_z" value="0.001"/>
-  <xacro:property name="mass_main" value="0.00037311"/>
+  <xacro:property name="mass_main" value="0.000337311"/>
+  <xacro:property name="mass_" value="0.01"/>
   <xacro:arg name="targetID" default="right_t1"/>
   <xacro:arg name="parent_link" default="world"/>
@@ -72,10 +73,10 @@
         </geometry>
     </visual>
-    <collision>
+    <collision name="$(arg targetID)_target_main_link_collision">
         <origin rpy="0 0 0" xyz="0.0 0.0 0.0"/>
         <geometry>
           <!-- <box size="${2*sphere_radius} ${2*sphere_radius} ${2*sphere_radius}"/> -->
           <!-- <sphere radius="${sphere_radius}"/> -->
-          <mesh filename="package://surgical_sim/models/meshes/stl/target/target_translated_collision.STL" scale="1.1 1.1 1.1"/>
+          <mesh filename="package://surgical_sim/models/meshes/stl/target/target_translated_collision.STL" scale="1.2 1.1 1.1"/>
         </geometry>
     </collision>
@@ -85,12 +86,12 @@
         rpy="0 0 0" />
       <mass
-        value="${mass_main}" />
-      <inertia
-        ixx="2.99391393770835E-08"
-        ixy="-1.99518680567514E-09"
-        ixz="2.72589485952597E-15"
-        iyy="8.27991394391801E-09"
-        iyz="3.38023650313121E-14"
-        izz="3.77117809466761E-08" />
+        value="${mass_}" />
+              <inertia
+        ixx="${2.99391393770835E-08 * mass_/mass_main}"
+        ixy="${-1.99518680567514E-09 * mass_/mass_main}"
+        ixz="${2.72589485952597E-15 * mass_/mass_main}"
+        iyy="${8.27991394391801E-09 * mass_/mass_main}"
+        iyz="${3.38023650313121E-14 * mass_/mass_main}"
+        izz="${3.77117809466761E-08 * mass_/mass_main}" />
     </inertial>
   </link>
@@ -105,5 +106,5 @@
      <parent link="$(arg targetID)_target_base_link"/>
      <child link="$(arg targetID)_target_y_link"/>
-     <limit lower="-${linear_lim}" upper="${linear_lim}" effort="1000.0" velocity=".4"/>
+     <limit lower="-${linear_lim}" upper="${linear_lim}" effort="1000.0" velocity="10.0"/>
   </joint>
   <joint name="$(arg targetID)_target_y_joint" type="prismatic">
@@ -112,5 +113,5 @@
      <parent link="$(arg targetID)_target_y_link"/>
      <child link="$(arg targetID)_target_z_link"/>
-     <limit lower="-${linear_lim}" upper="${linear_lim}" effort="1000.0" velocity=".4"/>
+     <limit lower="-${linear_lim}" upper="${linear_lim}" effort="1000.0" velocity="10.0"/>
   </joint>
   <joint name="$(arg targetID)_target_z_joint" type="prismatic">
@@ -119,5 +120,5 @@
      <parent link="$(arg targetID)_target_z_link"/>
      <child link="$(arg targetID)_target_z2_link"/>
-     <limit lower="-${0.5*linear_lim}" upper="${2*linear_lim}" effort="1000.0" velocity=".4"/>
+     <limit lower="-${0.05*linear_lim}" upper="${2*linear_lim}" effort="1000.0" velocity="10.0"/>
   </joint>
    <joint name="$(arg targetID)_target_z2_joint" type="continuous">
@@ -126,5 +127,5 @@
      <parent link="$(arg targetID)_target_z2_link"/>
      <child link="$(arg targetID)_target_main_link"/>
-     <limit effort="1000.0" velocity=".4"/>
+     <limit effort="1000.0" velocity="10.0"/>
   </joint>
   <xacro:gazebo_links name="$(arg parent_link)"/>
@@ -132,5 +133,26 @@
   <xacro:gazebo_links name="$(arg targetID)_target_y_link"/>
   <xacro:gazebo_links name="$(arg targetID)_target_z_link"/>
-  <xacro:gazebo_links name="$(arg targetID)_target_main_link"/>
+  <!-- <xacro:gazebo_links name="$(arg targetID)_target_main_link"/> -->
+	<gazebo reference="$(arg targetID)_target_main_link">
+			<turnGravityOff>false</turnGravityOff>
+			<mu1>200</mu1>
+			<mu2>200</mu2>
+			<kd>10000000000000000000000.0</kd>
+			<selfCollide>true</selfCollide>
+			<maxVel>0.000001</maxVel>
+			<minDepth>1</minDepth>
+			<dampingFactor>0.05</dampingFactor>
+      <collision name="$(arg targetID)_target_main_link_collision">
+      <surface>
+        <friction>
+          <torsional>
+            <coefficient>1.0</coefficient>
+            <use_patch_radius>true</use_patch_radius>
+            <patch_radius>0.05</patch_radius>
+          </torsional>
+        </friction>
+      </surface>
+    </collision>
+	</gazebo>
   <xacro:gazebo_joints name="$(arg targetID)_target_base_joint"/>
   <xacro:gazebo_joints name="$(arg targetID)_target_x_joint"/>

File: surgical_sim/models/urdf/target_object/templates/gazebo.joints.xacro (robot description, xacro)
@@ -3,5 +3,5 @@
 	<xacro:macro name="gazebo_joints" params="name">
 		<gazebo reference="${name}">
-			<implicitSpringDamper>0</implicitSpringDamper>
+			<!-- <implicitSpringDamper>0</implicitSpringDamper> -->
 			<!--provideFeedback>1</provideFeedback> -->
 		</gazebo>

File: surgical_sim/models/urdf/target_object/templates/gazebo.links.xacro (robot description, xacro)
@@ -1,8 +1,8 @@
 <?xml version="1.0"?>
 <robot xmlns:xacro="http://www.ros.org/wiki/xacro">
-	<xacro:property name="fricCoeff1" value="10.0"/>
-	<xacro:property name="fricCoeff2" value="10.0"/>
+	<xacro:property name="fricCoeff1" value="0.01"/>
+	<xacro:property name="fricCoeff2" value="0.01"/>
 	<xacro:property name="kpCollision" value="10000000.0"/>
-	<xacro:property name="kdCollision" value="1000000000000.0"/>
+	<xacro:property name="kdCollision" value="100000000000000000000.0"/>
 	<xacro:macro name="gazebo_links" params="name">
 		<gazebo reference="${name}">
@@ -11,9 +11,10 @@
 			<mu2>${fricCoeff2}</mu2>
 			<!-- <kp>${kpCollision}</kp>  -->
-			<kd>${kdCollision}</kd>
+			<!-- <kd>${kdCollision}</kd> -->
 			<selfCollide>true</selfCollide>
-			<maxVel>0.00000001</maxVel>
-			<minDepth>0.0000001</minDepth>
+			<maxVel>0.01</maxVel>
+			<minDepth>0.01</minDepth>
 			<dampingFactor>0.05</dampingFactor>
+			<!-- <maxContacts>5</maxContacts> -->
 		</gazebo>
 	</xacro:macro>
