Commit message: include again the kinematic simulations with random variable size of the target.

File: surgical_sim/models/urdf/surgical_tool/tool_forceps/tool_t_forceps.links.xacro (robot description, xacro)
@@ -65,5 +65,5 @@
         <origin rpy="0 0 -3.1415926" xyz="0 0 0.00195"/>
         <geometry>
-          <mesh filename="package://surgical_sim/models/meshes/stl/tool/tool_wrist_forceps_link_2_right.stl"/>
+          <mesh filename="package://surgical_sim/models/meshes/stl/tool/tool_wrist_forceps_link_2_left.stl"/>
         </geometry>
       </visual>
@@ -71,5 +71,5 @@
         <origin rpy="0 0 -3.1415926" xyz="0 0 0.00195"/>
         <geometry>
-          <mesh filename="package://surgical_sim/models/meshes/stl/tool/tool_wrist_forceps_link_fill_cube_6.stl"/>
+          <mesh filename="package://surgical_sim/models/meshes/stl/tool/tool_wrist_forceps_link_fill_cube_3.stl"/>
         </geometry>
       </collision>
