Commit message: changes in the origin args for urdf. noetic doesn't accept .x .y it has to be _x _y

File: surgical_sim/models/urdf/body/body_create.urdf.xacro (robot description, xacro)
@@ -6,16 +6,16 @@
   <xacro:arg name="with_liver" default="false"/>
   <xacro:arg name="attached_to" default="world"/>
-  <xacro:arg name="bodyOrigin.x" default="0.0"/>
-  <xacro:arg name="bodyOrigin.y" default="0.5"/>
-  <xacro:arg name="bodyOrigin.z" default="1.1"/>
-  <xacro:arg name="bodyOrigin.ax" default="0.0"/>
-  <xacro:arg name="bodyOrigin.ay" default="0.0"/>
-  <xacro:arg name="bodyOrigin.az" default="0.0"/>
+  <xacro:arg name="bodyOrigin_x" default="0.0"/>
+  <xacro:arg name="bodyOrigin_y" default="0.5"/>
+  <xacro:arg name="bodyOrigin_z" default="1.1"/>
+  <xacro:arg name="bodyOrigin_ax" default="0.0"/>
+  <xacro:arg name="bodyOrigin_ay" default="0.0"/>
+  <xacro:arg name="bodyOrigin_az" default="0.0"/>
  <!--                                                   -->
   <link name="$(arg attached_to)"/>
    <xacro:create_torso
         parent_link="$(arg attached_to)"
-        xyz="$(arg bodyOrigin.x) $(arg bodyOrigin.y) $(arg bodyOrigin.z)"
-        rpy="$(arg bodyOrigin.ax) $(arg bodyOrigin.ay) $(arg bodyOrigin.az)"/>
+        xyz="$(arg bodyOrigin_x) $(arg bodyOrigin_y) $(arg bodyOrigin_z)"
+        rpy="$(arg bodyOrigin_ax) $(arg bodyOrigin_ay) $(arg bodyOrigin_az)"/>
   <!-- <xacro:if value="$(arg with_liver)">
     <xacro:attach_liver

File: surgical_sim/models/urdf/franka/panda_arm.urdf.xacro (robot description, xacro)
@@ -3,10 +3,10 @@
 	<xacro:arg name="gazebo" default="true"/>
 	<xacro:arg name="arm_id" default="right"/>
-  <xacro:arg name="origin.x" default="0"/>
-  <xacro:arg name="origin.y" default="0"/>
-  <xacro:arg name="origin.z" default="0"/>
-  <xacro:arg name="origin.ax" default="0"/>
-  <xacro:arg name="origin.ay" default="0"/>
-  <xacro:arg name="origin.az" default="0"/>
+  <xacro:arg name="origin_x" default="0"/>
+  <xacro:arg name="origin_y" default="0"/>
+  <xacro:arg name="origin_z" default="0"/>
+  <xacro:arg name="origin_ax" default="0"/>
+  <xacro:arg name="origin_ay" default="0"/>
+  <xacro:arg name="origin_az" default="0"/>
   <gazebo reference="world">
   </gazebo>
@@ -14,4 +14,4 @@
   	<xacro:arg name="gazebo" value="${gazebo}"/>
   </xacro:include>
-  <xacro:panda_arm connected_to='world' arm_id="$(arg arm_id)" xyz='$(arg origin.x) $(arg origin.y) $(arg origin.z)' rpy='$(arg origin.ax) $(arg origin.ay) $(arg origin.az)'/>
+  <xacro:panda_arm connected_to='world' arm_id="$(arg arm_id)" xyz='$(arg origin_x) $(arg origin_y) $(arg origin_z)' rpy='$(arg origin_ax) $(arg origin_ay) $(arg origin_az)'/>
 </robot>

File: surgical_sim/models/urdf/surgical_tool/tool_create.urdf.xacro (robot description, xacro)
@@ -9,7 +9,7 @@
   <xacro:arg name="with_forceps" default="true"/>
   <xacro:arg name="toolID" default="right"/>
-  <xacro:arg name="originTrocar.x" default="0.015"/>
-  <xacro:arg name="originTrocar.y" default="0.515"/>
-  <xacro:arg name="originTrocar.z" default="1.3"/>
+  <xacro:arg name="originTrocar_x" default="0.015"/>
+  <xacro:arg name="originTrocar_y" default="0.515"/>
+  <xacro:arg name="originTrocar_z" default="1.3"/>
  <!--  -->
   <link name="world"/>
@@ -35,5 +35,5 @@
       <parent link="world"/>
       <child link="$(arg toolID)_tool_base_link"/>
-      <origin rpy="0 0 0" xyz="$(arg originTrocar.x) $(arg originTrocar.y) $(arg originTrocar.z)"/>
+      <origin rpy="0 0 0" xyz="$(arg originTrocar_x) $(arg originTrocar_y) $(arg originTrocar_z)"/>
   </joint>
   <xacro:gazebo_links name="$(arg toolID)_tool_base_link"/>
